File: hardware/amod_a.kicad_sch (KiCad schematic)
At the start: 114 parts, among them J101 USB-C, J102 rails, J1101 SMA, J1102 TX, J1103 RX, J1104 Pmod, J201 SMA, J202 SMA, J301 SMA, J302 SMA, J401 SMA, J402 SMA, J501 SMA, J502 R, J601 SMA, J801 SMA, Q1101 AO3401A, Q201 AO3401A, Q301 AO3401A, Q401 AO3401A, Q501 AO3401A, Q601 AO3401A, Q801 AO3401A, Q802 AO3400A, SW1101 ON, SW201 ON, SW301 ON, SW401 ON, SW501 ON, SW502 DIP2, SW601 ON, SW801 ON, U101 LM2664, U102 3.3V, U1101 DRV8837, U1102 OPA810, U201 OPA810, U301 OPA810, U401 OPA847, U501 LT6230, U601 TLV3501, U801 TMP235

Commit message: AMOD-A A7 (4046 PLL) and A9 (MC1496 mixer) at DRC 0; the Pmod corridor moved left of A9's LO jack; 0402 passives
Co-Authored-By: Claude Fable 5.1 <noreply@anthropic.com>
Claude-Session: https://claude.ai/code/session_01RKeoKvFFzjk3cEBLCXXHnB
Parts:
- added C701, C702, C704: 100n, Capacitor_SMD:C_0402_1005Metric, symbol Device:C
- added C703: 1n, Capacitor_SMD:C_0402_1005Metric, symbol Device:C
- added C901, C902, C903, C904, C905: 100n, Capacitor_SMD:C_0603_1608Metric, symbol Device:C
- added J701, J702, J901, J902, J903: SMA, amod:SMA_BWSMA-KE-Z001_Vertical, symbol Connector:Conn_Coaxial
- added Q701, Q901: AO3401A, Package_TO_SOT_SMD:SOT-23, symbol Transistor_FET:AO3401A
- added R701, R902: 1k, Resistor_SMD:R_0402_1005Metric, symbol Device:R_US
- added R702, R703: 10k, Resistor_SMD:R_0402_1005Metric, symbol Device:R_US
- added R704: 470, Resistor_SMD:R_0402_1005Metric, symbol Device:R_US
- added R901, R903, R907, R908: 51, Resistor_SMD:R_0402_1005Metric, symbol Device:R_US
- added R904: 3.9k, Resistor_SMD:R_0402_1005Metric, symbol Device:R_US
- added R905: 1.5k, Resistor_SMD:R_0402_1005Metric, symbol Device:R_US
- added R906: 1.5k, Resistor_SMD:R_0805_2012Metric, symbol Device:R_US
- added R909, R910: 10k, Resistor_SMD:R_0603_1608Metric, symbol Device:R_US
- added SW701, SW901: ON, amod:SW_SPDT_Shouhan_MSK12C02, symbol Switch:SW_SPDT
- added U701: HC4046, Package_SO:SOIC-16_3.9x9.9mm_P1.27mm, symbol 4xxx:4046
- added U901: MC1496, Package_SO:SOIC-14_3.9x8.7mm_P1.27mm, symbol amod:MC1496
Connections:
- net +5V: now also Q701.2 (S), Q901.2 (S), SW701.3 (C), SW901.3 (C)
- net -5V: now also R904.2, U901.14 (VEE)
- net GND: now also C702.2, C704.2, C903.2, C904.2, J701.2 (Ext), J702.2 (Ext), J901.2 (Ext), J902.2 (Ext), J903.2 (Ext), R703.2, R901.2, R903.2, R910.2, SW701.1 (A), SW901.1 (A), U701.5 (Inh), U701.8 (VSS)
- new net A7_C1A: C703.2, U701.6 (C1)
- new net A7_C1B: C703.1, U701.7 (C2)
- new net A7_G: Q701.1 (G), SW701.2 (B)
- new net A7_IN: C701.1, J701.1 (In)
- new net A7_INA: C701.2, R701.1
- new net A7_NODE: C702.1, R702.2, U701.9 (VCOin)
- new net A7_OUT: J702.1 (In), R704.1
- new net A7_PC2: R702.1, U701.13 (PC2)
- new net A7_R1: R703.1, U701.11 (R1)
- new net A7_SIG: R701.2, U701.14 (SigIn)
- new net A7_VCO_A: R704.2, U701.3 (RefIn), U701.4 (FOUT)
- new net A7_VS: C704.1, Q701.3 (D), U701.16 (VDD)
- new net A9_BIAS: R904.1, U901.5 (BIAS)
- new net A9_CARA: C902.2, R908.1, U901.8 (CAR+)
- new net A9_CARB: R907.1, U901.10 (CAR-)
- new net A9_CB: C903.1, R907.2, R908.2, R909.2, R910.1
- new net A9_G: Q901.1 (G), SW901.2 (B)
- new net A9_GAIN2: R902.1, U901.2 (GAIN)
- new net A9_GAIN3: R902.2, U901.3 (GAIN)
- new net A9_IF: C905.2, J903.1 (In)
- new net A9_LO: C902.1, J902.1 (In)
- new net A9_OUTA: C905.1, R905.1, U901.6 (OUT+), U901.7 (NC)
- new net A9_OUTB: R906.1, U901.12 (OUT-)
- new net A9_RF: C901.1, J901.1 (In)
- new net A9_SIGA: C901.2, R901.1, U901.1 (SIG+)
- new net A9_SIGB: R903.1, U901.4 (SIG-)
- new net A9_VS: C904.1, Q901.3 (D), R905.2, R906.2, R909.1
- no-connect marks 17 -> 25
Other:
- note added: "A7 PLL 4046"
- note added: "A9 mixer, MC1496"
- note added: "CD74HC4046A: R1 10 k, C1 1 nF put the VCO near 100 kHz (R2 open: it can go down to 0). PC2 (the edge-triggered"
- note added: "EXPECT: IF OUT = RF x LO (sum and difference frequencies, about 0.3 V peak per volt of RF at 0.3 V of LO); a balanced mixer, the carrier mostly cancels"
- note added: "EXPECT: VCO OUT locks to a 50-200 kHz square or sine on IN; pin 9 is the demodulated FM, pin 13 the phase detector"
- note added: "Gilbert cell on +-5 V: signal pair at ground (51 ohm), carrier pair at 2.5 V (51 ohm to the 10 k / 10 k bias), 1 mA"
- note added: "IF"
- note added: "LO"
- note added: "RF"
- note added: "cell (1,1)"
- note added: "cells (0,2), (1,2)"
- note added: "per side (3.9 k), 1.5 k loads. Keep RF under 0.3 V and LO near 0.3 V peak (above that the carrier pair just switches,"
- note added: "through 100 n / 1 k (any level above 0.4 V peak). VCO OUT is 5 V CMOS through 470 ohm. Probe pins 9 and 13."
- note added: "tri-state detector) through 10 k / 100 n into VCOin: a lag filter, so expect ringing on lock. IN self-biases"
- note added: "tutorial 1.10, 6.02 (+-5 V)"
- note added: "tutorial 4.01 (+5 V)"
- note added: "which is fine for a product detector). IF OUT is single-ended from pin 6 through 100 n: a 1.5 k source, so read it"
- note added: "with a high-impedance input, not 50 ohm. No carrier-null trimmer: expect -40 dB of LO feedthrough."
- note added: "±0.3 V"
- note added: "±1 V"

Commit message: AMOD-A complete: A10 (light) and A12 (audio) at DRC 0; all twelve tiles, the Pmod lines and the -5 V pour across both gutters
Co-Authored-By: Claude Fable 5.1 <noreply@anthropic.com>
Claude-Session: https://claude.ai/code/session_01RKeoKvFFzjk3cEBLCXXHnB
Parts:
- added C1001: 10p, Capacitor_SMD:C_0805_2012Metric, symbol Device:C
- added C1002, C1003, C1004, C1005, C1205: 100n, Capacitor_SMD:C_0603_1608Metric, symbol Device:C
- added C1201, C1207: 1u, Capacitor_SMD:C_0805_2012Metric, symbol Device:C
- added C1202: 10n, Capacitor_SMD:C_0805_2012Metric, symbol Device:C
- added C1203, C1204: 1u, Capacitor_SMD:C_0603_1608Metric, symbol Device:C
- added C1206: 10u, Capacitor_SMD:C_0805_2012Metric, symbol Device:C
- added C1208, C1209: 100n, Capacitor_SMD:C_0805_2012Metric, symbol Device:C
- added D1001: PD70, amod:Photodiode_PD70-01C, symbol Device:D_Photo
- added J1001, J1002, J1201, J1202: SMA, amod:SMA_BWSMA-KE-Z001_Vertical, symbol Connector:Conn_Coaxial
- added J1203: SPK, amod:TerminalBlock_KF301_1x02_P5.00mm, symbol Connector:Screw_Terminal_01x02
- added J1204: MIC, Connector_PinSocket_2.54mm:PinSocket_1x02_P2.54mm_Vertical, symbol Connector_Generic:Conn_01x02
- added LED1001: LED, amod:LED_SideView_3.2x1.0mm_E6C1204, symbol Device:LED
- added Q1001, Q1201: AO3401A, Package_TO_SOT_SMD:SOT-23, symbol Transistor_FET:AO3401A
- added Q1002: 2N7002, Package_TO_SOT_SMD:SOT-23, symbol Transistor_FET:2N7002
- added R1001, R1004, R1201: 10k, Resistor_SMD:R_0603_1608Metric, symbol Device:R_US
- added R1002, R1205: 49.9, Resistor_SMD:R_0805_2012Metric, symbol Device:R_US
- added R1003: 1k, Resistor_SMD:R_0805_2012Metric, symbol Device:R_US
- added R1005: 22, Resistor_SMD:R_0805_2012Metric, symbol Device:R_US
- added R1202: 2.2k, Resistor_SMD:R_0805_2012Metric, symbol Device:R_US
- added R1203: 10k, Resistor_SMD:R_0805_2012Metric, symbol Device:R_US
- added R1204: 100R, Resistor_SMD:R_0805_2012Metric, symbol Device:R_US
- added SW1001, SW1201: ON, amod:SW_SPDT_Shouhan_MSK12C02, symbol Switch:SW_SPDT
- added TP1201: OUT, amod:TestPoint_Loop_RH-5019, symbol Connector:TestPoint
- added U1001, U1002, U1202: OPA810, Package_TO_SOT_SMD:SOT-23-5, symbol amod:OPA_SOT23-5
- added U1201: PAM8302A, Package_SO:SOIC-8_3.9x4.9mm_P1.27mm, symbol amod:PAM8302_SOIC8
Connections:
- net +5V: now also Q1001.2 (S), Q1201.2 (S), SW1001.3 (C), SW1201.3 (C)
- net -5V: now also C1002.1, C1004.1, C1209.1, U1001.2 (V-), U1002.2 (V-), U1202.2 (V-)
- net GND: now also C1002.2, C1003.2, C1004.2, C1005.2, C1202.2, C1203.2, C1204.2, C1205.2, C1206.2, C1208.2, C1209.2, J1001.2 (Ext), J1002.2 (Ext), J1201.2 (Ext), J1202.2 (Ext), J1204.2 (Pin_2), Q1002.2 (S), R1004.2, R1005.2, R1204.2, SW1001.1 (A), SW1201.1 (A), U1001.3 (+IN), U1201.7 (GND)
- net PMOD7: now reaches J1104.6 (Pin_6)
- net PMOD7: now also R1201.2
- net PMOD4: now reaches J1104.7 (Pin_7)
- net PMOD4: now also Q1002.1 (G), R1004.1
- new net A10_DRV: J1002.1 (In), R1003.2
- new net A10_DRV_O: LED1001.2 (A), U1002.1 (OUT)
- new net A10_FB: C1001.2, D1001.2 (A), R1001.2, U1001.4 (-IN)
- new net A10_G: Q1001.1 (G), SW1001.2 (B)
- new net A10_INP: Q1002.3 (D), R1003.1, U1002.3 (+IN)
- new net A10_OUTA: C1001.1, R1001.1, R1002.2, U1001.1 (OUT)
- new net A10_PD: J1001.1 (In), R1002.1
- new net A10_SENSE: LED1001.1 (K), R1005.1, U1002.4 (-IN)
- new net A10_VS: C1003.1, C1005.1, D1001.1 (K), Q1001.3 (D), U1001.5 (V+), U1002.5 (V+)
- new net A12_AIN: C1201.1, J1201.1 (In)
- new net A12_BYP: C1204.1, U1201.2 (BYP)
- new net A12_FB: R1203.2, R1204.1, U1202.4 (-IN)
- new net A12_G: Q1201.1 (G), SW1201.2 (B)
- new net A12_IN: C1207.2, U1202.3 (+IN)
- new net A12_INM: C1203.1, U1201.4 (IN-)
- new net A12_MICP: C1207.1, J1204.1 (Pin_1), R1202.2
- new net A12_NODE: C1201.2, C1202.1, R1201.1, U1201.3 (IN+)
- new net A12_OUT: J1202.1 (In), R1205.2, TP1201.1
- new net A12_OUT_A: R1203.1, R1205.1, U1202.1 (OUT)
- new net A12_VOM: J1203.2 (Pin_2), U1201.8 (VO-)
- new net A12_VOP: J1203.1 (Pin_1), U1201.5 (VO+)
- new net A12_VS: C1205.1, C1206.1, C1208.1, Q1201.3 (D), R1202.1, U1201.1 (SD), U1201.6 (VDD), U1202.5 (V+)
- no-connect marks 25 -> 23
Other:
- note added: "+ side, 2.2 k from VS) through 1 u into an OPA810 at x100: a few hundred millivolts for speech."
- note added: "0-1 V"
- note added: "A10 light, LED + PD"
- note added: "A12 audio"
- note added: "AIN"
- note added: "DRV"
- note added: "EXPECT: 45 mA of LED current per volt on DRIVE IN (0-1 V, blanked while Pmod 4 is high); PD OUT climbs 10 V per mA of photocurrent"
- note added: "EXPECT: a speaker on SPK follows AUDIO IN (2.5 W into 4 ohm) or the one-bit stream on Pmod 7 (10 k / 10 n); MIC OUT is the electret x100"
- note added: "PAM8302A: 1 u couples AUDIO IN to IN+ (IN- grounded through 1 u), the one-bit DAC on Pmod 7 arrives through 10 k"
- note added: "PD"
- note added: "The current source: the op amp holds 22 ohm at the input voltage, so the LED carries V / 22 ohm (0.9 V is the LED's"
- note added: "a few MHz. The photodiode (5 V reverse) into 10 k with 10 pF: 1.6 MHz; daylight on the PD gives millivolts, the LED"
- note added: "cells (2,2), (3,2)"
- note added: "cells (2,3), (3,3)"
- note added: "full 40 mA; above 1.1 V the op amp runs out of headroom). A 2N7002 from Pmod 4 shorts the input: TTL modulation to"
- note added: "into 10 n (1.6 kHz) at the same node, so both play. BYP 1 u, SD high: on with the tile. The electret (pin 1 is the"
- note added: "of a second board across a desk gives tens. The LED looks out of the board's right edge, the photodiode looks up."
- note added: "tutorial 1.05, 6.04 (+-5 V)"
- note added: "tutorial 4.07 (+-5 V)"
- moved on the sheet: C101, C102, C103, C104, C105, C106, C1101, C1102, C1103, C1104, C1105, C201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

Commit message: AMOD-A: the fab package passes every check; stand-in 3D models for three library footprints; gen_docs (handbook, manufacturing, design notes); the chat log
Co-Authored-By: Claude Fable 5.1 <noreply@anthropic.com>
Claude-Session: https://claude.ai/code/session_01RKeoKvFFzjk3cEBLCXXHnB
Parts:
- U701: LCSC C1519916 -> C6542; MPN CD74HC4046AM -> CD74HC4046AM96
Changed lines of the file:
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@@
 	)
 	(rectangle
-		(start 25.4 30.48)
-		(end 210.82 152.4)
+		(start 596.9 157.48)
+		(end 782.32 279.4)
 		(stroke
 			(width 0.25)
@@
 	)
 	(rectangle
-		(start 406.4 30.48)
-		(end 591.82 152.4)
+		(start 25.4 30.48)
+		(end 210.82 152.4)
 		(stroke
 			(width 0.25)
@@
 	)
 	(rectangle
-		(start 215.9 30.48)
-		(end 401.32 152.4)
+		(start 596.9 30.48)
+		(end 782.32 152.4)
 		(stroke
 			(width 0.25)
@@
 	)
 	(rectangle
-		(start 596.9 157.48)
-		(end 782.32 279.4)
+		(start 25.4 411.48)
+		(end 401.32 533.4)
 		(stroke
 			(width 0.25)
@@
 	)
 	(rectangle
-		(start 596.9 30.48)
-		(end 782.32 152.4)
+		(start 406.4 284.48)
+		(end 782.32 406.4)
 		(stroke
 			(width 0.25)
@@
 	)
 	(rectangle
-		(start 25.4 284.48)
-		(end 401.32 406.4)
+		(start 406.4 411.48)
+		(end 782.32 533.4)
 		(stroke
 			(width 0.25)
@@
 	)
 	(rectangle
-		(start 25.4 411.48)
-		(end 401.32 533.4)
+		(start 25.4 284.48)
+		(end 401.32 406.4)
 		(stroke
 			(width 0.25)
@@
 	)
 	(rectangle
-		(start 215.9 157.48)
-		(end 401.32 279.4)
+		(start 25.4 157.48)
+		(end 210.82 279.4)
 		(stroke
 			(width 0.25)
@@
 	)
 	(rectangle
-		(start 25.4 157.48)
-		(end 210.82 279.4)
+		(start 406.4 157.48)
+		(end 591.82 279.4)
 		(stroke
 			(width 0.25)
@@
 	)
 	(rectangle
-		(start 406.4 411.48)
-		(end 782.32 533.4)
+		(start 215.9 157.48)
+		(end 401.32 279.4)
 		(stroke
 			(width 0.25)
@@
 	)
 	(rectangle
-		(start 406.4 284.48)
-		(end 782.32 406.4)
+		(start 406.4 30.48)
+		(end 591.82 152.4)
 		(stroke
 			(width 0.25)
@@
 	)
 	(rectangle
-		(start 406.4 157.48)
-		(end 591.82 279.4)
+		(start 215.9 30.48)
+		(end 401.32 152.4)
 		(stroke
 			(width 0.25)
@@
 			)
 		)
-		(property "LCSC" "C1519916"
+		(property "LCSC" "C6542"
 			(at 335.28 203.2 0)
 			(hide yes)
@@
 			)
 		)
-		(property "MPN" "CD74HC4046AM"
+		(property "MPN" "CD74HC4046AM96"
 			(at 335.28 203.2 0)
 			(hide yes)
