File: hardware/amod_a.kicad_sch (KiCad schematic)
At the start: 190 parts, among them J1001 SMA, J1002 SMA, J101 USB-C, J102 rails, J1101 SMA, J1102 TX, J1103 RX, J1104 Pmod, J1201 SMA, J1202 SMA, J1203 SPK, J1204 MIC, J201 SMA, J202 SMA, J301 SMA, J302 SMA, J401 SMA, J402 SMA, J501 SMA, J502 R, J601 SMA, J701 SMA, J702 SMA, J801 SMA, J901 SMA, J902 SMA, J903 SMA, Q1001 AO3401A, Q1002 2N7002, Q1101 AO3401A, Q1201 AO3401A, Q201 AO3401A, Q301 AO3401A, Q401 AO3401A, Q501 AO3401A, Q601 AO3401A, Q701 AO3401A, Q801 AO3401A, Q802 AO3400A, Q901 AO3401A, SW1001 ON, SW1101 ON, SW1201 ON, SW201 ON, SW301 ON, SW401 ON, SW501 ON, SW502 DIP2, SW601 ON, SW701 ON, SW801 ON, SW901 ON, U1001 OPA810, U1002 OPA810, U101 LM2664, U102 3.3V, U1101 DRV8837, U1102 OPA810, U1201 PAM8302A, U1202 OPA810, U201 OPA810, U301 OPA810, U401 OPA847, U501 LT6230, U601 TLV3501, U701 HC4046, U801 TMP235, U901 MC1496

Commit message: RF-MOD: the two MAX2871 synthesizer tiles (R10 host of the Pmod plug, R11) at DRC 0; a Fine net class at 0.127 mm with 0.45/0.25 vias for the QFN fan-out, V33 islands on L3, FRONT_WIRES; the fab package passes
Co-Authored-By: Claude Fable 5.1 <noreply@anthropic.com>
Claude-Session: https://claude.ai/code/session_01RKeoKvFFzjk3cEBLCXXHnB
Other:
- moved on the sheet: J1001, J1101, J1202, J202, J302, J402, J501, J702, J801, J903

Commit message: Pmod plugs: fix the mirrored pinout on AMOD-A and RF-MOD (JLCPCB's numbering of the PZ254R runs opposite to KiCad's): plug two columns left, nets renamed to the standard IO numbers, a fab check of every plug pad; mounting holes replaced by four marked rubber feet on both boards
Co-Authored-By: Claude Opus 5.5 <noreply@anthropic.com>
Claude-Session: https://claude.ai/code/session_01RKeoKvFFzjk3cEBLCXXHnB
Parts:
- removed MH1, MH2, MH3, MH4: MountingHole, MountingHole:MountingHole_3.2mm_M3, symbol Mechanical:MountingHole
Connections:
- net GND: now also J1104.3 (Pin_3), J1104.4 (Pin_4); no longer J1104.10 (Pin_10), J1104.9 (Pin_9)
- net PMOD2: now also J1104.10 (Pin_10), R1201.2; no longer J1104.3 (Pin_3), TP601.1, U601.5
- net PMOD3: now also J1104.8 (Pin_8), U1101.6 (IN1); no longer J1104.5 (Pin_5), Q802.1 (G), R803.1
- net PMOD4: now also J1104.6 (Pin_6), U1101.5 (IN2); no longer J1104.7 (Pin_7), Q1002.1 (G), R1004.1
- net PMOD5: now also J1104.11 (Pin_11), Q1002.1 (G), R1004.1; no longer J1104.2 (Pin_2), U1101.5 (IN2)
- net PMOD6: now also J1104.9 (Pin_9), Q802.1 (G), R803.1; no longer J1104.4 (Pin_4), U1101.6 (IN1)
- net PMOD7: now also J1104.7 (Pin_7), TP601.1, U601.5; no longer J1104.6 (Pin_6), R1201.2
- net PMOD_VCC: now also J1104.1 (Pin_1), J1104.2 (Pin_2); no longer J1104.11 (Pin_11), J1104.12 (Pin_12)
- net PMOD1 renamed PMOD8
- net PMOD8: now also J1104.5 (Pin_5); no longer J1104.1 (Pin_1)
Other:
- note added: "no mounting holes: four stick-on rubber feet, marked on the back"
- note removed: "M3 mounting holes, one per corner"

Commit message: Docs: PLAN as built for RF-MOD and the adapter, the Pmod renumbering in AMOD-A's prose and table, the DOA lists and the review brief
Co-Authored-By: Claude Opus 5.5 <noreply@anthropic.com>
Claude-Session: https://claude.ai/code/session_01RKeoKvFFzjk3cEBLCXXHnB
Other:
- note added: "Drive IN1/IN2 (Pmod IO4, IO3) in antiphase at 40 kHz for 8-20 cycles: the bridge puts 10 V peak to peak across the TX"
- note added: "EXPECT: 0.83 W into the board when Pmod IO6 is high (the FET's drain), 10 mV/K + 500 mV on OUT"
- note added: "EXPECT: 45 mA of LED current per volt on DRIVE IN (0-1 V, blanked while Pmod IO5 is high); PD OUT climbs 10 V per mA of photocurrent"
- note added: "EXPECT: a 40 kHz burst from Pmod IO4/IO3 leaves the TX transducer; its echo arrives x100 on RX OUT (hold a reflector over the board)"
- note added: "EXPECT: a one-bit stream on Pmod IO7 whose density follows IN; the FPGA closes the loop through Pmod IO8 (the handbook's gateware)"
- note added: "EXPECT: a speaker on SPK follows AUDIO IN (2.5 W into 4 ohm) or the one-bit stream on Pmod IO2 (10 k / 10 n); MIC OUT is the electret x100"
- note added: "PAM8302A: 1 u couples AUDIO IN to IN+ (IN- grounded through 1 u), the one-bit DAC on Pmod IO2 arrives through 10 k"
- note added: "Two 15 ohm in series: 30 ohm, 170 mA, 0.83 W from the switched 5 V when Pmod IO6 is high (10 k keeps it off otherwise)."
- note added: "full 40 mA; above 1.1 V the op amp runs out of headroom). A 2N7002 from Pmod IO5 shorts the input: TTL modulation to"
- note removed: "Drive IN1/IN2 (Pmod 5, 6) in antiphase at 40 kHz for 8-20 cycles: the bridge puts 10 V peak to peak across the TX"
- note removed: "EXPECT: 0.83 W into the board when Pmod 3 is high (the FET's drain), 10 mV/K + 500 mV on OUT"
- note removed: "EXPECT: 45 mA of LED current per volt on DRIVE IN (0-1 V, blanked while Pmod 4 is high); PD OUT climbs 10 V per mA of photocurrent"
- note removed: "EXPECT: a 40 kHz burst from Pmod 5/6 leaves the TX transducer; its echo arrives x100 on RX OUT (hold a reflector over the board)"
- note removed: "EXPECT: a one-bit stream on Pmod 2 whose density follows IN; the FPGA closes the loop through Pmod 1 (the handbook's gateware)"
- note removed: "EXPECT: a speaker on SPK follows AUDIO IN (2.5 W into 4 ohm) or the one-bit stream on Pmod 7 (10 k / 10 n); MIC OUT is the electret x100"
- note removed: "PAM8302A: 1 u couples AUDIO IN to IN+ (IN- grounded through 1 u), the one-bit DAC on Pmod 7 arrives through 10 k"
- note removed: "Two 15 ohm in series: 30 ohm, 170 mA, 0.83 W from the switched 5 V when Pmod 3 is high (10 k keeps it off otherwise)."
- note removed: "full 40 mA; above 1.1 V the op amp runs out of headroom). A 2N7002 from Pmod 4 shorts the input: TTL modulation to"
Changed lines of the file:
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@@
+	)
+	(rectangle
+		(start 25.4 30.48)
+		(end 210.82 152.4)
+		(stroke
+			(width 0.25)
+			(type default)
+		)
+		(fill
+			(type none)
+		)
 	)
 	(rectangle
@@
 	)
 	(rectangle
-		(start 25.4 30.48)
-		(end 210.82 152.4)
+		(start 25.4 411.48)
+		(end 401.32 533.4)
+		(stroke
+			(width 0.25)
+			(type default)
+		)
+		(fill
+			(type none)
+		)
+	)
+	(rectangle
+		(start 25.4 157.48)
+		(end 210.82 279.4)
+		(stroke
+			(width 0.25)
+			(type default)
+		)
+		(fill
+			(type none)
+		)
+	)
+	(rectangle
+		(start 215.9 30.48)
+		(end 401.32 152.4)
+		(stroke
+			(width 0.25)
+			(type default)
+		)
+		(fill
+			(type none)
+		)
+	)
+	(rectangle
+		(start 406.4 157.48)
+		(end 591.82 279.4)
 		(stroke
 			(width 0.25)
@@
 	)
 	(rectangle
-		(start 406.4 157.48)
-		(end 591.82 279.4)
+		(start 596.9 30.48)
+		(end 782.32 152.4)
+		(stroke
+			(width 0.25)
+			(type default)
+		)
+		(fill
+			(type none)
+		)
+	)
+	(rectangle
+		(start 406.4 411.48)
+		(end 782.32 533.4)
+		(stroke
+			(width 0.25)
+			(type default)
+		)
+		(fill
+			(type none)
+		)
+	)
+	(rectangle
+		(start 406.4 284.48)
+		(end 782.32 406.4)
 		(stroke
 			(width 0.25)
@@
 		)
 	)
-	(rectangle
-		(start 406.4 284.48)
-		(end 782.32 406.4)
-		(stroke
-			(width 0.25)
-			(type default)
-		)
-		(fill
-			(type none)
-		)
-	)
-	(rectangle
-		(start 406.4 411.48)
-		(end 782.32 533.4)
-		(stroke
-			(width 0.25)
-			(type default)
-		)
-		(fill
-			(type none)
-		)
-	)
-	(rectangle
-		(start 215.9 30.48)
-		(end 401.32 152.4)
-		(stroke
-			(width 0.25)
-			(type default)
-		)
-		(fill
-			(type none)
-		)
-	)
-	(rectangle
-		(start 25.4 157.48)
-		(end 210.82 279.4)
-		(stroke
-			(width 0.25)
-			(type default)
-		)
-		(fill
-			(type none)
-		)
-	)
-	(rectangle
-		(start 596.9 30.48)
-		(end 782.32 152.4)
-		(stroke
-			(width 0.25)
-			(type default)
-		)
-		(fill
-			(type none)
-		)
-	)
-	(rectangle
-		(start 25.4 411.48)
-		(end 401.32 533.4)
-		(stroke
-			(width 0.25)
-			(type default)
-		)
-		(fill
-			(type none)
-		)
-	)
 	(text "OUT"
 		(exclude_from_sim no)
@@
 		)
 	)
-	(text "Drive IN1/IN2 (Pmod 5, 6) in antiphase at 40 kHz for 8-20 cycles: the bridge puts 10 V peak to peak across the TX"
+	(text "The TMP235 reads 750 mV at 25 C and climbs 10 mV per kelvin.  A feedback-control experiment: hold the TMP235 at a"
+		(exclude_from_sim no)
+		(at 408.94 274.22 0)
+		(effects
+			(font
+				(size 1.2 1.2)
+			)
+			(justify left)
+		)
+	)
+	(text "Drive IN1/IN2 (Pmod IO4, IO3) in antiphase at 40 kHz for 8-20 cycles: the bridge puts 10 V peak to peak across the TX"
 		(exclude_from_sim no)
 		(at 27.94 522.94 0)
@@
 		)
 	)
-	(text "The TMP235 reads 750 mV at 25 C and climbs 10 mV per kelvin.  A feedback-control experiment: hold the TMP235 at a"
-		(exclude_from_sim no)
-		(at 408.94 274.22 0)
-		(effects
-			(font
-				(size 1.2 1.2)
-			)
-			(justify left)
-		)
-	)
 	(text "First-order delta-sigma: the comparator decides, the FPGA registers the bit and feeds it back through 10 k into the"
 		(exclude_from_sim no)
@@
 		)
 	)
-	(text "EXPECT: 45 mA of LED current per volt on DRIVE IN (0-1 V, blanked while Pmod 4 is high); PD OUT climbs 10 V per mA of photocurrent"
+	(text "EXPECT: 45 mA of LED current per volt on DRIVE IN (0-1 V, blanked while Pmod IO5 is high); PD OUT climbs 10 V per mA of photocurrent"
 		(exclude_from_sim no)
 		(at 408.94 393.3 0)
@@
 		)
 	)
-	(text "PAM8302A: 1 u couples AUDIO IN to IN+ (IN- grounded through 1 u), the one-bit DAC on Pmod 7 arrives through 10 k"
+	(text "PAM8302A: 1 u couples AUDIO IN to IN+ (IN- grounded through 1 u), the one-bit DAC on Pmod IO2 arrives through 10 k"
 		(exclude_from_sim no)
 		(at 408.94 525.58 0)
@@
 		)
 	)
-	(text "EXPECT: 0.83 W into the board when Pmod 3 is high (the FET's drain), 10 mV/K + 500 mV on OUT"
+	(text "EXPECT: 0.83 W into the board when Pmod IO6 is high (the FET's drain), 10 mV/K + 500 mV on OUT"
 		(exclude_from_sim no)
 		(at 408.94 268.94 0)
@@
 		)
 	)
-	(text "EXPECT: a 40 kHz burst from Pmod 5/6 leaves the TX transducer; its echo arrives x100 on RX OUT (hold a reflector over the board)"
+	(text "EXPECT: a 40 kHz burst from Pmod IO4/IO3 leaves the TX transducer; its echo arrives x100 on RX OUT (hold a reflector over the board)"
 		(exclude_from_sim no)
 		(at 27.94 520.3 0)
@@
 		)
 	)
-	(text "full 40 mA; above 1.1 V the op amp runs out of headroom).  A 2N7002 from Pmod 4 shorts the input: TTL modulation to"
+	(text "full 40 mA; above 1.1 V the op amp runs out of headroom).  A 2N7002 from Pmod IO5 shorts the input: TTL modulation to"
 		(exclude_from_sim no)
 		(at 408.94 398.58 0)
@@
 		)
 	)
-	(text "EXPECT: a speaker on SPK follows AUDIO IN (2.5 W into 4 ohm) or the one-bit stream on Pmod 7 (10 k / 10 n); MIC OUT is the electret x100"
+	(text "EXPECT: a speaker on SPK follows AUDIO IN (2.5 W into 4 ohm) or the one-bit stream on Pmod IO2 (10 k / 10 n); MIC OUT is the electret x100"
 		(exclude_from_sim no)
 		(at 408.94 522.94 0)
@@
 		)
 	)
-	(text "EXPECT: a one-bit stream on Pmod 2 whose density follows IN; the FPGA closes the loop through Pmod 1 (the handbook's gateware)"
+	(text "EXPECT: a one-bit stream on Pmod IO7 whose density follows IN; the FPGA closes the loop through Pmod IO8 (the handbook's gateware)"
 		(exclude_from_sim no)
 		(at 27.94 268.94 0)
@@
 		)
 	)
-	(text "Two 15 ohm in series: 30 ohm, 170 mA, 0.83 W from the switched 5 V when Pmod 3 is high (10 k keeps it off otherwise)."
+	(text "Two 15 ohm in series: 30 ohm, 170 mA, 0.83 W from the switched 5 V when Pmod IO6 is high (10 k keeps it off otherwise)."
 		(exclude_from_sim no)
 		(at 408.94 271.58 0)
