File: hardware/amod_a.kicad_sch (KiCad schematic)
At the start: 189 parts, among them J1001 SMA, J1002 SMA, J1003 SMA, J1004 SMA, J101 USB-C, J102 rails, J1101 SMA, J1102 TX, J1103 RX, J1104 Pmod, J1201 SMA, J1202 SMA, J1203 SPK, J1204 MIC, J201 SMA, J202 SMA, J301 SMA, J302 SMA, J401 SMA, J402 SMA, J501 SMA, J502 HB100, J601 SMA, J701 SMA, J702 SMA, J801 SMA, J901 SMA, J902 SMA, J903 SMA, Q1001 AO3401A, Q1101 AO3401A, Q1201 AO3401A, Q201 AO3401A, Q301 AO3401A, Q401 AO3401A, Q501 AO3401A, Q601 AO3401A, Q701 AO3401A, Q801 AO3401A, Q802 AO3400A, Q901 AO3401A, SW1001 ON, SW1002 DIP4, SW1101 ON, SW1201 ON, SW201 ON, SW301 ON, SW401 ON, SW501 ON, SW601 ON, SW701 ON, SW801 ON, SW901 ON, U1001 OPA810, U1002 OPA810, U101 LM2664, U102 3.3V, U1101 DRV8837, U1102 OPA810, U1201 PAM8302A, U1202 OPA810, U201 OPA810, U301 OPA810, U401 OPA847, U501 OPA810, U601 TLV3501, U701 74HC4046A, U801 TMP235, U901 MC1496

Commit message: Silkscreen says what each tile is and whose jack is whose: jack names on their own tile's frame, titles in words on the top frame, ranges and levels placed inside; tutorial section numbers off the boards; README tables of every tile (what, chip link, specs, limits, experiments, use, what to buy) and handbook entries as tables with a picture of each tile, both from boards/tile_docs.py
Co-Authored-By: Claude Opus 5.5 <noreply@anthropic.com>
Claude-Session: https://claude.ai/code/session_01RKeoKvFFzjk3cEBLCXXHnB
Other:
- note added: "tutorial A counter on the LEDs"
- note added: "tutorial A faster DAC: PLLs (+5 V)"
- note added: "tutorial ADC samples to Python, MSK and GMSK (+-5 V)"
- note added: "tutorial An AM radio, PSK and QPSK (+-5 V)"
- note added: "tutorial RC and LC circuits, More ideas for one board (+-5 V)"
- note added: "tutorial The speed of sound at 40 kHz (+-5 V)"
- note added: "tutorial The speed of sound at 40 kHz, Warming a crystal (+-5 V)"
- note added: "tutorial The speed of sound at 40 kHz, What time is it over there? (+-5 V)"
- note added: "tutorial Trading speed for bits (+3.3 V)"
- note added: "tutorial Warming a crystal, Control at the speed of the cable (+5 V)"
- note added: "tutorial With a little more hardware (+-5 V)"
- note removed: "tutorial 1.01"
- note removed: "tutorial 1.05, 6.04 (+-5 V)"
- note removed: "tutorial 1.10, 6.02 (+-5 V)"
- note removed: "tutorial 4.01 (+5 V)"
- note removed: "tutorial 4.02, 4.10 (+-5 V)"
- note removed: "tutorial 4.06 (+-5 V)"
- note removed: "tutorial 4.06, 5.02 (+-5 V)"
- note removed: "tutorial 4.06, 5.03 (+-5 V)"
- note removed: "tutorial 5.02, 7.06 (+5 V)"
- note removed: "tutorial 5.08 (+-5 V)"
- note removed: "tutorial 7.05 (+3.3 V)"

Commit message: A12: the speaker channel's jack is SPEAKER IN (whose input: the speaker's), beside MIC OUT; A11's docs say its 5 V powers the TX bridge and the RX op amp
Co-Authored-By: Claude Opus 5.5 <noreply@anthropic.com>
Claude-Session: https://claude.ai/code/session_01RKeoKvFFzjk3cEBLCXXHnB
Other:
- note added: "EXPECT: a speaker on SPK follows SPEAKER IN (2.5 W into 4 ohm) or the one-bit stream on Pmod IO2 (10 k / 10 n); MIC OUT is the electret x100"
- note added: "PAM8302A: 1 u couples SPEAKER IN to IN+ (IN- grounded through 1 u), the one-bit DAC on Pmod IO2 arrives through 10 k"
- note added: "in pins 1 and 5 (10.16 mm; their leads are 10 mm apart). The slide switch's 5 V powers the bridge and the op amp's + rail."
- note removed: "EXPECT: a speaker on SPK follows AUDIO IN (2.5 W into 4 ohm) or the one-bit stream on Pmod IO2 (10 k / 10 n); MIC OUT is the electret x100"
- note removed: "PAM8302A: 1 u couples AUDIO IN to IN+ (IN- grounded through 1 u), the one-bit DAC on Pmod IO2 arrives through 10 k"
- note removed: "in pins 1 and 5 (10.16 mm; their leads are 10 mm apart)."
Changed lines of the file:
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@@
+		)
+	)
+	(text "PAM8302A: 1 u couples SPEAKER IN to IN+ (IN- grounded through 1 u), the one-bit DAC on Pmod IO2 arrives through 10 k"
+		(exclude_from_sim no)
+		(at 408.94 525.58 0)
+		(effects
+			(font
+				(size 1.2 1.2)
+			)
+			(justify left)
 		)
 	)
@@
 		)
 	)
-	(text "PAM8302A: 1 u couples AUDIO IN to IN+ (IN- grounded through 1 u), the one-bit DAC on Pmod IO2 arrives through 10 k"
-		(exclude_from_sim no)
-		(at 408.94 525.58 0)
-		(effects
-			(font
-				(size 1.2 1.2)
-			)
-			(justify left)
-		)
-	)
 	(text "which is fine for a product detector).  IF OUT is single-ended from pin 6 through 100 n: a 1.5 k source, so read it"
 		(exclude_from_sim no)
@@
 		)
 	)
-	(text "in pins 1 and 5 (10.16 mm; their leads are 10 mm apart)."
+	(text "in pins 1 and 5 (10.16 mm; their leads are 10 mm apart).  The slide switch's 5 V powers the bridge and the op amp's + rail."
 		(exclude_from_sim no)
 		(at 27.94 530.86 0)
@@
 		)
 	)
-	(text "EXPECT: a speaker on SPK follows AUDIO IN (2.5 W into 4 ohm) or the one-bit stream on Pmod IO2 (10 k / 10 n); MIC OUT is the electret x100"
+	(text "EXPECT: a speaker on SPK follows SPEAKER IN (2.5 W into 4 ohm) or the one-bit stream on Pmod IO2 (10 k / 10 n); MIC OUT is the electret x100"
 		(exclude_from_sim no)
 		(at 408.94 522.94 0)

Commit message: Silk case convention on all six boards (Jason, Prompt 17: "To distinguish whole-tile labels from SMA or port labels, use different cases")
Ports (the jacks' names, terminal and loop names, a port named inside a note) stay UPPER CASE.  A tile's label (its
title on the frame, its name in the corner) is Mixed case: the first letter capitalised and the rest as written ("RC
low-pass", "Synthesizer", "I/Q demodulator"; tiles.label_case).  Ranges, values and notes are lower case except units,
acronyms and part numbers ("loss 1.7 dB", "OUT floats").  RF-MOD-2's X1 and X2 take word titles with their chips in
the info; RF-MOD's and RF-MOD-2's LNA tiles are titled "Preamp" ("Low-noise amp" does not fit a cell's frame); a few
two-line labels moved 0.15-0.3 mm for the descenders mixed case brings.  AMOD-P2's tile records (tile_docs), its DOA
list, KIT.md's AMOD-P2 section; X5's calibration points at P14.  All six boards: ERC 0, DRC 0, all fab checks.

Co-Authored-By: Claude Opus 5.5 <noreply@anthropic.com>
Claude-Session: https://claude.ai/code/session_01RKeoKvFFzjk3cEBLCXXHnB
Changed lines of the file:
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@@
 	(wire
 		(pts
+			(xy 370.84 441.96) (xy 365.76 441.96)
+		)
+		(stroke
+			(width 0)
+			(type default)
+		)
+	)
+	(wire
+		(pts
+			(xy 751.84 314.96) (xy 746.76 314.96)
+		)
+		(stroke
+			(width 0)
+			(type default)
+		)
+	)
+	(wire
+		(pts
 			(xy 261.62 353.06) (xy 264.16 353.06)
 		)
@@
 	(wire
 		(pts
-			(xy 365.76 314.96) (xy 370.84 314.96)
-		)
-		(stroke
-			(width 0)
-			(type default)
-		)
-	)
-	(wire
-		(pts
 			(xy 419.1 447.04) (xy 419.1 449.58)
 		)
@@
 	(wire
 		(pts
+			(xy 180.34 60.96) (xy 175.26 60.96)
+		)
+		(stroke
+			(width 0)
+			(type default)
+		)
+	)
+	(wire
+		(pts
 			(xy 172.72 541.02) (xy 172.72 543.56)
 		)
@@
 	(wire
 		(pts
+			(xy 370.84 60.96) (xy 365.76 60.96)
+		)
+		(stroke
+			(width 0)
+			(type default)
+		)
+	)
+	(wire
+		(pts
 			(xy 279.4 76.2) (xy 276.86 76.2)
 		)
@@
 	(wire
 		(pts
+			(xy 726.44 314.96) (xy 721.36 314.96)
+		)
+		(stroke
+			(width 0)
+			(type default)
+		)
+	)
+	(wire
+		(pts
 			(xy 566.42 66.04) (xy 566.42 68.58)
 		)
@@
 	(wire
 		(pts
-			(xy 556.26 60.96) (xy 561.34 60.96)
-		)
-		(stroke
-			(width 0)
-			(type default)
-		)
-	)
-	(wire
-		(pts
 			(xy 115.57 322.58) (xy 113.03 322.58)
 		)
@@
 	(wire
 		(pts
+			(xy 751.84 60.96) (xy 746.76 60.96)
+		)
+		(stroke
+			(width 0)
+			(type default)
+		)
+	)
+	(wire
+		(pts
 			(xy 213.36 457.2) (xy 210.82 457.2)
 		)
@@
 	(wire
 		(pts
-			(xy 556.26 187.96) (xy 561.34 187.96)
-		)
-		(stroke
-			(width 0)
-			(type default)
-		)
-	)
-	(wire
-		(pts
 			(xy 538.48 330.2) (xy 538.48 332.74)
 		)
@@
 	(wire
 		(pts
-			(xy 365.76 60.96) (xy 370.84 60.96)
-		)
-		(stroke
-			(width 0)
-			(type default)
-		)
-	)
-	(wire
-		(pts
 			(xy 76.2 353.06) (xy 73.66 353.06)
 		)
@@
 	(wire
 		(pts
-			(xy 365.76 187.96) (xy 370.84 187.96)
-		)
-		(stroke
-			(width 0)
-			(type default)
-		)
-	)
-	(wire
-		(pts
 			(xy 528.32 492.76) (xy 525.78 492.76)
 		)
@@
 	(wire
 		(pts
+			(xy 561.34 187.96) (xy 556.26 187.96)
+		)
+		(stroke
+			(width 0)
+			(type default)
+		)
+	)
+	(wire
+		(pts
 			(xy 287.02 208.28) (xy 287.02 210.82)
 		)
@@
 	(wire
 		(pts
-			(xy 695.96 314.96) (xy 701.04 314.96)
-		)
-		(stroke
-			(width 0)
-			(type default)
-		)
-	)
-	(wire
-		(pts
 			(xy 218.44 353.06) (xy 215.9 353.06)
 		)
@@
 	(wire
 		(pts
-			(xy 746.76 60.96) (xy 751.84 60.96)
-		)
-		(stroke
-			(width 0)
-			(type default)
-		)
-	)
-	(wire
-		(pts
 			(xy 71.12 459.74) (xy 73.66 459.74)
 		)
@@
 	(wire
 		(pts
-			(xy 746.76 441.96) (xy 751.84 441.96)
-		)
-		(stroke
-			(width 0)
-			(type default)
-		)
-	)
-	(wire
-		(pts
 			(xy 495.3 332.74) (xy 492.76 332.74)
 		)
@@
 	(wire
 		(pts
-			(xy 721.36 314.96) (xy 726.44 314.96)
-		)
-		(stroke
-			(width 0)
-			(type default)
-		)
-	)
-	(wire
-		(pts
 			(xy 571.5 353.06) (xy 574.04 353.06)
 		)
@@
 	(wire
 		(pts
-			(xy 175.26 60.96) (xy 180.34 60.96)
-		)
-		(stroke
-			(width 0)
-			(type default)
-		)
-	)
-	(wire
-		(pts
 			(xy 287.02 81.28) (xy 287.02 83.82)
 		)
@@
 	(wire
 		(pts
+			(xy 561.34 60.96) (xy 556.26 60.96)
+		)
+		(stroke
+			(width 0)
+			(type default)
+		)
+	)
+	(wire
+		(pts
 			(xy 702.31 186.69) (xy 704.85 186.69)
 		)
@@
 	(wire
 		(pts
+			(xy 370.84 187.96) (xy 365.76 187.96)
+		)
+		(stroke
+			(width 0)
+			(type default)
+		)
+	)
+	(wire
+		(pts
 			(xy 133.35 322.58) (xy 135.89 322.58)
 		)
@@
 	(wire
 		(pts
+			(xy 370.84 314.96) (xy 365.76 314.96)
+		)
+		(stroke
+			(width 0)
+			(type default)
+		)
+	)
+	(wire
+		(pts
 			(xy 261.62 205.74) (xy 264.16 205.74)
 		)
@@
 	(wire
 		(pts
-			(xy 365.76 441.96) (xy 370.84 441.96)
-		)
-		(stroke
-			(width 0)
-			(type default)
-		)
-	)
-	(wire
-		(pts
 			(xy 563.88 353.06) (xy 561.34 353.06)
 		)
@@
 	(wire
 		(pts
-			(xy 182.88 365.76) (xy 180.34 365.76)
+			(xy 751.84 441.96) (xy 746.76 441.96)
 		)
 		(stroke
@@
 	(wire
 		(pts
-			(xy 154.94 353.06) (xy 157.48 353.06)
+			(xy 182.88 365.76) (xy 180.34 365.76)
 		)
 		(stroke
@@
 	(wire
 		(pts
-			(xy 421.64 365.76) (xy 419.1 365.76)
+			(xy 154.94 353.06) (xy 157.48 353.06)
 		)
 		(stroke
@@
 	(wire
 		(pts
-			(xy 642.62 73.66) (xy 645.16 73.66)
+			(xy 421.64 365.76) (xy 419.1 365.76)
 		)
 		(stroke
@@
 	(wire
 		(pts
-			(xy 116.84 462.28) (xy 114.3 462.28)
+			(xy 642.62 73.66) (xy 645.16 73.66)
 		)
 		(stroke
@@
 	(wire
 		(pts
-			(xy 88.9 457.2) (xy 86.36 457.2)
+			(xy 116.84 462.28) (xy 114.3 462.28)
 		)
 		(stroke
@@
 	(wire
 		(pts
-			(xy 746.76 314.96) (xy 751.84 314.96)
+			(xy 88.9 457.2) (xy 86.36 457.2)
 		)
 		(stroke
@@
 		)
 		(stroke
+			(width 0)
+			(type default)
+		)
+	)
+	(wire
+		(pts
+			(xy 701.04 314.96) (xy 695.96 314.96)
+		)
+		(stroke

Commit message: One letter per board, tiles in lower case: AMOD-P2 is AMOD-N (n1-n11), RF-MOD-2 is IQ-MOD (q1-q11), PhMOD's tiles h1-h10
Jason, Prompt 19: "If we can have a nice, well justified single-letter designator for each board, it would make
everything much more clear", and "d11, q11, and c11 don't look like obvious electronics or PCB things".

- p passive, n networks (AMOD-P2's P14, P16-P25), a active, r radio, h PhMOD (Y1-Y10), q quadrature (RF-MOD-2's X1-X11);
  c, m and b are taken for the conversion, motor and brushless boards to come.  PLAN.md section 13 has the table and
  the reasons (no letter moves to another board, no retired name is reused, no s: s11 is the reflection coefficient).
- Every tile name in lower case on the silk, in the code (Tile ids, BACK/BACK_PLOTS/DOCS keys, the nets built on them),
  the handbooks, README, DOA lists, KIT, PLAN and the review brief; pin names (USB-C A1...), the 4046's R1/C1, nets
  named N1/P1, part numbers ending -R7 and the paper size A1 left alone.  tiles.dump refuses a tile not named
  <letter><n>, a number twice, and a BACK key for a tile that does not exist.
- Board and file renames: boards/amod_n.py, boards/iq_mod.py, docs/DOA_amod_n.md, docs/DOA_iq_mod.md, the handbooks,
  the generated hardware, outputs and pictures.  Silk nudged where a lower-case p or q hung onto the line below.
- All six boards rebuilt: ERC 0, DRC 0, every check.

Co-Authored-By: Claude Opus 5.5 <noreply@anthropic.com>
Claude-Session: https://claude.ai/code/session_01RKeoKvFFzjk3cEBLCXXHnB
Connections:
- net A10_FB renamed a10_FB
- net A10_G renamed a10_G
- net A10_IN renamed a10_IN
- net A10_OUT renamed a10_OUT
- net A10_OUT_A renamed a10_OUT_A
- net A10_R1 renamed a10_R1
- net A10_R2 renamed a10_R2
- net A10_R3 renamed a10_R3
- net A10_R4 renamed a10_R4
- net A10_VS renamed a10_VS
- net A10_X renamed a10_X
- net A10_XF renamed a10_XF
- net A10_XO renamed a10_XO
- net A11_FB renamed a11_FB
- net A11_G renamed a11_G
- net A11_IN renamed a11_IN
- net A11_OUT renamed a11_OUT
- net A11_OUT1 renamed a11_OUT1
- net A11_OUT2 renamed a11_OUT2
- net A11_OUT_A renamed a11_OUT_A
- net A11_RXA renamed a11_RXA
- net A11_VS renamed a11_VS
- net A12_AIN renamed a12_AIN
- net A12_BYP renamed a12_BYP
- net A12_FB renamed a12_FB
- net A12_G renamed a12_G
- net A12_IN renamed a12_IN
- net A12_INM renamed a12_INM
- net A12_MICP renamed a12_MICP
- net A12_NODE renamed a12_NODE
- net A12_OUT renamed a12_OUT
- net A12_OUT_A renamed a12_OUT_A
- net A12_VOM renamed a12_VOM
- net A12_VOP renamed a12_VOP
- net A12_VS renamed a12_VS
- net A1_CAPN renamed a1_CAPN
- net A1_CAPP renamed a1_CAPP
- net A1_CC1 renamed a1_CC1
- net A1_CC2 renamed a1_CC2
- net A1_LEDG renamed a1_LEDG
- net A1_LEDR renamed a1_LEDR
- net A1_VBUS renamed a1_VBUS
- net A2_FB renamed a2_FB
- net A2_G renamed a2_G
- net A2_IN renamed a2_IN
- net A2_OUT renamed a2_OUT
- net A2_OUT_A renamed a2_OUT_A
- net A2_VS renamed a2_VS
- net A3_FB renamed a3_FB
- net A3_G renamed a3_G
- net A3_IN renamed a3_IN
- net A3_OUT renamed a3_OUT
- net A3_OUT_A renamed a3_OUT_A
- net A3_VS renamed a3_VS
- net A4_FB renamed a4_FB
- net A4_G renamed a4_G
- net A4_IN renamed a4_IN
- net A4_OUT renamed a4_OUT
- net A4_OUT_A renamed a4_OUT_A
- net A4_VS renamed a4_VS
- net A5_FB renamed a5_FB
- net A5_G renamed a5_G
- net A5_IF renamed a5_IF
- net A5_IN renamed a5_IN
- net A5_OUT renamed a5_OUT
- net A5_OUT_A renamed a5_OUT_A
- net A5_VS renamed a5_VS
- net A6_G renamed a6_G
- net A6_IN renamed a6_IN
- net A6_NODE renamed a6_NODE
- net A6_VREF renamed a6_VREF
- net A6_VS renamed a6_VS
- net A7_C1A renamed a7_C1A
- net A7_C1B renamed a7_C1B
- net A7_G renamed a7_G
- net A7_IN renamed a7_IN
- net A7_INA renamed a7_INA
- net A7_NODE renamed a7_NODE
- net A7_OUT renamed a7_OUT
- net A7_PC2 renamed a7_PC2
- net A7_R1 renamed a7_R1
- net A7_SIG renamed a7_SIG
- net A7_VCO_A renamed a7_VCO_A
- net A7_VS renamed a7_VS
- net A8_DRN renamed a8_DRN
- net A8_G renamed a8_G
- net A8_HTR renamed a8_HTR
- net A8_OUT renamed a8_OUT
- net A8_VS renamed a8_VS
- net A9_BIAS renamed a9_BIAS
- net A9_CARA renamed a9_CARA
- net A9_CARB renamed a9_CARB
- net A9_CB renamed a9_CB
- net A9_G renamed a9_G
- net A9_GAIN2 renamed a9_GAIN2
- net A9_GAIN3 renamed a9_GAIN3
- net A9_IF renamed a9_IF
- net A9_LO renamed a9_LO
- net A9_OUTA renamed a9_OUTA
- net A9_OUTB renamed a9_OUTB
- net A9_RF renamed a9_RF
- net A9_SIGA renamed a9_SIGA
- net A9_SIGB renamed a9_SIGB
- net A9_VS renamed a9_VS
Other:
- note added: "a1 power, USB-C 5 V in: +5, -5, +3.3 out"
- note added: "a10 impedance, V and I"
- note added: "a11 ultrasound"
- note added: "a12 audio"
- note added: "a2 x10, 14 MHz"
- note added: "a3 x100, 1.4MHz"
- note added: "a4 LNA, 30 MHz"
- note added: "a5 Doppler, HB100"
- note added: "a6 1-bit ADC"
- note added: "a7 PLL 4046"
- note added: "a8 heat"
- note added: "a9 mixer, MC1496"
- note added: "in series with the output. For 40 dB out to 30 MHz use a4 (the OPA847 LNA); this tile is the FET-input, high-impedance"
- note added: "its colour (p12) gives Planck's constant; a crystal (p8) shows its series and parallel resonances."
- note removed: "A1 power, USB-C 5 V in: +5, -5, +3.3 out"
- note removed: "A10 impedance, V and I"
- note removed: "A11 ultrasound"
- note removed: "A12 audio"
- note removed: "A2 x10, 14 MHz"
- note removed: "A3 x100, 1.4MHz"
- note removed: "A4 LNA, 30 MHz"
- note removed: "A5 Doppler, HB100"
- note removed: "A6 1-bit ADC"
- note removed: "A7 PLL 4046"
- note removed: "A8 heat"
- note removed: "A9 mixer, MC1496"
- note removed: "in series with the output. For 40 dB out to 30 MHz use A4 (the OPA847 LNA); this tile is the FET-input, high-impedance"
- note removed: "its colour (P12) gives Planck's constant; a crystal (P8) shows its series and parallel resonances."

Commit message: Pre-order checks from CLAUDE_PCB.md's new lessons (Prompt 21): the KF301 terminals turned for their wire openings (CPL +180, body 3.7 / 4.0, a wire-face check), four oversold parts swapped (27R, 6.8k, 220n, OPA847IDBVT at its own +180), fourteen vias moved out of SMD pads (check_layout.py gates it and RF detours), 200-250 mW terminations, assembly drawings from Fab and silk fitted to Letter (fit_pdf.py from CostasLink), the stock gate on JLCPCB's free count, electrolytics in the rotation check, the RF gates surveyed (rf_extract.py, rf_survey.py) and written into the DOA lists; all nine boards rebuilt: ERC 0, DRC 0, every check
Co-Authored-By: Claude Opus 5.5 <noreply@anthropic.com>
Claude-Session: https://claude.ai/code/session_01RKeoKvFFzjk3cEBLCXXHnB
Parts:
- R1001, R1003, R1009, R1103, R1204, R201, R203, R301, R303, R401, R403, R503: LCSC C23185 -> C6230117; MPN 0603WAF499JT5E -> SR0603FR-7T49R9L
- U401: LCSC C160422 -> C2059024; MPN OPA847IDBVR -> OPA847IDBVT
Changed lines of the file:
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@@
 			)
 		)
-		(property "LCSC" "C23185"
+		(property "LCSC" "C6230117"
 			(at 532.13 353.06 90)
 			(hide yes)
@@
 			)
 		)
-		(property "MPN" "0603WAF499JT5E"
+		(property "MPN" "SR0603FR-7T49R9L"
 			(at 532.13 353.06 90)
 			(hide yes)
@@
 			)
 		)
-		(property "LCSC" "C23185"
+		(property "LCSC" "C6230117"
 			(at 425.45 353.06 90)
 			(hide yes)
@@
 			)
 		)
-		(property "MPN" "0603WAF499JT5E"
+		(property "MPN" "SR0603FR-7T49R9L"
 			(at 425.45 353.06 90)
 			(hide yes)
@@
 			)
 		)
-		(property "LCSC" "C23185"
+		(property "LCSC" "C6230117"
 			(at 425.45 99.06 90)
 			(hide yes)
@@
 			)
 		)
-		(property "MPN" "0603WAF499JT5E"
+		(property "MPN" "SR0603FR-7T49R9L"
 			(at 425.45 99.06 90)
 			(hide yes)
@@
 			)
 		)
-		(property "LCSC" "C160422"
+		(property "LCSC" "C2059024"
 			(at 500.38 76.2 0)
 			(hide yes)
@@
 			)
 		)
-		(property "MPN" "OPA847IDBVR"
+		(property "MPN" "OPA847IDBVT"
 			(at 500.38 76.2 0)
 			(hide yes)
@@
 			)
 		)
-		(property "LCSC" "C23185"
+		(property "LCSC" "C6230117"
 			(at 461.01 492.76 90)
 			(hide yes)
@@
 			)
 		)
-		(property "MPN" "0603WAF499JT5E"
+		(property "MPN" "SR0603FR-7T49R9L"
 			(at 461.01 492.76 90)
 			(hide yes)
@@
 			)
 		)
-		(property "LCSC" "C23185"
+		(property "LCSC" "C6230117"
 			(at 151.13 99.06 90)
 			(hide yes)
@@
 			)
 		)
-		(property "MPN" "0603WAF499JT5E"
+		(property "MPN" "SR0603FR-7T49R9L"
 			(at 151.13 99.06 90)
 			(hide yes)
@@
 			)
 		)
-		(property "LCSC" "C23185"
+		(property "LCSC" "C6230117"
 			(at 234.95 99.06 90)
 			(hide yes)
@@
 			)
 		)
-		(property "MPN" "0603WAF499JT5E"
+		(property "MPN" "SR0603FR-7T49R9L"
 			(at 234.95 99.06 90)
 			(hide yes)
@@
 			)
 		)
-		(property "LCSC" "C23185"
+		(property "LCSC" "C6230117"
 			(at 425.45 365.76 90)
 			(hide yes)
@@
 			)
 		)
-		(property "MPN" "0603WAF499JT5E"
+		(property "MPN" "SR0603FR-7T49R9L"
 			(at 425.45 365.76 90)
 			(hide yes)
@@
 			)
 		)
-		(property "LCSC" "C23185"
+		(property "LCSC" "C6230117"
 			(at 257.81 482.6 90)
 			(hide yes)
@@
 			)
 		)
-		(property "MPN" "0603WAF499JT5E"
+		(property "MPN" "SR0603FR-7T49R9L"
 			(at 257.81 482.6 90)
 			(hide yes)
@@
 			)
 		)
-		(property "LCSC" "C23185"
+		(property "LCSC" "C6230117"
 			(at 44.45 99.06 90)
 			(hide yes)
@@
 			)
 		)
-		(property "MPN" "0603WAF499JT5E"
+		(property "MPN" "SR0603FR-7T49R9L"
 			(at 44.45 99.06 90)
 			(hide yes)
@@
 			)
 		)
-		(property "LCSC" "C23185"
+		(property "LCSC" "C6230117"
 			(at 758.19 99.06 90)
 			(hide yes)
@@
 			)
 		)
-		(property "MPN" "0603WAF499JT5E"
+		(property "MPN" "SR0603FR-7T49R9L"
 			(at 758.19 99.06 90)
 			(hide yes)
@@
 			)
 		)
-		(property "LCSC" "C23185"
+		(property "LCSC" "C6230117"
 			(at 341.63 99.06 90)
 			(hide yes)
@@
 			)
 		)
-		(property "MPN" "0603WAF499JT5E"
+		(property "MPN" "SR0603FR-7T49R9L"
 			(at 341.63 99.06 90)
 			(hide yes)
@@
 			)
 		)
-		(property "LCSC" "C23185"
+		(property "LCSC" "C6230117"
 			(at 532.13 99.06 90)
 			(hide yes)
@@
 			)
 		)
-		(property "MPN" "0603WAF499JT5E"
+		(property "MPN" "SR0603FR-7T49R9L"
 			(at 532.13 99.06 90)
 			(hide yes)

Commit message: AMOD-A's PAM8302 on its real MSOP-8 (Prompt 22: JLCPCB's preview showed the MSOP-8 on our SOIC-8 pads; a12 re-laid, pin 2 NC); check_overlay.py lays JLCPCB's drawing on our pads in every build (a wrong package with the right pin order failed nothing before); check_pinouts pairs EasyEDA's names by the printed pin number; the order steps say Specify Stackup No (JLC04161H-7628's construction), the via size and Plugged; the chat log
Co-Authored-By: Claude Opus 5.5 <noreply@anthropic.com>
Claude-Session: https://claude.ai/code/session_01RKeoKvFFzjk3cEBLCXXHnB
Parts:
- removed C1209: 100n, Capacitor_SMD:C_0603_1608Metric, symbol Device:C
- C1204, C1207: value 1u -> 100n; LCSC C15849 -> C14663; MPN CL10A105KB8NNNC -> CC0603KRX7R9BB104
- C1205: value 100n -> 10u; footprint Capacitor_SMD:C_0603_1608Metric -> Capacitor_SMD:C_0805_2012Metric; LCSC C14663 -> C15850; MPN CC0603KRX7R9BB104 -> CL21A106KAYNNNE
- C1206: value 10u -> 1u; footprint Capacitor_SMD:C_0805_2012Metric -> Capacitor_SMD:C_0603_1608Metric; LCSC C15850 -> C15849; MPN CL21A106KAYNNNE -> CL10A105KB8NNNC
- U1201: footprint Package_SO:SOIC-8_3.9x4.9mm_P1.27mm -> Package_SO:MSOP-8_3x3mm_P0.65mm; symbol amod:PAM8302_SOIC8 -> amod:PAM8302_MSOP8
Connections:
- net -5V: now also C1207.2; no longer C1208.2
- net GND: now also C1207.1; no longer C1206.2
- net a12_IN: now also C1206.2; no longer C1207.2
- net a12_MICP: now also C1206.1; no longer C1207.1
- net a12_VS: now also C1204.1, C1208.2; no longer C1206.1
- net a12_BYP: no longer names the net of U1201.2 (NC)
- net a12_BYP: no longer C1204.1
- no-connect marks 23 -> 24
Other:
- note added: "into 10 n (1.6 kHz) at the same node, so both play. SD high: on with the tile (pin 2 is NC). The electret (pin 1 is the"
- note removed: "into 10 n (1.6 kHz) at the same node, so both play. BYP 1 u, SD high: on with the tile. The electret (pin 1 is the"
- moved on the sheet: C1206, C1208, R1202, R1203, R1204, R1205
