File: hardware/rf_mod.kicad_sch (KiCad schematic)
At the start: 63 parts, among them J1201 SMA, J1202 SMA, J201 SMA, J202 SMA, J401 SMA, J402 SMA, J501 SMA, J502 SMA, J901 USB-C, J902 SMA, Q1201 AO3401A, Q501 AO3401A, SW1201 ON, SW501 ON, U1201 GALI-84+, U501 GALI-84+, U901 MT3608, U902 3.3V, U903 74LVC1G17, X901 25 MHz

Commit message: RF-MOD: the two MAX2871 synthesizer tiles (R10 host of the Pmod plug, R11) at DRC 0; a Fine net class at 0.127 mm with 0.45/0.25 vias for the QFN fan-out, V33 islands on L3, FRONT_WIRES; the fab package passes
Co-Authored-By: Claude Fable 5.1 <noreply@anthropic.com>
Claude-Session: https://claude.ai/code/session_01RKeoKvFFzjk3cEBLCXXHnB
Parts:
- added C1001, C1002, C1101, C1102: 1u, Capacitor_SMD:C_0805_2012Metric, symbol Device:C
- added C1003, C1103: 470p, Capacitor_SMD:C_0603_1608Metric, symbol Device:C
- added C1004, C1104: 6.8n, Capacitor_SMD:C_0603_1608Metric, symbol Device:C
- added C1005, C1006, C1007, C1008, C1011, C1105, C1106, C1107, C1108, C1111: 100n, Capacitor_SMD:C_0402_1005Metric, symbol Device:C
- added C1009, C1010, C1109, C1110: 100p, Capacitor_SMD:C_0402_1005Metric, symbol Device:C
- added C1012, C1014, C1015, C1112, C1114, C1115: 1u, Capacitor_SMD:C_0402_1005Metric, symbol Device:C
- added C1013, C1113: 100p, Capacitor_SMD:C_0603_1608Metric, symbol Device:C
- added J1001, J1002, J1101, J1102: SMA, amod:SMA_BWSMA-KE-Z001_Vertical, symbol Connector:Conn_Coaxial
- added J1003: Pmod, amod:PinHeader_2x06_P2.54mm_Horizontal_PZ254R-12-12P, symbol Connector_Generic:Conn_02x06_Odd_Even
- added L1001, L1002, L1101, L1102: 27n, Inductor_SMD:L_0402_1005Metric, symbol Device:L
- added LED1001, LED1101: LOCK, amod:LED_0805_2012Metric_Kbar, symbol Device:LED
- added Q1001, Q1101: AO3401A, Package_TO_SOT_SMD:SOT-23, symbol Transistor_FET:AO3401A
- added R1001, R1101: 470, Resistor_SMD:R_0402_1005Metric, symbol Device:R_US
- added R1002, R1102: 820, Resistor_SMD:R_0402_1005Metric, symbol Device:R_US
- added R1003, R1103: 100k, Resistor_SMD:R_0402_1005Metric, symbol Device:R_US
- added R1004, R1104: 1k, Resistor_SMD:R_0402_1005Metric, symbol Device:R_US
- added R1005, R1105: 51R, Resistor_SMD:R_0402_1005Metric, symbol Device:R_US
- added R1006, R1106: 5.1k, Resistor_SMD:R_0402_1005Metric, symbol Device:R_US
- added SW1001, SW1101: ON, amod:SW_SPDT_Shouhan_MSK12C02, symbol Switch:SW_SPDT
- added U1001, U1101: 3.3V, Package_TO_SOT_SMD:SOT-23-5, symbol Regulator_Linear:TPS7A20xxxDBV
- added U1002, U1102: MAX2871, Package_DFN_QFN:QFN-32-1EP_5x5mm_P0.5mm_EP3.1x3.1mm, symbol amod:MAX2871
Connections:
- net +5V: now also Q1001.2 (S), Q1101.2 (S), SW1001.3 (C), SW1101.3 (C)
- net GND: now also C1001.2, C1002.2, C1003.2, C1004.2, C1005.2, C1006.2, C1008.2, C1011.2, C1012.2, C1013.2, C1014.2, C1015.2, C1101.2, C1102.2, C1103.2, C1104.2, C1105.2, C1106.2, C1108.2, C1111.2, C1112.2, C1113.2, C1114.2, C1115.2, J1001.2 (Ext), J1002.2 (Ext), J1003.10 (Pin_10), J1003.9 (Pin_9), J1101.2 (Ext), J1102.2 (Ext), LED1001.1 (K), LED1101.1 (K), R1003.1, R1005.2, R1006.2, R1103.1, R1105.2, R1106.2, SW1001.1 (A), SW1101.1 (A), U1001.2 (GND), U1002.11 (GND), U1002.18 (GND), U1002.21 (GND), U1002.27 (GND), U1002.31 (GND), U1002.33 (EP), U1002.8 (GND), U1002.9 (GND), U1101.2 (GND), U1102.11 (GND), U1102.18 (GND), U1102.21 (GND), U1102.27 (GND), U1102.31 (GND), U1102.33 (EP), U1102.8 (GND), U1102.9 (GND)
- new net PMOD3: J1003.5 (Pin_5), R1103.2, U1102.3 (LE)
- new net PMOD4: J1003.7 (Pin_7), U1102.30 (MUX)
- new net PMOD5: J1003.2 (Pin_2), R1003.2, U1002.3 (LE)
- new net PMOD6: J1003.4 (Pin_4), U1002.1 (CLK), U1102.1 (CLK)
- new net PMOD7: J1003.6 (Pin_6), U1002.2 (DATA), U1102.2 (DATA)
- new net PMOD8: J1003.8 (Pin_8), U1002.30 (MUX)
- new net PMOD_VCC: J1003.11 (Pin_11), J1003.12 (Pin_12)
- new net R10_AN: C1010.1, L1002.1, U1002.13 (RFOUTA-)
- new net R10_AP: C1009.2, L1001.2, U1002.12 (RFOUTA+)
- new net R10_BF: C1014.1, U1002.23 (BIAS_FILT)
- new net R10_CP: C1003.1, R1001.2, R1002.2, U1002.7 (CP_OUT)
- new net R10_G: Q1001.1 (G), SW1001.2 (B)
- new net R10_LD: R1004.1, U1002.25 (LD)
- new net R10_LEDA: LED1001.2 (A), R1004.2
- new net R10_N2: C1004.1, R1002.1
- new net R10_NF: C1012.1, U1002.19 (NOISE_FILT)
- new net R10_OUTA: C1009.1, J1001.1 (In)
- new net R10_REF: C1007.2, J1002.1 (In)
- new net R10_REFI: C1007.1, U1002.29 (REF_IN)
- new net R10_REG: C1015.1, U1002.24 (REG)
- new net R10_RS: R1006.1, U1002.22 (RSET)
- new net R10_TN: C1013.1, R1001.1, U1002.20 (TUNE)
- new net R10_TRM: C1010.2, R1005.1
- new net R10_V33: C1002.1, C1005.1, C1006.1, C1008.1, C1011.1, L1001.1, L1002.2, U1001.5 (OUT), U1002.10 (VCC_PLL), U1002.16 (VCC_RF), U1002.17 (VCC_VCO), U1002.26 (RFOUT_EN), U1002.28 (VCC_DIG), U1002.32 (VCC_SD), U1002.4 (CE), U1002.6 (VCC_CP)
- new net R10_VS: C1001.1, Q1001.3 (D), U1001.1 (IN), U1001.3 (EN)
- new net R11_AN: C1110.1, L1102.1, U1102.13 (RFOUTA-)
- new net R11_AP: C1109.2, L1101.2, U1102.12 (RFOUTA+)
- new net R11_BF: C1114.1, U1102.23 (BIAS_FILT)
- new net R11_CP: C1103.1, R1101.2, R1102.2, U1102.7 (CP_OUT)
- new net R11_G: Q1101.1 (G), SW1101.2 (B)
- new net R11_LD: R1104.1, U1102.25 (LD)
- new net R11_LEDA: LED1101.2 (A), R1104.2
- new net R11_N2: C1104.1, R1102.1
- new net R11_NF: C1112.1, U1102.19 (NOISE_FILT)
- new net R11_OUTA: C1109.1, J1101.1 (In)
- new net R11_REF: C1107.2, J1102.1 (In)
- new net R11_REFI: C1107.1, U1102.29 (REF_IN)
- new net R11_REG: C1115.1, U1102.24 (REG)
- new net R11_RS: R1106.1, U1102.22 (RSET)
- new net R11_TN: C1113.1, R1101.1, U1102.20 (TUNE)
- new net R11_TRM: C1110.2, R1105.1
- new net R11_V33: C1102.1, C1105.1, C1106.1, C1108.1, C1111.1, L1101.1, L1102.2, U1101.5 (OUT), U1102.10 (VCC_PLL), U1102.16 (VCC_RF), U1102.17 (VCC_VCO), U1102.26 (RFOUT_EN), U1102.28 (VCC_DIG), U1102.32 (VCC_SD), U1102.4 (CE), U1102.6 (VCC_CP)
- new net R11_VS: C1101.1, Q1101.3 (D), U1101.1 (IN), U1101.3 (EN)
- no-connect marks 10 -> 20
Other:
- note added: "100 pF; RFOUTA- is terminated in 51 ohm the same way; RFOUTB is open and must stay disabled. CE and RFOUT_EN are"
- note added: "25 MHz, 3.3 V CMOS"
- note added: "EXPECT: +5 V from the USB-C (up to 1.5 A), +7.8 V at 250 mA for the gain blocks (yellow LED), a 25 MHz square wave on REF OUT"
- note added: "EXPECT: any frequency from 23.5 MHz to 6 GHz on OUT A (-4 to +5 dBm in steps), locked to the 25 MHz on REF IN; the red LED says locked"
- note added: "LE; MUXOUT back). The loop filter is third order, 80-120 kHz with 61 degrees of margin for both 915 MHz (VCO / 4)"
- note added: "MAX2871 as CostasLink built it: fractional-N PLL with four VCOs, programmed over SPI from the Pmod (SCLK, SDATA,"
- note added: "OUT A"
- note added: "R10 synthesizer, MAX2871"
- note added: "R11 synthesizer, MAX2871"
- note added: "REF IN"
- note added: "REF OUT (51 ohm: 1.6 Vpp into 50 ohm, 3.3 Vpp into a synthesizer's unterminated REF IN; a tee feeds both synthesizers)."
- note added: "and 2.4 GHz (VCO / 2) at ICP 2.56 mA (RSET 5.1 k, CP = 7). RFOUTA+ feeds the jack through 27 nH to 3.3 V and"
- note added: "cells (0,3), (1,3)"
- note added: "cells (2,3), (3,3)"
- note added: "tied high, LE has 100 k down. REF IN is unterminated: one REF OUT drives both synthesizers through a tee."
- note removed: "EXPECT: +5 V from the USB-C (up to 1.5 A), +7.8 V at 250 mA for the gain blocks (yellow LED), 25 MHz square wave on REF OUT and the REF25 bus"
- note removed: "REF OUT (51 ohm: 1.6 Vpp into 50 ohm) and the REF25 line on the back to the synthesizers' jumpers (3.3 Vpp open)."
- moved on the sheet: J1202, J202, J402, J502, J902

Commit message: RF-MOD filled: ADL5350 mixers R7/R8, a resistive splitter R1, ten tiles on sixteen cells at ERC/DRC 0 and the fab package passing; stand-in 3D bodies scaled 1/2.54 (VRML unit) on every board
Co-Authored-By: Claude Opus 5.5 <noreply@anthropic.com>
Claude-Session: https://claude.ai/code/session_01RKeoKvFFzjk3cEBLCXXHnB
Parts:
- added C701, C801: 1u, Capacitor_SMD:C_0805_2012Metric, symbol Device:C
- added C702, C802: 4.7u, Capacitor_SMD:C_0805_2012Metric, symbol Device:C
- added C703, C704, C803, C804: 15p, Capacitor_SMD:C_0402_1005Metric, symbol Device:C
- added C705, C805: 100n, Capacitor_SMD:C_0402_1005Metric, symbol Device:C
- added C706, C707, C806, C807: 100p, Capacitor_SMD:C_0402_1005Metric, symbol Device:C
- added J101, J102, J103, J701, J702, J703, J801, J802, J803: SMA, amod:SMA_BWSMA-KE-Z001_Vertical, symbol Connector:Conn_Coaxial
- added L701, L702, L801, L802: 47n, Inductor_SMD:L_0402_1005Metric, symbol Device:L
- added L703, L803: 10n, Inductor_SMD:L_0402_1005Metric, symbol Device:L
- added Q701, Q801: AO3401A, Package_TO_SOT_SMD:SOT-23, symbol Transistor_FET:AO3401A
- added R101, R102, R103: 18R, Resistor_SMD:R_0402_1005Metric, symbol Device:R_US
- added R701, R801: 0R, Resistor_SMD:R_0402_1005Metric, symbol Device:R_US
- added SW701, SW801: ON, amod:SW_SPDT_Shouhan_MSK12C02, symbol Switch:SW_SPDT
- added U701, U801: 3.3V, Package_TO_SOT_SMD:SOT-23-5, symbol Regulator_Linear:TPS7A20xxxDBV
- added U702, U802: ADL5350, amod:LFCSP-8_2x3mm_P0.5mm_ADL5350, symbol amod:ADL5350
Connections:
- net +5V: now also Q701.2 (S), Q801.2 (S), SW701.3 (C), SW801.3 (C)
- net GND: now also C701.2, C702.2, C704.2, C707.2, C801.2, C802.2, C804.2, C807.2, J101.2 (Ext), J102.2 (Ext), J103.2 (Ext), J701.2 (Ext), J702.2 (Ext), J703.2 (Ext), J801.2 (Ext), J802.2 (Ext), J803.2 (Ext), L701.2, L801.2, SW701.1 (A), SW801.1 (A), U701.2 (GND), U702.2 (GND), U702.4 (NC), U702.5 (GND), U702.7 (NC), U702.9 (EP), U801.2 (GND), U802.2 (GND), U802.4 (NC), U802.5 (GND), U802.7 (NC), U802.9 (EP)
- new net R1_N: R101.2, R102.1, R103.1
- new net R1_P1: J101.1 (In), R101.1
- new net R1_P2: J102.1 (In), R102.2
- new net R1_P3: J103.1 (In), R103.2
- new net R7_G: Q701.1 (G), SW701.2 (B)
- new net R7_IF: C705.2, J703.1 (In)
- new net R7_IFN: C704.1, C705.1, L702.2
- new net R7_LOC: C706.1, R701.2
- new net R7_LOJ: C706.2, J702.1 (In)
- new net R7_LON: R701.1, U702.3 (LOIN)
- new net R7_RFIF: C703.2, L702.1, U702.1 (RF/IF), U702.8 (RF/IF)
- new net R7_RFN: C703.1, J701.1 (In), L701.1
- new net R7_V33: C702.1, L703.2, U701.5 (OUT)
- new net R7_VPOS: C707.1, L703.1, U702.6 (VPOS)
- new net R7_VS: C701.1, Q701.3 (D), U701.1 (IN), U701.3 (EN)
- new net R8_G: Q801.1 (G), SW801.2 (B)
- new net R8_IF: C805.2, J803.1 (In)
- new net R8_IFN: C804.1, C805.1, L802.2
- new net R8_LOC: C806.1, R801.2
- new net R8_LOJ: C806.2, J802.1 (In)
- new net R8_LON: R801.1, U802.3 (LOIN)
- new net R8_RFIF: C803.2, L802.1, U802.1 (RF/IF), U802.8 (RF/IF)
- new net R8_RFN: C803.1, J801.1 (In), L801.1
- new net R8_V33: C802.1, L803.2, U801.5 (OUT)
- new net R8_VPOS: C807.1, L803.1, U802.6 (VPOS)
- new net R8_VS: C801.1, Q801.3 (D), U801.1 (IN), U801.3 (EN)
- no-connect marks 20 -> 22
Other:
- note added: "(series 15 pF + shunt 47 nH toward RF, series 47 nH + shunt 15 pF toward IF, corner 200 MHz) in place of the"
- note added: "+20 dBm"
- note added: "0 to +6 dBm"
- note added: "ADL5350: a GaAs FET switch mixer with its own LO buffer; the RF and IF pins are one node, split by a crossover"
- note added: "Both images appear: filter the RF side with R2 or R4."
- note added: "EXPECT: 6.2 dB from any port to either other port, every port within 2 ohm of 50, DC to 6 GHz (the resistors' parasitics set the top)"
- note added: "EXPECT: RF x LO to IF (or IF x LO to RF) with 7-9 dB of loss from 400 MHz to 2.5 GHz and an IF of 0.1-30 MHz; +4 dBm of LO is enough"
- note added: "IF"
- note added: "LO"
- note added: "P1"
- note added: "P2"
- note added: "P3"
- note added: "Passive, so the same tile up-converts a DAC tone (IF in, RF out) or down-converts an antenna's signal (RF in, IF out)."
- note added: "R1 splitter, 3 x 18 ohm, 6 dB"
- note added: "R7 TX mixer, ADL5350"
- note added: "R8 RX mixer, ADL5350"
- note added: "RF"
- note added: "Three 18 ohm resistors to one node: the textbook resistive divider, 6 dB per path and no isolation between the two"
- note added: "both synthesizers' REF IN, one synthesizer's OUT A to both mixers, or two tones into one gain block."
- note added: "cells (0,0), (1,0)"
- note added: "cells (0,2), (1,2)"
- note added: "cells (2,2), (3,2)"
- note added: "datasheet's 3-8 nH for one band); the LO bias choke is 10 nH (the datasheet: 24 nH at 780 MHz, 2 nH at 2 GHz)."
- note added: "datasheet's band-tuned tanks: a few dB more loss, every band at once. The LO's series element is 0 ohm (fit the"
- note added: "outputs beyond those 6 dB (a Wilkinson would give 3 dB and 20 dB of isolation, at one band). Feed R9's REF OUT to"

Commit message: Pmod plugs: fix the mirrored pinout on AMOD-A and RF-MOD (JLCPCB's numbering of the PZ254R runs opposite to KiCad's): plug two columns left, nets renamed to the standard IO numbers, a fab check of every plug pad; mounting holes replaced by four marked rubber feet on both boards
Co-Authored-By: Claude Opus 5.5 <noreply@anthropic.com>
Claude-Session: https://claude.ai/code/session_01RKeoKvFFzjk3cEBLCXXHnB
Parts:
- removed MH1, MH2, MH3, MH4: MountingHole, MountingHole:MountingHole_3.2mm_M3, symbol Mechanical:MountingHole
Connections:
- net GND: now also J1003.3 (Pin_3), J1003.4 (Pin_4); no longer J1003.10 (Pin_10), J1003.9 (Pin_9)
- net PMOD3: now also J1003.8 (Pin_8), U1002.1 (CLK), U1102.1 (CLK); no longer J1003.5 (Pin_5), R1103.2, U1102.3 (LE)
- net PMOD4: now also J1003.6 (Pin_6), R1003.2, U1002.3 (LE); no longer J1003.7 (Pin_7), U1102.30 (MUX)
- net PMOD5: now also J1003.11 (Pin_11), U1102.30 (MUX); no longer J1003.2 (Pin_2), R1003.2, U1002.3 (LE)
- net PMOD6: now also J1003.9 (Pin_9), R1103.2, U1102.3 (LE); no longer J1003.4 (Pin_4), U1002.1 (CLK), U1102.1 (CLK)
- net PMOD_VCC: now also J1003.1 (Pin_1), J1003.2 (Pin_2); no longer J1003.11 (Pin_11), J1003.12 (Pin_12)
- net PMOD7 renamed PMOD2
- net PMOD2: now also J1003.10 (Pin_10); no longer J1003.6 (Pin_6)
- net PMOD8 renamed PMOD1
- net PMOD1: now also J1003.12 (Pin_12); no longer J1003.8 (Pin_8)
Other:
- note added: "REF OUT (51 ohm: 1.6 Vpp into 50 ohm, 3.3 Vpp into a synthesizer's unterminated REF IN; R1 feeds both synthesizers)."
- note added: "no mounting holes: four stick-on rubber feet, marked on the back"
- note added: "tied high, LE has 100 k down. REF IN is unterminated: one REF OUT drives both synthesizers through R1."
- note removed: "M3 mounting holes, one per corner"
- note removed: "REF OUT (51 ohm: 1.6 Vpp into 50 ohm, 3.3 Vpp into a synthesizer's unterminated REF IN; a tee feeds both synthesizers)."
- note removed: "tied high, LE has 100 k down. REF IN is unterminated: one REF OUT drives both synthesizers through a tee."
