File: hardware/rf_mod.kicad_sch (KiCad schematic)
At the start: 162 parts, among them J1001 SMA, J1002 SMA, J1003 Pmod, J101 SMA, J102 SMA, J103 SMA, J1101 SMA, J1102 SMA, J1201 SMA, J1202 SMA, J201 SMA, J202 SMA, J401 SMA, J402 SMA, J501 SMA, J502 SMA, J701 SMA, J702 SMA, J703 SMA, J801 SMA, J802 SMA, J803 SMA, J901 USB-C, J902 SMA, Q1001 AO3401A, Q1101 AO3401A, Q1201 AO3401A, Q501 AO3401A, Q701 AO3401A, Q801 AO3401A, SW1001 ON, SW1101 ON, SW1201 ON, SW501 ON, SW701 ON, SW801 ON, U1001 3.3V, U1002 MAX2871, U1101 3.3V, U1102 MAX2871, U1201 GALI-84+, U501 GALI-84+, U701 3.3V, U702 ADL5350, U801 3.3V, U802 ADL5350, U901 MT3608, U902 3.3V, U903 74LVC1G17, X901 25 MHz

Commit message: RF-MOD rev A: the QPL9547 LNA in R5 and the TRF3722 quadrature transmitter as R13 (Prompt 13)
- R5: QPL9547TR7 (C5367093, 5,070 in stock; rev A's search had missed the reel) on
  Qorvo's evaluation circuit, in place of a second GALI-84+: 0.3 dB of noise figure
  for every receiver.  R12 stays the GALI-84+ gain block; the 7.8 V strip now ends at it.
- R13 (cells of the old R11): TRF3722 (C1850395, 2,218) with I and Q from the ECP5
  board's two DACs through resistor networks to its 0.25 V common mode, TI's
  fractional loop filter, a TLV75733 in the WSON (0.56 W) on a 3.3 V island, the
  reference from R10's REF IN on the back, SPI shared with R10 (LE IO6, readback IO5).
  Jason's "Yes. Add that tile." from Appendix D's questions.
- The second MAX2871 (R11) is gone: R13 has its own PLL and VCO.
- Symbols: stacked hidden pins for the TRF3722's grounds; the generic schematic block
  closes up its rows when they would reach the notes.  A DFN-8 stand-in 3D body.
- PLAN_LEVEL2.md: the plan for AMOD-2 and RF-MOD-2 and the first level checked again.

RF-MOD: ERC 0, DRC 0, every fab check passed, $57.18 of parts a board.

Co-Authored-By: Claude Opus 5.5 <noreply@anthropic.com>
Claude-Session: https://claude.ai/code/session_01RKeoKvFFzjk3cEBLCXXHnB
Parts:
- removed C1101, C1102: 1u, Capacitor_SMD:C_0805_2012Metric, symbol Device:C
- removed C1103: 470p, Capacitor_SMD:C_0603_1608Metric, symbol Device:C
- removed C1104: 6.8n, Capacitor_SMD:C_0603_1608Metric, symbol Device:C
- removed C1105, C1106, C1107, C1108, C1111: 100n, Capacitor_SMD:C_0402_1005Metric, symbol Device:C
- removed C1109, C1110: 100p, Capacitor_SMD:C_0402_1005Metric, symbol Device:C
- removed C1112, C1114, C1115: 1u, Capacitor_SMD:C_0402_1005Metric, symbol Device:C
- removed C1113: 100p, Capacitor_SMD:C_0603_1608Metric, symbol Device:C
- removed J1101, J1102: SMA, amod:SMA_BWSMA-KE-Z001_Vertical, symbol Connector:Conn_Coaxial
- removed L1101, L1102: 27n, Inductor_SMD:L_0402_1005Metric, symbol Device:L
- removed LED1101: LOCK, amod:LED_0805_2012Metric_Kbar, symbol Device:LED
- removed Q1101: AO3401A, Package_TO_SOT_SMD:SOT-23, symbol Transistor_FET:AO3401A
- removed R1101: 470, Resistor_SMD:R_0402_1005Metric, symbol Device:R_US
- removed R1102: 820, Resistor_SMD:R_0402_1005Metric, symbol Device:R_US
- removed R1103: 100k, Resistor_SMD:R_0402_1005Metric, symbol Device:R_US
- removed R1104: 1k, Resistor_SMD:R_0402_1005Metric, symbol Device:R_US
- removed R1105: 51R, Resistor_SMD:R_0402_1005Metric, symbol Device:R_US
- removed R1106: 5.1k, Resistor_SMD:R_0402_1005Metric, symbol Device:R_US
- removed SW1101: ON, amod:SW_SPDT_Shouhan_MSK12C02, symbol Switch:SW_SPDT
- removed U1101: 3.3V, Package_TO_SOT_SMD:SOT-23-5, symbol Regulator_Linear:TPS7A20xxxDBV
- removed U1102: MAX2871, Package_DFN_QFN:QFN-32-1EP_5x5mm_P0.5mm_EP3.1x3.1mm, symbol amod:MAX2871
- added C1301, C1304, C1306, C1307, C1311: 100n, Capacitor_SMD:C_0402_1005Metric, symbol Device:C
- added C1302, C1303, C505: 100p, Capacitor_SMD:C_0402_1005Metric, symbol Device:C
- added C1305: 4.7p, Capacitor_SMD:C_0402_1005Metric, symbol Device:C
- added C1308: 1n, Capacitor_SMD:C_0402_1005Metric, symbol Device:C
- added C1309: 10n, Capacitor_SMD:C_0402_1005Metric, symbol Device:C
- added C1310: 330p, Capacitor_SMD:C_0402_1005Metric, symbol Device:C
- added C1312, C1313: 1u, Capacitor_SMD:C_0603_1608Metric, symbol Device:C
- added C506: 10u, Capacitor_SMD:C_0805_2012Metric, symbol Device:C
- added J1301, J1302, J1303: SMA, amod:SMA_BWSMA-KE-Z001_Vertical, symbol Connector:Conn_Coaxial
- added LED1301: LOCK, amod:LED_0805_2012Metric_Kbar, symbol Device:LED
- added Q1301: AO3401A, Package_TO_SOT_SMD:SOT-23, symbol Transistor_FET:AO3401A
- added R1301, R1302: 1.1k, Resistor_SMD:R_0402_1005Metric, symbol Device:R_US
- added R1303, R1309: 75, Resistor_SMD:R_0402_1005Metric, symbol Device:R_US
- added R1304, R1306, R1310, R1312: 910, Resistor_SMD:R_0402_1005Metric, symbol Device:R_US
- added R1305, R1311: 270, Resistor_SMD:R_0402_1005Metric, symbol Device:R_US
- added R1307, R1313: 100, Resistor_SMD:R_0402_1005Metric, symbol Device:R_US
- added R1308, R1314: 56, Resistor_SMD:R_0402_1005Metric, symbol Device:R_US
- added R1315: 1k, Resistor_SMD:R_0402_1005Metric, symbol Device:R_US
- added SW1301: ON, amod:SW_SPDT_Shouhan_MSK12C02, symbol Switch:SW_SPDT
- added U1301: TRF3722, Package_DFN_QFN:Texas_RGZ0048A_VQFN-48-1EP_7x7mm_P0.5mm_EP5.15x5.15mm, symbol amod:TRF3722
- added U1302: 3.3V, Package_SON:WSON-6-1EP_2x2mm_P0.65mm_EP1x1.6mm, symbol Regulator_Linear:TLV75733PDRV
- C504: value 10u -> 1u; footprint Capacitor_SMD:C_0805_2012Metric -> Capacitor_SMD:C_0402_1005Metric; LCSC C15850 -> C14445; MPN CL21A106KAYNNNE -> CL05A105KP5NNNC
- L501: value 27n -> 18n; LCSC C882469 -> C91622; MPN LQW15AN27NG80D -> LQW15AN18NG00D
- R501: value 22R -> 3.3k; footprint Resistor_SMD:R_2512_6332Metric -> Resistor_SMD:R_0402_1005Metric; LCSC C27258 -> C25890; MPN 25121WJ0220T4E -> 0402WGF3301TCE
- U501: value GALI-84+ -> QPL9547; footprint Package_TO_SOT_SMD:SOT-89-3 -> Package_DFN_QFN:DFN-8-1EP_2x2mm_P0.5mm_EP0.9x1.6mm; symbol amod:GALI84 -> amod:QPL9547; LCSC C3193261 -> C5367093; MPN GALI-84+ -> QPL9547TR7
Connections:
- net R5_VD is gone; now on net R5_VS: C503.1, L501.1, R501.2
- net +5V: now also Q501.2 (S), SW501.3 (C), Q1301.2 (S), SW1301.3 (C)
- net +8V: no longer Q501.2 (S), SW501.3 (C)
- net GND: now also C504.2, U501.3 (NC), U501.4 (NC), U501.5 (NC), U501.6 (SD), U501.8 (NC), U501.9 (GND), C1301.2, C1302.2, C1303.2, C1304.2, C1306.1, C1307.2, C1308.2, C1309.2, C1310.2, C1312.2, C1313.1, C505.1, C506.1, J1301.2 (Ext), J1302.2 (Ext), J1303.2 (Ext), LED1301.1 (K), R1303.2, R1307.2, R1308.2, R1309.2, R1313.2, R1314.2, SW1301.1 (A), U1301.1 (PD), U1301.11 (GND), U1301.15 (GND), U1301.17 (GND), U1301.19 (GND), U1301.20 (GND), U1301.22 (GND), U1301.26 (GND), U1301.30 (GND), U1301.37 (GND), U1301.40 (GND), U1301.43 (GND), U1301.45 (GND), U1301.49 (GND), U1301.5 (GND), U1301.7 (GND), U1302.3 (GND), U1302.7 (GND); no longer C504.1, U501.2 (GND)
- net PMOD2: now also U1301.47 (DATA)
- net PMOD3: now also U1301.48 (CLK)
- net PMOD5: now also U1301.2 (RDBK)
- net PMOD6: now also U1301.46 (LE)
- net R5_IN_A: now also U501.2 (RF_IN); no longer U501.1 (IN)
- net R5_OUT_A: now also U501.7 (RF_OUT); no longer U501.3 (OUT)
- net R5_VS: now also C504.1, C506.2; no longer C504.2, R501.1
- net R10_REF renamed REF25
- net REF25: now also C1311.1
- new net R13_BBI: J1301.1 (In), R1305.2, R1308.1
- new net R13_BBQ: J1302.1 (In), R1311.2, R1314.1
- new net R13_BIN: R1303.1, R1304.1, U1301.29 (BBI_N)
- new net R13_BIP: R1305.1, R1306.1, R1307.1, U1301.27 (BBI_P)
- new net R13_BQN: R1309.1, R1310.1, U1301.8 (BBQ_N)
- new net R13_BQP: R1311.1, R1312.1, R1313.1, U1301.10 (BBQ_P)
- new net R13_CP: C1308.1, R1301.1, R1302.1, U1301.41 (CP_OUT)
- new net R13_G: Q1301.1 (G), SW1301.2 (B)
- new net R13_LD: R1315.1, U1301.3 (LD)
- new net R13_LEDA: LED1301.2 (A), R1315.2
- new net R13_N2: C1309.1, R1301.2
- new net R13_REFI: C1311.2, U1301.44 (REFIN)
- new net R13_RFO: C1305.1, U1301.18 (RFOUT)
- new net R13_RFOUT: C1305.2, J1303.1 (In)
- new net R13_V33: C1301.1, C1302.1, C1303.1, C1304.1, C1306.2, C1307.1, C1313.2, R1304.2, R1306.2, R1310.2, R1312.2, U1301.14 (VCC_MOD1), U1301.16 (VCC_MOD2), U1301.21 (VCC_MOD3), U1301.23 (VCC_MOD4), U1301.32 (VCC_TK), U1301.33 (VCC_VCO), U1301.35 (VCC_LO2), U1301.4 (VCC_DIG), U1301.42 (VCC_PLL), U1301.6 (VCC_LO1), U1302.1 (OUT)
- new net R13_VS: C1312.1, Q1301.3 (D), U1302.4 (EN), U1302.6 (IN)
- new net R13_VT: C1310.1, R1302.2, U1301.34 (VTUNE)
- new net R5_VB: C505.2, R501.1, U501.1 (VBIAS)
- no-connect marks 22 -> 30
Other:
- note added: "(0.6 V x 13 from 12 k / 1 k) for the GALI-84+ tile, R12 (100 mA); the +8V rail is a strip under row 1 that their"
- note added: "+-1 V into 50 ohm"
- note added: "-20 dBm"
- note added: "56 ohm at the jack, 270 ohm to a node held at 0.25 V (+-0.25 V for +-1 V). DC on I alone is a CW carrier."
- note added: "EXPECT: 19.5 dB of gain and a 0.3-0.5 dB noise figure from 0.5 to 3 GHz (datasheet: 0.3 dB at 1.9 GHz, OIP3 +39 dBm); 65 mA from 5 V"
- note added: "EXPECT: I + jQ from two DACs on 0.4-4.2 GHz, about -3 dBm, image-free (-42 dBc untrimmed)"
- note added: "I IN"
- note added: "Never cable a transmitter into it without 30 dB of attenuation (22 dBm absolute maximum at the input)."
- note added: "Q IN"
- note added: "Qorvo QPL9547: a GaAs pHEMT LNA, internally matched to 50 ohm, 0.1-6 GHz. It sets the noise figure of every receiver"
- note added: "R13 I/Q transmitter, TRF3722"
- note added: "R5 LNA, QPL9547"
- note added: "RF OUT"
- note added: "Sweep it with R10 or R13 into a power meter, or with a DAC harmonic comb and the ADC."
- note added: "TRF3722 (PLL, VCO, I/Q modulator) on SPI from the Pmod (LE IO6, readback IO5); reference from R10's REF IN. Each DAC:"
- note added: "The 18 nH wire-wound choke (Qorvo's value) feeds 5 V into the output pin; 3.3 k from 5 V to Vbias sets 65 mA."
- note added: "here, so put it first (before the filter) unless a strong neighbour overloads it; +39 dBm OIP3 makes that rare."
- note removed: "(0.6 V x 13 from 12 k / 1 k) for the two GALI-84+ tiles (200 mA); the +8V rail is a strip under row 1 that their"
- note removed: "R11 synthesizer, MAX2871"
- note removed: "R5 gain block, GALI-84+"
- note removed: "Sweep it with the synthesizer R10 or R11 into a power meter, or with a DAC harmonic comb and the ADC."
- moved on the sheet: C1008, C1009, C1010, C1011, C1012, C1013, C1014, C1015, C504, L1001, L1002, LED1001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

Commit message: RF-MOD-2 rev A: the coherent I/Q transceiver board (Prompt 13)
Eleven tiles for the ECP5-2ADC-2DAC board: an ADL5375-05 modulator fed by its
DACs (X1), an ADL5380 demodulator with two OPA810 difference amplifiers into its
ADCs (X2), RF-MOD's MAX2871 synthesizer with its own REF IN (X3) split by a
resistive splitter into both LOs (X5), the QPL9547 LNA (X4), an AD8318 log
detector (X6), a switched avalanche noise source with an ADL5611 and a 20 dB
pad (X7), a GNSS front end (bias-T, SAW, MAX2659, SAW: X8), a loop for NV
centres' ODMR with every plane cleared under it (X9), USB-C and -5 V (X10) and
a SKY13370 absorptive SPDT on two Pmod lines (X11).  ERC, DRC and every fab
check pass; parts $98.61 a board.  ADL5380's 14 in stock is recorded as Jason's
accepted exception in parts.py and check_outputs reports it.

Generators: per-tile copper voids; hidden stacked symbol pins are passive (a
hidden power input made a global net of its name); schematic chips spaced by
their labels' widths and wrapped; the result note's real height sizes the
part rows; synth_tile can carry REF IN at BR1 and extra Pmod pads.

Co-Authored-By: Claude Opus 5.5 <noreply@anthropic.com>
Claude-Session: https://claude.ai/code/session_01RKeoKvFFzjk3cEBLCXXHnB
Other:
- moved on the sheet: D902, J1003, J901, Q1001, Q1201, Q1301, Q501, Q701, Q801, U1001, U1002, U1201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
