File: hardware/amod_p.kicad_sch (KiCad schematic)
At the start: 150 parts, among them J1001 SMA, J1002 SMA, J101 SMA, J102 SMA, J1101 SMA, J1102 SMA, J1103 SMA, J1104 SMA, J1105 SMA, J1201 SMA, J1301 SMA, J1302 coil, J201 SMA, J202 SMA, J301 SMA, J302 SMA, J401 SMA, J402 SMA, J501 SMA, J502 SMA, J601 SMA, J602 SMA, J701 SMA, J702 SMA, J801 SMA, J802 SMA, J901 SMA, J902 SMA, SW1201 DIP4, SW1301 DIP4, SW401 DIP2, Y801 4 MHz, Y901 455 kHz

Commit message: Jacks in a checkerboard on every board (Prompt 12): every pair 14.85 mm or more
IN at a cell's top-left slot, OUT at its bottom-right, a two-cell tile's third jack
at its right cell's top-left.  geometry.py now asserts 14.3 mm between every pair.

- AMOD-P: all thirteen tiles re-laid; P8's crystal and P9's resonator at 45 degrees
  (P8's jacks 0.5 mm further out, slots TLo/BRo); P11's taps on TL/BR slots.
- AMOD-A: A2-A4 share opa_tile_br; A4's OPA847 now SOT-23-6 (C160422); A7 now
  Nexperia's 74HC4046APW-Q100J in TSSOP-16 (C546981, 234 in stock); A8, A9 and A11
  re-laid with OUT at the bottom-right; the back's QR code moved.  $50.90 of parts.
- RF-MOD: the mixers' LO jacks moved from the top middle to TL1.
- Assembler's notes say the 45-degree parts are meant; PLAN, DOA, review brief,
  README and the chat log updated.

All three boards: ERC 0, DRC 0, every fab check passed.

Co-Authored-By: Claude Opus 5.5 <noreply@anthropic.com>
Claude-Session: https://claude.ai/code/session_01RKeoKvFFzjk3cEBLCXXHnB
Parts:
- TP401: value OUT -> IN
Connections:
- net P11_T1: now also R1101.1; no longer R1101.2
- net P11_T2: now also R1102.1; no longer R1102.2
- net P4_IN: now also TP401.1
- net P4_OUT: now also C402.2, C403.2; no longer C402.1, C403.1, TP401.1
- net at SW401.1: now also C403.1; no longer C403.2
- net at SW401.2: now also C402.1; no longer C402.2
- net at J1103.1 (In): now also R1102.2; no longer R1102.1
- net at J1102.1 (In): now also R1101.2; no longer R1101.1
Other:
- note added: "the peak; a resonant plant for 7.06, a lockbox's cavity before the real one. No OUT loop (the switch took its corner)."
- note removed: "the peak; a resonant plant for 7.06, a lockbox's cavity before the real one. No IN loop (the switch took its corner)."
- moved on the sheet: C402, C403, R1101, R1102
Changed lines of the file:
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@@
 	)
 	(rectangle
-		(start 25.4 30.48)
-		(end 210.82 152.4)
+		(start 406.4 30.48)
+		(end 591.82 152.4)
 		(stroke
 			(width 0.25)
@@
 	)
 	(rectangle
-		(start 25.4 157.48)
-		(end 210.82 279.4)
+		(start 215.9 284.48)
+		(end 782.32 406.4)
 		(stroke
 			(width 0.25)
@@
 	)
 	(rectangle
-		(start 25.4 411.48)
-		(end 210.82 533.4)
+		(start 215.9 411.48)
+		(end 591.82 533.4)
 		(stroke
 			(width 0.25)
@@
 	)
 	(rectangle
-		(start 406.4 30.48)
-		(end 591.82 152.4)
+		(start 25.4 284.48)
+		(end 210.82 406.4)
 		(stroke
 			(width 0.25)
@@
 	)
 	(rectangle
-		(start 215.9 284.48)
-		(end 782.32 406.4)
+		(start 406.4 157.48)
+		(end 591.82 279.4)
 		(stroke
 			(width 0.25)
@@
 	)
 	(rectangle
-		(start 596.9 30.48)
-		(end 782.32 152.4)
+		(start 215.9 157.48)
+		(end 401.32 279.4)
 		(stroke
 			(width 0.25)
@@
 	)
 	(rectangle
-		(start 596.9 411.48)
-		(end 782.32 533.4)
+		(start 596.9 30.48)
+		(end 782.32 152.4)
 		(stroke
 			(width 0.25)
@@
 	)
 	(rectangle
-		(start 406.4 157.48)
-		(end 591.82 279.4)
+		(start 25.4 30.48)
+		(end 210.82 152.4)
 		(stroke
 			(width 0.25)
@@
 	)
 	(rectangle
-		(start 215.9 157.48)
-		(end 401.32 279.4)
+		(start 215.9 30.48)
+		(end 401.32 152.4)
 		(stroke
 			(width 0.25)
@@
 	)
 	(rectangle
-		(start 215.9 30.48)
-		(end 401.32 152.4)
+		(start 25.4 411.48)
+		(end 210.82 533.4)
 		(stroke
 			(width 0.25)
@@
 	)
 	(rectangle
-		(start 596.9 157.48)
-		(end 782.32 279.4)
+		(start 25.4 157.48)
+		(end 210.82 279.4)
 		(stroke
 			(width 0.25)
@@
 	)
 	(rectangle
-		(start 25.4 284.48)
-		(end 210.82 406.4)
+		(start 596.9 411.48)
+		(end 782.32 533.4)
 		(stroke
 			(width 0.25)
@@
 	)
 	(rectangle
-		(start 215.9 411.48)
-		(end 591.82 533.4)
+		(start 596.9 157.48)
+		(end 782.32 279.4)
 		(stroke
 			(width 0.25)
@@
 		)
 	)
-	(text "the peak; a resonant plant for 7.06, a lockbox's cavity before the real one.  No IN loop (the switch took its corner)."
+	(text "the peak; a resonant plant for 7.06, a lockbox's cavity before the real one.  No OUT loop (the switch took its corner)."
 		(exclude_from_sim no)
 		(at 599.44 149.86 0)
@@
 	)
 	(junction
+		(at 617.22 60.96)
+		(diameter 0)
+		(color 0 0 0 0)
+	)
+	(junction
 		(at 334.01 335.28)
 		(diameter 0)
@@
 	)
 	(junction
-		(at 641.35 60.96)
-		(diameter 0)
-		(color 0 0 0 0)
-	)
-	(junction
 		(at 264.16 187.96)
 		(diameter 0)
@@
 	(symbol
 		(lib_id "Device:C")
-		(at 632.46 86.36 90)
+		(at 632.46 86.36 270)
+		(mirror x)
 		(unit 1)
 		(body_style 1)
@@
 	(symbol
 		(lib_id "Device:R_US")
-		(at 274.32 368.3 270)
-		(mirror x)
+		(at 274.32 368.3 90)
 		(unit 1)
 		(body_style 1)
@@
 	(symbol
 		(lib_id "Connector:TestPoint")
-		(at 641.35 60.96 0)
+		(at 617.22 60.96 0)
 		(unit 1)
 		(body_style 1)
@@
 		(dnp no)
 		(property "Reference" "TP401"
-			(at 641.35 53.34 0)
+			(at 617.22 53.34 0)
 			(hide yes)
 			(show_name no)
@@
 			)
 		)
-		(property "Value" "OUT"
-			(at 642.15 57.76 0)
+		(property "Value" "IN"
+			(at 616.42 57.76 0)
 			(show_name no)
 			(do_not_autoplace no)
@@
 					(size 1.27 1.27)
 				)
-				(justify left)
+				(justify right)
 			)
 		)
 		(property "Footprint" "amod:TestPoint_Loop_RH-5019"
-			(at 641.35 60.96 0)
+			(at 617.22 60.96 0)
 			(hide yes)
 			(show_name no)
@@
 		)
 		(property "Datasheet" ""
-			(at 641.35 60.96 0)
+			(at 617.22 60.96 0)
 			(hide yes)
 			(show_name no)
@@
 		)
 		(property "Description" ""
-			(at 641.35 60.96 0)
+			(at 617.22 60.96 0)
 			(hide yes)
 			(show_name no)
@@
 		)
 		(property "LCSC" "C5199800"
-			(at 641.35 60.96 0)
+			(at 617.22 60.96 0)
 			(hide yes)
 			(show_name no)
@@
 		)
 		(property "MPN" "RH-5019"
-			(at 641.35 60.96 0)
+			(at 617.22 60.96 0)
 			(hide yes)
 			(show_name no)
@@
 	(symbol
 		(lib_id "Device:R_US")
-		(at 233.68 368.3 270)
-		(mirror x)
+		(at 233.68 368.3 90)
 		(unit 1)
 		(body_style 1)
@@
 	(symbol
 		(lib_id "Device:C")
-		(at 632.46 83.82 90)
+		(at 632.46 83.82 270)
+		(mirror x)
 		(unit 1)
 		(body_style 1)
