File: hardware/amod_p.kicad_sch (KiCad schematic)
At the start: 151 parts, among them J1001 SMA, J1002 SMA, J101 SMA, J102 SMA, J1101 SMA, J1102 SMA, J1103 SMA, J1104 SMA, J1105 SMA, J1201 SMA, J1301 SMA, J1302 coil, J1303 VAR C, J201 SMA, J202 SMA, J301 SMA, J302 SMA, J401 SMA, J402 SMA, J501 SMA, J502 SMA, J601 SMA, J602 SMA, J701 SMA, J702 SMA, J801 SMA, J802 SMA, J901 SMA, J902 SMA, SW1201 DIP4, SW1301 DIP4, SW401 DIP2, Y801 4 MHz, Y901 455 kHz

Commit message: One letter per board, tiles in lower case: AMOD-P2 is AMOD-N (n1-n11), RF-MOD-2 is IQ-MOD (q1-q11), PhMOD's tiles h1-h10
Jason, Prompt 19: "If we can have a nice, well justified single-letter designator for each board, it would make
everything much more clear", and "d11, q11, and c11 don't look like obvious electronics or PCB things".

- p passive, n networks (AMOD-P2's P14, P16-P25), a active, r radio, h PhMOD (Y1-Y10), q quadrature (RF-MOD-2's X1-X11);
  c, m and b are taken for the conversion, motor and brushless boards to come.  PLAN.md section 13 has the table and
  the reasons (no letter moves to another board, no retired name is reused, no s: s11 is the reflection coefficient).
- Every tile name in lower case on the silk, in the code (Tile ids, BACK/BACK_PLOTS/DOCS keys, the nets built on them),
  the handbooks, README, DOA lists, KIT, PLAN and the review brief; pin names (USB-C A1...), the 4046's R1/C1, nets
  named N1/P1, part numbers ending -R7 and the paper size A1 left alone.  tiles.dump refuses a tile not named
  <letter><n>, a number twice, and a BACK key for a tile that does not exist.
- Board and file renames: boards/amod_n.py, boards/iq_mod.py, docs/DOA_amod_n.md, docs/DOA_iq_mod.md, the handbooks,
  the generated hardware, outputs and pictures.  Silk nudged where a lower-case p or q hung onto the line below.
- All six boards rebuilt: ERC 0, DRC 0, every check.

Co-Authored-By: Claude Opus 5.5 <noreply@anthropic.com>
Claude-Session: https://claude.ai/code/session_01RKeoKvFFzjk3cEBLCXXHnB
Connections:
- net P10_IN renamed p10_IN
- net P10_OUT renamed p10_OUT
- net P11_OUT renamed p11_OUT
- net P11_T1 renamed p11_T1
- net P11_T2 renamed p11_T2
- net P11_T3 renamed p11_T3
- net P12_BUS renamed p12_BUS
- net P13_HOT renamed p13_HOT
- net P13_TAP renamed p13_TAP
- net P1_IN renamed p1_IN
- net P1_OUT renamed p1_OUT
- net P2_IN renamed p2_IN
- net P2_OUT renamed p2_OUT
- net P3_IN renamed p3_IN
- net P3_OUT renamed p3_OUT
- net P4_IN renamed p4_IN
- net P4_N1 renamed p4_N1
- net P4_OUT renamed p4_OUT
- net P5_IN renamed p5_IN
- net P5_N1 renamed p5_N1
- net P5_OUT renamed p5_OUT
- net P6_IN renamed p6_IN
- net P6_OUT renamed p6_OUT
- net P7_IN renamed p7_IN
- net P7_N1 renamed p7_N1
- net P7_N2 renamed p7_N2
- net P7_N3 renamed p7_N3
- net P7_OUT renamed p7_OUT
- net P8_IN renamed p8_IN
- net P8_OUT renamed p8_OUT
- net P9_IN renamed p9_IN
- net P9_OUT renamed p9_OUT
Other:
- note added: "EXPECT: a pass near 455 kHz and a notch a few kHz above: a resonator with a Q of a few hundred, between p4's LC and p8's quartz"
- note added: "The mirror image of p2: the same 1 k and 1 nF the other way round. A step in gives a spike that decays in 1 us."
- note added: "Turns a one-bit (delta-sigma) DAC stream into a tone; a slow plant for feedback control, with p2."
- note added: "p1 pi pad, -20 dB"
- note added: "p10 clipper, 1N4148 ±0.6 V"
- note added: "p11 delay line, 400 ns, a tap every 100"
- note added: "p12 LEDs"
- note added: "p13 AM loopstick, 0.5-1.7 MHz"
- note added: "p2 RC low-pass, 159 kHz"
- note added: "p3 RC high-pass, 159 kHz"
- note added: "p4 series RLC, 100uH 220pF"
- note added: "p5 LC low-pass, 9 MHz"
- note added: "p6 LC low-pass, 100 kHz"
- note added: "p7 band-pass, 4.7-7.5 MHz"
- note added: "p8 quartz crystal, 4 MHz"
- note added: "p9 ceramic res., 455 kHz"
- note added: "to a4"
- note added: "variable with a big knob tunes the whole band alone, switches off); its frame to GND. Into a4's LNA and the AM radio gateware."
- note removed: "EXPECT: a pass near 455 kHz and a notch a few kHz above: a resonator with a Q of a few hundred, between P4's LC and P8's quartz"
- note removed: "P1 pi pad, -20 dB"
- note removed: "P10 clipper, 1N4148 ±0.6 V"
- note removed: "P11 delay line, 400 ns, a tap every 100"
- note removed: "P12 LEDs"
- note removed: "P13 AM loopstick, 0.5-1.7 MHz"
- note removed: "P2 RC low-pass, 159 kHz"
- note removed: "P3 RC high-pass, 159 kHz"
- note removed: "P4 series RLC, 100uH 220pF"
- note removed: "P5 LC low-pass, 9 MHz"
- note removed: "P6 LC low-pass, 100 kHz"
- note removed: "P7 band-pass, 4.7-7.5 MHz"
- note removed: "P8 quartz crystal, 4 MHz"
- note removed: "P9 ceramic res., 455 kHz"
- note removed: "The mirror image of P2: the same 1 k and 1 nF the other way round. A step in gives a spike that decays in 1 us."
- note removed: "Turns a one-bit (delta-sigma) DAC stream into a tone; a slow plant for feedback control, with P2."
- note removed: "to A4"
- note removed: "variable with a big knob tunes the whole band alone, switches off); its frame to GND. Into A4's LNA and the AM radio gateware."
