File: hardware/amod_2.kicad_sch (KiCad schematic)
At the start: 101 parts, among them J101 USB-C, J201 SMA, J202 SMA, J301 SMA, J302 SMA, J303 SMA, J304 SMA, J501 SMA, J502 SMA, J503 SMA, J504 SMA, J505 Pmod, Q301 AO3401A, Q501 AO3401A, SW301 ON, SW501 ON, U101 TPS65131, U102 LM2664, U201 THS3491, U301 OPA847, U501 LMH6629, U502 LMH6629

Commit message: AMOD-2 in progress: Y9 switched noise source, Y7 reflection bridge (INC and REFL = 2A - 2B), Y8 passive coupled resonators with capacitive ports
ERC 0, DRC 0.  IO8 reaches Y9 round the left and top margins; Y9's -5 V up a finger of L3 from the gutter.

Co-Authored-By: Claude Opus 5.5 <noreply@anthropic.com>
Claude-Session: https://claude.ai/code/session_01RKeoKvFFzjk3cEBLCXXHnB
Parts:
- added C701, C702, C703, C704, C809, C902, C904, C908: 100n, Capacitor_SMD:C_0402_1005Metric, symbol Device:C
- added C801, C803, C805, C808: 2.2p, Capacitor_SMD:C_0402_1005Metric, symbol Device:C
- added C802: 4.7p, Capacitor_SMD:C_0402_1005Metric, symbol Device:C
- added C804: 1p, Capacitor_SMD:C_0402_1005Metric, symbol Device:C
- added C806: 1n, Capacitor_SMD:C_0402_1005Metric, symbol Device:C
- added C807: 6.8p, Capacitor_SMD:C_0402_1005Metric, symbol Device:C
- added C901, C905, C906, C907: 1u, Capacitor_SMD:C_0402_1005Metric, symbol Device:C
- added C903: 100p, Capacitor_SMD:C_0402_1005Metric, symbol Device:C
- added D801, D802, D803, D804: BB133, Diode_SMD:D_SOD-323, symbol Device:D_Capacitance
- added J701, J702, J703, J704, J801, J802, J803, J804, J901: SMA, amod:SMA_BWSMA-KE-Z001_Vertical, symbol Connector:Conn_Coaxial
- added L801, L802: 10u, Inductor_SMD:L_1210_3225Metric, symbol Device:L
- added Q701, Q801, Q901: AO3401A, Package_TO_SOT_SMD:SOT-23, symbol Transistor_FET:AO3401A
- added Q902: MMBT3904, Package_TO_SOT_SMD:SOT-23, symbol Transistor_BJT:MMBT3904
- added R701, R702, R703, R706, R709, R801, R906: 49.9, Resistor_SMD:R_0402_1005Metric, symbol Device:R_US
- added R704, R705, R707, R708: 499, Resistor_SMD:R_0402_1005Metric, symbol Device:R_US
- added R802, R803, R805, R806: 100k, Resistor_SMD:R_0402_1005Metric, symbol Device:R_US
- added R804, R807: 2k, Resistor_SMD:R_0402_1005Metric, symbol Device:R_US
- added R901: 680, Resistor_SMD:R_0402_1005Metric, symbol Device:R_US
- added R902, R903: 10k, Resistor_SMD:R_0402_1005Metric, symbol Device:R_US
- added R904: 240, Resistor_SMD:R_0402_1005Metric, symbol Device:R_US
- added R905: 27, Resistor_SMD:R_0402_1005Metric, symbol Device:R_US
- added SW701, SW801, SW901: ON, amod:SW_SPDT_Shouhan_MSK12C02, symbol Switch:SW_SPDT
- added SW802: DIP4, amod:SW_DIP_SPSTx04_Slide_1.27mm_DSHP04, symbol Switch:SW_DIP_x04
- added U701, U702: OPA810, Package_TO_SOT_SMD:SOT-23-5, symbol amod:OPA_SOT23-5
- added U901: TPS22917, Package_TO_SOT_SMD:SOT-23-6, symbol Power_Management:TPS22917DBV
- added U902: LMH6629, Package_TO_SOT_SMD:SOT-23-5, symbol amod:OPA_SOT23-5
Connections:
- net +5V: now also Q701.2 (S), Q801.2 (S), Q901.2 (S), SW701.3 (C), SW801.3 (C), SW901.3 (C)
- net -5V: now also C701.1, C702.1, C903.1, C904.1, Q902.1 (B), U701.2 (V-), U702.2 (V-)
- net GND: now also C701.2, C702.2, C703.2, C704.2, C802.2, C807.2, C809.2, C901.2, C902.2, C903.2, C904.2, C906.2, C908.2, D802.2 (A), D804.2 (A), J701.2 (Ext), J702.2 (Ext), J703.2 (Ext), J704.2 (Ext), J801.2 (Ext), J802.2 (Ext), J803.2 (Ext), J804.2 (Ext), J901.2 (Ext), L801.2, L802.2, R703.2, R705.1, R801.2, R803.2, R903.1, SW701.1 (A), SW801.1 (A), SW802.3, SW802.4, SW901.1 (A), U901.2 (GND), U902.2 (V-)
- net PMOD8: now reaches J505.5 (Pin_5)
- net PMOD8: now also U901.3 (ON)
- new net Y7_A: J703.1 (In), R701.2, U702.3 (+IN)
- new net Y7_B: R702.2, R703.1, U701.3 (+IN)
- new net Y7_DRV: J701.1 (In), R701.1, R702.1
- new net Y7_G: Q701.1 (G), SW701.2 (B)
- new net Y7_INC: J702.1 (In), R706.2
- new net Y7_N1: R704.1, R705.2, U701.4 (-IN)
- new net Y7_N2: R707.2, R708.1, U702.4 (-IN)
- new net Y7_O1: R704.2, R706.1, R707.1, U701.1 (OUT)
- new net Y7_O2: R708.2, R709.1, U702.1 (OUT)
- new net Y7_REFL: J704.1 (In), R709.2
- new net Y7_VS: C703.1, C704.1, Q701.3 (D), U701.5 (V+), U702.5 (V+)
- new net Y8_CA: C804.2, SW802.8
- new net Y8_CB: C805.2, SW802.7
- new net Y8_G: Q801.1 (G), SW801.2 (B)
- new net Y8_K1: D801.1 (K), D802.1 (K), R802.2, R803.1
- new net Y8_K2: C806.1, D803.1 (K), D804.1 (K), R805.1, R806.1
- new net Y8_OUT1: C803.2, J802.1 (In)
- new net Y8_OUT2: C808.2, J804.1 (In)
- new net Y8_RDA: R804.2, SW802.6
- new net Y8_RDB: R807.2, SW802.5
- new net Y8_SIG: C801.1, J801.1 (In), R801.1
- new net Y8_T1: C801.2, C802.1, C803.1, C804.1, C805.1, D801.2 (A), L801.1, R804.1
- new net Y8_T2: C807.1, C808.1, D803.2 (A), L802.1, R807.1, SW802.1, SW802.2
- new net Y8_TP: C806.2, J803.1 (In), R805.2
- new net Y8_VS: C809.1, Q801.3 (D), R802.1, R806.2
- new net Y9_CG: C906.1, R905.2
- new net Y9_FB: R904.1, R905.1, U902.4 (-IN)
- new net Y9_G: Q901.1 (G), SW901.2 (B)
- new net Y9_IN: C905.1, Q902.2 (E), R901.2
- new net Y9_IN2: C905.2, R902.1, R903.2, U902.3 (+IN)
- new net Y9_OA: C907.1, R904.2, U902.1 (OUT)
- new net Y9_OC: C907.2, R906.1
- new net Y9_OUT: J901.1 (In), R906.2
- new net Y9_VN: C902.1, R901.1, U901.6 (VOUT)
- new net Y9_VS: C901.1, C908.1, Q901.3 (D), R902.2, U901.1 (VIN), U902.5 (V+)
- no-connect marks 21 -> 23
Other:
- note added: "(a lossy tank coupled to a sharp one: the EIT analogue). A pump at twice the frequency on TUNE / PUMP: parametric gain."
- note added: "+-1 V into 50 ohm"
- note added: "+-2 V open"
- note added: "1 pF and 2.2 pF between the tanks (normal modes, the avoided crossing as TUNE sweeps tank 2), 2 k across tank 1 or tank 2"
- note added: "2-3 mA and its avalanche noise, many times kT's, goes straight into an LMH6629 at gain 9.9 and out through 49.9 ohm. IO8"
- note added: "A - B = B x Gamma. OPA810 U1 at gain 2 on B gives INC; U2, +IN on A and 499 / 499 ohm from U1's output, gives 2 A - 2 B,"
- note added: "A 50 ohm resistive bridge: D from DRIVE, 49.9 ohm to A (the DUT jack) and 49.9 + 49.9 ohm from D to ground with B between."
- note added: "An MMBT3904's emitter-base junction breaks down near 8 V; between -5 V and the switched 5 V through 680 ohm it carries"
- note added: "DRIVE"
- note added: "DUT"
- note added: "EXPECT: REFL / INC = Gamma (S11) from DC to about 30 MHz: 0 for 50 ohm, +1 open, -1 short; after open-short-load calibration, better than -35 dB"
- note added: "EXPECT: off: the amplifier's own noise (about 6 nV/rtHz at OUT); on: tens to hundreds of nV/rtHz from 10 kHz to 50 MHz, flat to about 1 dB"
- note added: "EXPECT: two 10 MHz tanks (Q about 30); coupled by 1, 2.2 or 3.2 pF they split by 0.4 - 1.2 MHz; TUNE moves tank 2 by +-5 %; a 20 MHz pump on it gives parametric gain"
- note added: "INC"
- note added: "OUT 1"
- note added: "OUT 2"
- note added: "REFL"
- note added: "REFL; each leaves through 49.9 ohm, so into the host's 50 ohm inputs REFL / INC = Gamma, magnitude and phase. Calibrate"
- note added: "SIG"
- note added: "SIG drives tank 1 through 2.2 pF; each tank feeds its OUT jack through 2.2 pF, -43 dB into the host's 50 ohm. The DIP:"
- note added: "TUNE / PUMP"
- note added: "Two LC tanks, 10 uH and about 25 pF each (fixed, two BB133 back to back at 2.5 V, the ports), near 10 MHz, Q about 30."
- note added: "Y7 reflection bridge, 2 x OPA810"
- note added: "Y8 coupled resonators, 2 x LC + BB133"
- note added: "Y9 noise source, MMBT3904 + LMH6629"
- note added: "cell (3,0)"
- note added: "cells (0,1), (1,1)"
- note added: "cells (0,2), (1,2)"
- note added: "cross-spectrum against the response on the host's second ADC is a transfer function."
- note added: "high turns it on (a TPS22917 switches its 5 V): hot and cold for a Y-factor noise figure, or a broadband stimulus whose"
- note added: "with an open, a short and a 50 ohm load on DUT (three complex numbers per frequency), then match an NMR probe or an antenna."

Commit message: AMOD-2 in progress: Y10 laser driver (100 mA/V high-side source, IO5 shunt, 20 MHz - 3 GHz bias-T, diode-voltage monitor)
ERC 0, DRC 0.  IO5 up the gutter at x 50.4; a foot moved off the LD jack.

Co-Authored-By: Claude Opus 5.5 <noreply@anthropic.com>
Claude-Session: https://claude.ai/code/session_01RKeoKvFFzjk3cEBLCXXHnB
Parts:
- added C1001, C1002, C1006: 100n, Capacitor_SMD:C_0402_1005Metric, symbol Device:C
- added C1003: 10n, Capacitor_SMD:C_0402_1005Metric, symbol Device:C
- added C1004: 10u, Capacitor_SMD:C_0805_2012Metric, symbol Device:C
- added C1005: 100p, Capacitor_SMD:C_0402_1005Metric, symbol Device:C
- added D1001: B5819W, Diode_SMD:D_SOD-123, symbol Device:D_Schottky
- added J1001, J1002, J1003, J1004: SMA, amod:SMA_BWSMA-KE-Z001_Vertical, symbol Connector:Conn_Coaxial
- added L1001: 330n, Inductor_SMD:L_0805_2012Metric, symbol Device:L
- added L1002: 27n, Inductor_SMD:L_0402_1005Metric, symbol Device:L
- added Q1001, Q1003: AO3401A, Package_TO_SOT_SMD:SOT-23, symbol Transistor_FET:AO3401A
- added Q1002: 2N7002, Package_TO_SOT_SMD:SOT-23, symbol Transistor_FET:2N7002
- added Q1004: AO3400A, Package_TO_SOT_SMD:SOT-23, symbol Transistor_FET:AO3400A
- added R1001: 49.9, Resistor_SMD:R_0402_1005Metric, symbol Device:R_US
- added R1002, R1003, R1004, R1006: 1k, Resistor_SMD:R_0402_1005Metric, symbol Device:R_US
- added R1005: 100, Resistor_SMD:R_0402_1005Metric, symbol Device:R_US
- added R1007: 10, Resistor_SMD:R_0805_2012Metric, symbol Device:R_US
- added R1008: 47, Resistor_SMD:R_0402_1005Metric, symbol Device:R_US
- added R1009: 10k, Resistor_SMD:R_0402_1005Metric, symbol Device:R_US
- added R1010: 100k, Resistor_SMD:R_0402_1005Metric, symbol Device:R_US
- added SW1001: ON, amod:SW_SPDT_Shouhan_MSK12C02, symbol Switch:SW_SPDT
- added U1001, U1002: OPA810, Package_TO_SOT_SMD:SOT-23-5, symbol amod:OPA_SOT23-5
Connections:
- net +5V: now also Q1001.2 (S), SW1001.3 (C)
- net GND: now also C1001.2, C1002.2, C1004.1, C1006.2, D1001.2 (A), J1001.2 (Ext), J1002.2 (Ext), J1003.2 (Ext), J1004.2 (Ext), Q1004.2 (S), R1001.2, R1003.2, R1010.2, SW1001.1 (A), U1001.2 (V-), U1002.2 (V-)
- net PMOD5: now reaches J505.11 (Pin_11)
- net PMOD5: now also Q1004.1 (G), R1010.1
- new net Y10_G: Q1001.1 (G), SW1001.2 (B)
- new net Y10_GA: C1003.2, R1005.1, U1002.1 (OUT)
- new net Y10_GB: Q1002.1 (G), U1001.1 (OUT)
- new net Y10_GQ: Q1003.1 (G), R1005.2
- new net Y10_ID: D1001.1 (K), L1001.1, Q1003.3 (D), Q1004.3 (D)
- new net Y10_LDN: J1004.1 (In), L1002.2, R1008.2, R1009.2
- new net Y10_LM: L1001.2, L1002.1
- new net Y10_MON: J1002.1 (In), R1009.1
- new net Y10_NA: C1003.1, R1006.2, U1002.4 (-IN)
- new net Y10_NS: Q1002.2 (S), R1003.1, U1001.4 (-IN)
- new net Y10_REF: Q1002.3 (D), R1004.2, U1002.3 (+IN)
- new net Y10_RF: C1005.1, J1003.1 (In)
- new net Y10_RFC: C1005.2, R1008.1
- new net Y10_SET: J1001.1 (In), R1001.1, R1002.1
- new net Y10_SETF: C1001.1, R1002.2, U1001.3 (+IN)
- new net Y10_SQ: Q1003.2 (S), R1006.1, R1007.2
- new net Y10_VS: C1002.1, C1004.2, C1006.1, Q1001.3 (D), R1004.1, R1007.1, U1001.5 (V+), U1002.5 (V+)
- no-connect marks 23 -> 22
Other:
- note added: "+10 dBm max"
- note added: "0-1 V: 0-100 mA"
- note added: "100 mA max"
- note added: "330 nH + 27 nH; RF IN joins through 100 pF + 47 ohm: the modulation for a rubidium CPT clock (3.4 GHz) or NV ODMR. IO5 high"
- note added: "A high-side current source: REF = VS - SET (OPA810 and a 2N7002 through 1 k / 1 k), OPA810 holds the AO3401's source at"
- note added: "EXPECT: 0-100 mA from 0-1 V on SET, about 10 kHz of loop bandwidth; IO5 blanks it in about 1 us; RF from about 20 MHz to 3 GHz rides on the current"
- note added: "LD"
- note added: "MON"
- note added: "REF so 10 ohm carries SET / 10 ohm, 100 mA per volt (start a VCSEL at a few millivolts). The drain feeds the diode through"
- note added: "RF IN"
- note added: "SET"
- note added: "Y10 laser driver, current source + bias-T"
- note added: "cells (2,2), (3,2)"
- note added: "shorts the drain (the AO3400) for pulses. MON = the diode's voltage / 200 into 50 ohm: with SET swept, its I-V curve."

Commit message: AMOD-2 rev A: all ten tiles (Y6 VLF loop amplifier, Y4 DRV8876 coil driver added); per-board fiducials
ERC 0, DRC 0.  IO6 / IO7 reach Y4 on the back along the bottom edge and across the top of Y6; the third fiducial
moves off Y4's coil terminal (FIDUCIALS in the board module, default unchanged).

Co-Authored-By: Claude Opus 5.5 <noreply@anthropic.com>
Claude-Session: https://claude.ai/code/session_01RKeoKvFFzjk3cEBLCXXHnB
Parts:
- added C401: 10u, Capacitor_SMD:C_0805_2012Metric, symbol Device:C
- added C402: 22n, Capacitor_SMD:C_0402_1005Metric, symbol Device:C
- added C403, C605: 100n, Capacitor_SMD:C_0402_1005Metric, symbol Device:C
- added C601, C602, C604: 1u, Capacitor_SMD:C_0402_1005Metric, symbol Device:C
- added C603: 100p, Capacitor_SMD:C_0402_1005Metric, symbol Device:C
- added D401, D402: B5819W, Diode_SMD:D_SOD-123, symbol Device:D_Schottky
- added J401, J601, J602: SMA, amod:SMA_BWSMA-KE-Z001_Vertical, symbol Connector:Conn_Coaxial
- added J402: VM in, amod:TerminalBlock_KF301_1x02_P5.00mm, symbol Connector:Screw_Terminal_01x02
- added J403: coil, amod:TerminalBlock_KF301_1x02_P5.00mm, symbol Connector:Screw_Terminal_01x02
- added Q401, Q601: AO3401A, Package_TO_SOT_SMD:SOT-23, symbol Transistor_FET:AO3401A
- added R401, R402, R601, R602: 100k, Resistor_SMD:R_0402_1005Metric, symbol Device:R_US
- added R403: 5.1k, Resistor_SMD:R_0402_1005Metric, symbol Device:R_US
- added R404: 3.3k, Resistor_SMD:R_0402_1005Metric, symbol Device:R_US
- added R405: 1.5k, Resistor_SMD:R_0402_1005Metric, symbol Device:R_US
- added R406, R605: 49.9, Resistor_SMD:R_0402_1005Metric, symbol Device:R_US
- added R603: 10k, Resistor_SMD:R_0402_1005Metric, symbol Device:R_US
- added R604: 100, Resistor_SMD:R_0402_1005Metric, symbol Device:R_US
- added SW401, SW601: ON, amod:SW_SPDT_Shouhan_MSK12C02, symbol Switch:SW_SPDT
- added U401: DRV8876, Package_SO:HTSSOP-16-1EP_4.4x5mm_P0.65mm_EP3.4x5mm_Mask2.66x2.46mm, symbol amod:DRV8876
- added U402, U601: OPA810, Package_TO_SOT_SMD:SOT-23-5, symbol amod:OPA_SOT23-5
Connections:
- net +5V: now also Q401.2 (S), Q601.2 (S), SW401.3 (C), SW601.3 (C)
- net GND: now also C401.1, C602.2, C605.2, J401.2 (Ext), J402.2 (Pin_2), J601.2 (Ext), J602.2 (Ext), R401.1, R402.1, R404.2, R405.1, R602.1, SW401.1 (A), SW601.1 (A), U401.15 (GND), U401.16 (PMODE), U401.17 (PAD), U401.7 (IMODE), U401.9 (PGND), U402.2 (V-), U601.2 (V-)
- net PMOD7: now reaches J505.7 (Pin_7)
- net PMOD7: now also R402.2, U401.2 (PH/IN2)
- net PMOD6: now reaches J505.9 (Pin_9)
- net PMOD6: now also R401.2, U401.1 (EN/IN1)
- new net Y4_CPH: C402.1, U401.13 (CPH)
- new net Y4_CPL: C402.2, U401.14 (CPL)
- new net Y4_G: Q401.1 (G), SW401.2 (B)
- new net Y4_IP: R405.2, U401.6 (IPROPI), U402.3 (+IN)
- new net Y4_MO: R406.2, U402.1 (OUT), U402.4 (-IN)
- new net Y4_MON: J401.1 (In), R406.1
- new net Y4_OUT1: J403.2 (Pin_2), U401.8 (OUT1)
- new net Y4_OUT2: J403.1 (Pin_1), U401.10 (OUT2)
- new net Y4_VCP: C403.2, U401.12 (VCP)
- new net Y4_VEXT: D402.2 (A), J402.1 (Pin_1)
- new net Y4_VM: C401.2, C403.1, D401.1 (K), D402.1 (K), U401.11 (VM), U402.5 (V+)
- new net Y4_VREF: R403.2, R404.1, U401.5 (VREF)
- new net Y4_VS: D401.2 (A), Q401.3 (D), R403.1, U401.3 (~{SLEEP})
- new net Y6_CG: C602.1, R604.2
- new net Y6_FB: C603.1, R603.1, R604.1, U601.4 (-IN)
- new net Y6_G: Q601.1 (G), SW601.2 (B)
- new net Y6_IN: C601.1, J601.1 (In)
- new net Y6_IN2: C601.2, R601.1, R602.2, U601.3 (+IN)
- new net Y6_OA: C603.2, C604.1, R603.2, U601.1 (OUT)
- new net Y6_OC: C604.2, R605.1
- new net Y6_OUT: J602.1 (In), R605.2
- new net Y6_VS: C605.1, Q601.3 (D), R601.2, U601.5 (V+)
- no-connect marks 22 -> 21
Other:
- note added: "(lightning, thousands of kilometres away), NAA's 24 kHz MSK, WWVB's 60 kHz time code. Two loops at right angles (this and"
- note added: "A loop's EMF is N A dB/dt: a 1 m square of 10 turns gives about 1 uV for 1 pT at 20 kHz. 1 uF into an OPA810 at half"
- note added: "DRV8876 in PH/EN mode: IO6 enables (PWM), IO7 the direction; VM = USB or 12-18 V (two B5819W); IPROPI buffered to MON."
- note added: "EXPECT: about 1.3 A either way into a coil, PWM on IO6; MON about 1.5 V per amp"
- note added: "EXPECT: gain 101 from 1.6 kHz to 160 kHz (the loop's EMF rises with frequency on top): sferics, the Navy's MSK stations near 24 kHz, WWVB at 60 kHz"
- note added: "IPROPI"
- note added: "LOOP"
- note added: "Y4 coil driver, DRV8876"
- note added: "Y5's IN A, or two boards) give a lightning stroke's bearing from the ratio of the two signals."
- note added: "Y6 VLF loop amplifier, OPA810 x101"
- note added: "cell (2,3)"
- note added: "cell (3,3)"
- note added: "mV"
- note added: "the supply (100 k / 100 k), gain 101 (10 k / 100 ohm to ground through 1 uF), 100 pF across 10 k: 1.6 - 160 kHz. Sferics"
