File: hardware/rf_mod_2.kicad_sch (KiCad schematic)
At the start: 184 parts, among them J1001 USB-C, J101 SMA, J102 SMA, J103 SMA, J104 SMA, J1101 SMA, J1102 SMA, J1103 SMA, J201 SMA, J202 SMA, J203 SMA, J204 SMA, J301 SMA, J302 SMA, J303 Pmod, J401 SMA, J402 SMA, J501 SMA, J502 SMA, J503 SMA, J601 SMA, J602 SMA, J701 SMA, J801 SMA, J802 SMA, J901 SMA, J902 SMA, Q101 AO3401A, Q201 AO3401A, Q301 AO3401A, Q401 AO3401A, Q601 AO3401A, Q701 AO3401A, Q702 MMBT3904, Q801 AO3401A, SW101 ON, SW201 ON, SW301 ON, SW401 ON, SW601 ON, SW701 ON, SW801 ON, U1001 LM2664, U101 ADL5375, U1101 SKY13370, U201 ADL5380, U202 OPA810, U203 OPA810, U301 3.3V, U302 MAX2871, U401 QPL9547, U601 AD8318, U701 TPS22917, U702 ADL5611, U801 MAX2659, U802 3.3V

Commit message: RF-MOD-2: X5 is a dual directional coupler (two HHM22137A1 back to back, 0.6-3.5 GHz, FWD and REFL 25 dB down, 20 dB directivity) in the splitter's place; X3's RFOUTA- on OUT A- (its right cell's bottom-right) so OUT A+ and OUT A- are X1's and X2's LOs, REF IN moved to the right cell's top-left with its line on the back; IO5 and IO6 lowered in the margin under OUT A-'s line
Co-Authored-By: Claude Opus 5.5 <noreply@anthropic.com>
Claude-Session: https://claude.ai/code/session_01RKeoKvFFzjk3cEBLCXXHnB
Parts:
- removed R306: 5.1k, Resistor_SMD:R_0402_1005Metric, symbol Device:R_US
- removed R503: 18R, Resistor_SMD:R_0402_1005Metric, symbol Device:R_US
- added J304: Pmod, amod:PinHeader_2x06_P2.54mm_Horizontal_PZ254R-12-12P, symbol Connector_Generic:Conn_02x06_Odd_Even
- added J504: SMA, amod:SMA_BWSMA-KE-Z001_Vertical, symbol Connector:Conn_Coaxial
- added U501, U502: HHM22137A1, amod:Coupler_1608-6P_HHM22137A1, symbol amod:HHM22137
- J303: value Pmod -> SMA; footprint amod:PinHeader_2x06_P2.54mm_Horizontal_PZ254R-12-12P -> amod:SMA_BWSMA-KE-Z001_Vertical; symbol Connector_Generic:Conn_02x06_Odd_Even -> Connector:Conn_Coaxial; LCSC C492434 -> C496549; MPN PZ254R-12-12P -> BWSMA-KE-Z001
- R305: value 51R -> 5.1k; LCSC C25125 -> C25905; MPN 0402WGF510JTCE -> 0402WGF5101TCE
- R501, R502: value 18R -> 51R; LCSC C25084 -> C25125; MPN 0402WGF180JTCE -> 0402WGF510JTCE
Connections:
- net X5_N is gone; now on net GND: R501.2, R502.1
- net GND: now also J303.2 (Ext), J304.3 (Pin_3), J304.4 (Pin_4), J504.2 (Ext), U501.2 (GND), U501.5 (GND), U502.2 (GND), U502.5 (GND); no longer J303.3 (Pin_3), J303.4 (Pin_4)
- net PMOD1: now also J304.12 (Pin_12); no longer J303.12 (Pin_12)
- net PMOD2: now also J304.10 (Pin_10); no longer J303.10 (Pin_10)
- net PMOD3: now also J304.8 (Pin_8); no longer J303.8 (Pin_8)
- net PMOD4: now also J304.6 (Pin_6); no longer J303.6 (Pin_6)
- net PMOD5: now also J304.11 (Pin_11); no longer J303.11 (Pin_11)
- net PMOD6: now also J304.9 (Pin_9); no longer J303.9 (Pin_9)
- net PMOD8: now also J304.5 (Pin_5); no longer J303.5 (Pin_5)
- net PMOD_VCC: now also J304.1 (Pin_1), J304.2 (Pin_2); no longer J303.1 (Pin_1), J303.2 (Pin_2)
- net X3_RS: now also R305.1
- net X3_TRM renamed X3_OUTAN
- net X3_OUTAN: now also J303.1 (In); no longer R305.1
- net X5_P1 renamed X5_IN
- net X5_IN: now also U501.3 (IN); no longer R501.1
- net X5_P2 renamed X5_FWD
- net X5_FWD: now also U501.4 (CPL)
- net X5_P3 renamed X5_REFL
- net X5_REFL: now also U502.4 (CPL); no longer R502.2
- new net X5_MID: U501.1 (OUT), U502.1 (OUT)
- new net X5_OUT: J504.1 (In), U502.3 (IN)
- new net X5_TA: R501.1, U501.6 (ISO)
- new net X5_TB: R502.2, U502.6 (ISO)
Other:
- note added: "3.3 V and 100 pF: two outputs, 180 degrees apart; put a 50 ohm terminator on one that is unused. RFOUTB is open and must"
- note added: "EXPECT: FWD 25 dB below the wave going from IN to OUT and REFL 25 dB below the wave coming back from OUT, 0.6-2.7 GHz (27 dB at 0.6, 14 dB at 3.5 GHz); 0.3 dB through; about 20 dB of directivity: with a device on OUT, REFL / FWD is its reflection coefficient"
- note added: "EXPECT: any frequency from 23.5 MHz to 6 GHz on OUT A+ and OUT A- (each -4 to +5 dBm, 180 degrees apart), locked to the 25 MHz on REF IN (the ECP5 board's CLK OUT or RF-MOD's REF OUT): OUT A+ is X1's LO and OUT A- X2's, one phase for both"
- note added: "FWD"
- note added: "OUT A+"
- note added: "OUT A-"
- note added: "REFL"
- note added: "REFL into X2 (and FWD into X6 or through X11): the device's S11 in magnitude and phase. Directivity (about 20 dB) limits"
- note added: "Two TDK HHM22137A1 directional couplers back to back, each with its isolated port in 51 ohm: the first samples the wave"
- note added: "X5 coupler, 2 x HHM22137A1"
- note added: "and 2.4 GHz (VCO / 2) at ICP 2.56 mA (RSET 5.1 k, CP = 7). RFOUTA+ and RFOUTA- each feed a jack through 27 nH to"
- note added: "and IP2). ADJ 1.5 k to 5 V suits 0.4-3 GHz (open it above 5 GHz). With X3's two outputs on the LOs: one coherent radio."
- note added: "board's CLK OUT or RF-MOD's REF OUT. OUT A+ into X1's LO and OUT A- into X2's at -1 dBm (X1 wants 0, X2 -6 to +6)."
- note added: "going from IN to OUT (FWD), the second, turned round, the wave coming back from OUT (REFL). X1 on IN, a device on OUT,"
- note added: "stay disabled. CE and RFOUT_EN are tied high, LE has 100 k down. REF IN is unterminated (3.3 V CMOS): the ECP5"
- note added: "the smallest reflection it sees; calibrate with open, short and load. +35 dBm through; terminate an unused port in 50 ohm."
- note removed: "+20 dBm"
- note removed: "100 pF; RFOUTA- is terminated in 51 ohm the same way; RFOUTB is open and must stay disabled. CE and RFOUT_EN are"
- note removed: "EXPECT: 6.2 dB from any port to either other port, every port within 2 ohm of 50, DC to 6 GHz"
- note removed: "EXPECT: any frequency from 23.5 MHz to 6 GHz on OUT A (-4 to +5 dBm), locked to the 25 MHz on REF IN (the ECP5 board's CLK OUT or RF-MOD's REF OUT); through X5 it is the LO of X1 and X2 at once"
- note removed: "Here it splits X3's OUT A into X1's and X2's LO inputs, so the transmitter and the receiver share one oscillator:"
- note removed: "OUT A"
- note removed: "P1"
- note removed: "P2"
- note removed: "P3"
- note removed: "RF-MOD's R1: three 18 ohm resistors to one node, 6 dB per path, no isolation between the outputs beyond those 6 dB."
- note removed: "Split OUT A with X5 to drive X1's and X2's LO inputs (-1 dBm each at the top power setting)."
- note removed: "X5 splitter, 3 x 18 ohm, 6 dB"
- note removed: "and 2.4 GHz (VCO / 2) at ICP 2.56 mA (RSET 5.1 k, CP = 7). RFOUTA+ feeds the jack through 27 nH to 3.3 V and"
- note removed: "and IP2). ADJ 1.5 k to 5 V suits 0.4-3 GHz (open it above 5 GHz). With X3 through X5 on both LOs: one coherent radio."
- note removed: "the radar's and the network analyzer's phase reference. Any two tiles can share a source through it."
- note removed: "tied high, LE has 100 k down. REF IN is unterminated (3.3 V CMOS from the ECP5 board's CLK OUT or RF-MOD's REF OUT)."
- moved on the sheet: C302, C303, C304, C305, C306, C307, C308, C309, C310, C311, C312, C313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

Commit message: Silk case convention on all six boards (Jason, Prompt 17: "To distinguish whole-tile labels from SMA or port labels, use different cases")
Ports (the jacks' names, terminal and loop names, a port named inside a note) stay UPPER CASE.  A tile's label (its
title on the frame, its name in the corner) is Mixed case: the first letter capitalised and the rest as written ("RC
low-pass", "Synthesizer", "I/Q demodulator"; tiles.label_case).  Ranges, values and notes are lower case except units,
acronyms and part numbers ("loss 1.7 dB", "OUT floats").  RF-MOD-2's X1 and X2 take word titles with their chips in
the info; RF-MOD's and RF-MOD-2's LNA tiles are titled "Preamp" ("Low-noise amp" does not fit a cell's frame); a few
two-line labels moved 0.15-0.3 mm for the descenders mixed case brings.  AMOD-P2's tile records (tile_docs), its DOA
list, KIT.md's AMOD-P2 section; X5's calibration points at P14.  All six boards: ERC 0, DRC 0, all fab checks.

Co-Authored-By: Claude Opus 5.5 <noreply@anthropic.com>
Claude-Session: https://claude.ai/code/session_01RKeoKvFFzjk3cEBLCXXHnB
Changed lines of the file:
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@@
 	(wire
 		(pts
+			(xy 370.84 441.96) (xy 365.76 441.96)
+		)
+		(stroke
+			(width 0)
+			(type default)
+		)
+	)
+	(wire
+		(pts
+			(xy 751.84 314.96) (xy 746.76 314.96)
+		)
+		(stroke
+			(width 0)
+			(type default)
+		)
+	)
+	(wire
+		(pts
 			(xy 264.16 111.76) (xy 261.62 111.76)
 		)
@@
 	(wire
 		(pts
-			(xy 365.76 314.96) (xy 370.84 314.96)
-		)
-		(stroke
-			(width 0)
-			(type default)
-		)
-	)
-	(wire
-		(pts
 			(xy 419.1 447.04) (xy 419.1 449.58)
 		)
@@
 	(wire
 		(pts
-			(xy 314.96 187.96) (xy 320.04 187.96)
-		)
-		(stroke
-			(width 0)
-			(type default)
-		)
-	)
-	(wire
-		(pts
 			(xy 619.76 241.3) (xy 622.3 241.3)
 		)
@@
 	(wire
 		(pts
+			(xy 180.34 60.96) (xy 175.26 60.96)
+		)
+		(stroke
+			(width 0)
+			(type default)
+		)
+	)
+	(wire
+		(pts
 			(xy 190.5 500.38) (xy 193.04 500.38)
 		)
@@
 	(wire
 		(pts
+			(xy 370.84 60.96) (xy 365.76 60.96)
+		)
+		(stroke
+			(width 0)
+			(type default)
+		)
+	)
+	(wire
+		(pts
 			(xy 279.4 76.2) (xy 276.86 76.2)
 		)
@@
 	(wire
 		(pts
+			(xy 726.44 314.96) (xy 721.36 314.96)
+		)
+		(stroke
+			(width 0)
+			(type default)
+		)
+	)
+	(wire
+		(pts
 			(xy 173.99 471.17) (xy 176.53 471.17)
 		)
@@
 	(wire
 		(pts
-			(xy 147.32 365.76) (xy 144.78 365.76)
+			(xy 345.44 441.96) (xy 340.36 441.96)
 		)
 		(stroke
@@
 	(wire
 		(pts
-			(xy 668.02 81.28) (xy 668.02 83.82)
+			(xy 147.32 365.76) (xy 144.78 365.76)
 		)
 		(stroke
@@
 	(wire
 		(pts
-			(xy 429.26 226.06) (xy 431.8 226.06)
+			(xy 668.02 81.28) (xy 668.02 83.82)
 		)
 		(stroke
@@
 	(wire
 		(pts
-			(xy 452.12 200.66) (xy 454.66 200.66)
+			(xy 429.26 226.06) (xy 431.8 226.06)
 		)
 		(stroke
@@
 	(wire
 		(pts
-			(xy 109.22 454.66) (xy 109.22 457.2)
+			(xy 452.12 200.66) (xy 454.66 200.66)
 		)
 		(stroke
@@
 	(wire
 		(pts
-			(xy 495.3 238.76) (xy 497.84 238.76)
+			(xy 109.22 454.66) (xy 109.22 457.2)
 		)
 		(stroke
@@
 	(wire
 		(pts
-			(xy 264.16 99.06) (xy 261.62 99.06)
+			(xy 495.3 238.76) (xy 497.84 238.76)
 		)
 		(stroke
@@
 	(wire
 		(pts
-			(xy 556.26 60.96) (xy 561.34 60.96)
+			(xy 264.16 99.06) (xy 261.62 99.06)
 		)
 		(stroke
@@
 	(wire
 		(pts
-			(xy 203.2 454.66) (xy 200.66 454.66)
+			(xy 751.84 60.96) (xy 746.76 60.96)
 		)
 		(stroke
@@
 	(wire
 		(pts
-			(xy 487.68 238.76) (xy 485.14 238.76)
+			(xy 203.2 454.66) (xy 200.66 454.66)
 		)
 		(stroke
@@
 	(wire
 		(pts
-			(xy 147.32 353.06) (xy 144.78 353.06)
+			(xy 487.68 238.76) (xy 485.14 238.76)
 		)
 		(stroke
@@
 	(wire
 		(pts
-			(xy 421.64 99.06) (xy 419.1 99.06)
+			(xy 147.32 353.06) (xy 144.78 353.06)
 		)
 		(stroke
@@
 	(wire
 		(pts
-			(xy 38.1 447.04) (xy 38.1 449.58)
+			(xy 421.64 99.06) (xy 419.1 99.06)
 		)
 		(stroke
@@
 	(wire
 		(pts
-			(xy 114.3 205.74) (xy 116.84 205.74)
+			(xy 38.1 447.04) (xy 38.1 449.58)
 		)
 		(stroke
@@
 	(wire
 		(pts
-			(xy 535.94 332.74) (xy 533.4 332.74)
+			(xy 114.3 205.74) (xy 116.84 205.74)
 		)
 		(stroke
@@
 	(wire
 		(pts
-			(xy 721.36 441.96) (xy 726.44 441.96)
+			(xy 535.94 332.74) (xy 533.4 332.74)
 		)
 		(stroke
@@
 	(wire
 		(pts
-			(xy 340.36 187.96) (xy 345.44 187.96)
-		)
-		(stroke
-			(width 0)
-			(type default)
-		)
-	)
-	(wire
-		(pts
 			(xy 490.22 365.76) (xy 492.76 365.76)
 		)
@@
 	(wire
 		(pts
-			(xy 556.26 187.96) (xy 561.34 187.96)
-		)
-		(stroke
-			(width 0)
-			(type default)
-		)
-	)
-	(wire
-		(pts
 			(xy 176.53 443.23) (xy 176.53 445.77)
 		)
@@
 	(wire
 		(pts
-			(xy 365.76 60.96) (xy 370.84 60.96)
-		)
-		(stroke
-			(width 0)
-			(type default)
-		)
-	)
-	(wire
-		(pts
 			(xy 76.2 353.06) (xy 73.66 353.06)
 		)
@@
 	(wire
 		(pts
-			(xy 365.76 187.96) (xy 370.84 187.96)
-		)
-		(stroke
-			(width 0)
-			(type default)
-		)
-	)
-	(wire
-		(pts
-			(xy 340.36 441.96) (xy 345.44 441.96)
-		)
-		(stroke
-			(width 0)
-			(type default)
-		)
-	)
-	(wire
-		(pts
 			(xy 48.26 223.52) (xy 50.8 223.52)
 		)
@@
 	(wire
 		(pts
+			(xy 561.34 187.96) (xy 556.26 187.96)
+		)
+		(stroke
+			(width 0)
+			(type default)
+		)
+	)
+	(wire
+		(pts
 			(xy 551.18 353.06) (xy 553.72 353.06)
 		)
@@
 	(wire
 		(pts
-			(xy 746.76 60.96) (xy 751.84 60.96)
-		)
-		(stroke
-			(width 0)
-			(type default)
-		)
-	)
-	(wire
-		(pts
 			(xy 71.12 459.74) (xy 73.66 459.74)
 		)
@@
 	(wire
 		(pts
-			(xy 746.76 441.96) (xy 751.84 441.96)
-		)
-		(stroke
-			(width 0)
-			(type default)
-		)
-	)
-	(wire
-		(pts
 			(xy 739.14 78.74) (xy 741.68 78.74)
 		)
@@
 	(wire
 		(pts
-			(xy 721.36 314.96) (xy 726.44 314.96)
-		)
-		(stroke
-			(width 0)
-			(type default)
-		)
-	)
-	(wire
-		(pts
 			(xy 454.66 251.46) (xy 452.12 251.46)
 		)
@@
 	(wire
 		(pts
-			(xy 175.26 60.96) (xy 180.34 60.96)
+			(xy 111.76 454.66) (xy 109.22 454.66)
 		)
 		(stroke
@@
 	(wire
 		(pts
-			(xy 111.76 454.66) (xy 109.22 454.66)
+			(xy 287.02 81.28) (xy 287.02 83.82)
 		)
 		(stroke
@@
 	(wire
 		(pts
-			(xy 287.02 81.28) (xy 287.02 83.82)
+			(xy 660.4 76.2) (xy 657.86 76.2)
 		)
 		(stroke
@@
 	(wire
 		(pts
-			(xy 660.4 76.2) (xy 657.86 76.2)
+			(xy 762 241.3) (xy 764.54 241.3)
 		)
 		(stroke
@@
 	(wire
 		(pts
-			(xy 762 241.3) (xy 764.54 241.3)
+			(xy 683.26 73.66) (xy 680.72 73.66)
 		)
 		(stroke
@@
 	(wire
 		(pts
-			(xy 683.26 73.66) (xy 680.72 73.66)
+			(xy 320.04 187.96) (xy 314.96 187.96)
 		)
 		(stroke
@@
 	(wire
 		(pts
+			(xy 561.34 60.96) (xy 556.26 60.96)
+		)
+		(stroke
+			(width 0)
+			(type default)
+		)
+	)
+	(wire
+		(pts
 			(xy 702.31 186.69) (xy 704.85 186.69)
 		)
@@
 	(wire
 		(pts
+			(xy 370.84 187.96) (xy 365.76 187.96)
+		)
+		(stroke
+			(width 0)
+			(type default)
+		)
+	)
+	(wire
+		(pts
 			(xy 261.62 365.76) (xy 264.16 365.76)
 		)
@@
 	(wire
 		(pts
+			(xy 370.84 314.96) (xy 365.76 314.96)
+		)
+		(stroke
+			(width 0)
+			(type default)
+		)
+	)
+	(wire
+		(pts
 			(xy 647.7 109.22) (xy 650.24 109.22)
 		)
@@
 	(wire
 		(pts
-			(xy 365.76 441.96) (xy 370.84 441.96)
-		)
-		(stroke
-			(width 0)
-			(type default)
-		)
-	)
-	(wire
-		(pts
 			(xy 726.44 228.6) (xy 728.98 228.6)
 		)
@@
 	(wire
 		(pts
+			(xy 751.84 441.96) (xy 746.76 441.96)
+		)
+		(stroke
+			(width 0)
+			(type default)
+		)
+	)
+	(wire
+		(pts
 			(xy 182.88 365.76) (xy 180.34 365.76)
 		)
@@
 	(wire
 		(pts
-			(xy 746.76 314.96) (xy 751.84 314.96)
+			(xy 238.76 124.46) (xy 241.3 124.46)
 		)
 		(stroke
@@
 	(wire
 		(pts
-			(xy 238.76 124.46) (xy 241.3 124.46)
+			(xy 695.96 365.76) (xy 693.42 365.76)
 		)
 		(stroke
@@
 	(wire
 		(pts
-			(xy 695.96 365.76) (xy 693.42 365.76)
+			(xy 726.44 441.96) (xy 721.36 441.96)
 		)
 		(stroke
@@
 		)
 		(stroke
+			(width 0)
+			(type default)
+		)
+	)
+	(wire
+		(pts
+			(xy 345.44 187.96) (xy 340.36 187.96)
+		)
+		(stroke
