File: hardware/amod_p2.kicad_sch (KiCad schematic)
At the start: 84 parts, among them J1401 SMA, J1402 SMA, J1403 SMA, J1404 SMA, J1405 SMA, J1406 SMA, J1501 SMA, J1502 SMA, J1601 SMA, J1602 SMA, J1603 SMA, J1701 SMA, J1702 SMA, J1703 SMA, J1801 SMA, J1802 SMA, J1901 SMA, J1902 SMA, J2001 SMA, J2002 SMA, J2101 SMA, J2102 SMA, J2201 SMA, J2202 SMA, J2203 Pmod, J2301 SMA, J2302 SMA, J2401 SMA, J2402 SMA, J2501 SMA, J2502 SMA, Q2301 AO3401A, Q2302 MMBT3904, SW2301 ON, SW2501 LOAD, T2401 TC1-1TG2+, T2501 TC4-1W+, U1701 ADP-2-1+, U2201 PE43711

Commit message: Back-side panels on all six boards; P22 set by hand or by the FPGA; P15 dropped
Jason, Prompt 18: "I hope that the silkscreen (including on the back) is appropriately used to document anything that a
user definitely needs to know to use the tiles successfully and without damaging anything.  If there is additional room
on the back, putting plots of expected responses or other relevant parameters would be great."

- gen_pcb.back_panels: under each tile, mirrored on the back silk, its number and title and the lines in its board's
  BACK dict (levels, loads, supplies, cautions), and where there is one its expected response as a small plot
  (BACK_PLOTS, or the ladder tiles' own simulation; scripts/backplots.py for the rest: amplifiers, datasheet tables,
  the open stub, P23's tuning curve, P10's clipping curve).  A panel goes as one block or in two to four parts, each
  below the one before, clear of the back's tracks and vias where it can be; every panel and plot placed, DRC 0.
- Front silk: Y2 says PULSES ONLY, Y10 "start at mV", R5 and X4 their input level (IN -20 dBm) in place of the noise
  figure.
- P22 (PE43711) on two cells with an 8-way DIP switch: way 1 SPI, ways 2-8 the bits (direct parallel mode with LE pulled
  high), 100 k pull-downs; it still needs the Pmod's 3.3 V.  P15 (two Smith-chart loads) dropped for the cell; P23 moved
  to (3,0).

Co-Authored-By: Claude Opus 5.5 <noreply@anthropic.com>
Claude-Session: https://claude.ai/code/session_01RKeoKvFFzjk3cEBLCXXHnB
Parts:
- removed C1501: 150p, Capacitor_SMD:C_0402_1005Metric, symbol Device:C
- removed J1501, J1502: SMA, amod:SMA_BWSMA-KE-Z001_Vertical, symbol Connector:Conn_Coaxial
- removed L1501: 1.5u, Inductor_SMD:L_0603_1608Metric, symbol Device:L
- removed R1501, R1502: 200, Resistor_SMD:R_0402_1005Metric, symbol Device:R_US
- added R2201, R2202, R2203, R2204, R2205, R2206, R2207, R2208, R2209: 100k, Resistor_SMD:R_0402_1005Metric, symbol Device:R_US
- added SW2201: SPI / dB, amod:SW_DIP_SPSTx08_Slide_1.27mm_DSHP08, symbol Switch:SW_DIP_x08
Connections:
- net GND: now also C2201.2, R2201.2, R2202.2, R2203.2, R2204.2, R2205.2, R2206.2, R2207.2, R2208.2; no longer C2203.2, U2201.1 (C0.25), U2201.19 (C16), U2201.20 (C8), U2201.21 (C4), U2201.22 (C2), U2201.23 (C1), U2201.24 (C0.5)
- net P22_IN: now also C2202.1; no longer C2201.1
- net P22_OUT: now also C2203.2; no longer C2202.1
- net P22_RA: now also C2202.2; no longer C2201.2
- net P22_RB: now also C2203.1; no longer C2202.2
- net PMOD4: now also R2209.1
- net PMOD_VCC: now also C2201.1, R2209.2, SW2201.10, SW2201.11, SW2201.12, SW2201.13, SW2201.14, SW2201.15, SW2201.16, SW2201.9; no longer C2203.1, U2201.3 (P/S)
- new net P22_B0: R2202.1, SW2201.2, U2201.1 (C0.25)
- new net P22_B1: R2203.1, SW2201.3, U2201.24 (C0.5)
- new net P22_B2: R2204.1, SW2201.4, U2201.23 (C1)
- new net P22_B3: R2205.1, SW2201.5, U2201.22 (C2)
- new net P22_B4: R2206.1, SW2201.6, U2201.21 (C4)
- new net P22_B5: R2207.1, SW2201.7, U2201.20 (C8)
- new net P22_B6: R2208.1, SW2201.8, U2201.19 (C16)
- new net P22_PS: R2201.1, SW2201.1, U2201.3 (P/S)
Other:
- note added: "EXPECT: 0 to 31.75 dB in 0.25 dB steps (1.5-2.8 dB of loss at 0 dB, rising with frequency), set by the switches or by an 8-bit word over the Pmod"
- note added: "FPGA's pin floats). By the FPGA: every bit off, SPI on, then shift 8 bits (bit 7 = 0, then 4 x dB, least significant"
- note added: "cells (0,3), (1,3)"
- note added: "first) on SDATA (IO2) with SCLK (IO3) while LE (IO4) is low, and raise LE. Either way it needs the Pmod's 3.3 V."
- note added: "pSemi PE43711. By hand: SPI off, the bits on the switch (direct parallel mode: P/S low, LE held high by 100 k when the"
- note removed: "200 OHM"
- note removed: "An L-network: 1.5 uH in series from the jack, 150 pF and 200 ohm to ground. Z = j w L + 200 / (1 + j w 200 C) is 50 ohm"
- note removed: "EXPECT: 0 to 31.75 dB in 0.25 dB steps (1.5-2.8 dB of loss at 0 dB, rising with frequency), set by an 8-bit word over the Pmod; 31.75 dB at power-up"
- note removed: "EXPECT: 200 OHM: Gamma = +0.6 (VSWR 4) at every frequency below 100 MHz. MATCHED: Gamma = 0 at 9.2 MHz, |Gamma| 0.5 at about 5 and 14 MHz"
- note removed: "MATCHED"
- note removed: "P15 two loads"
- note removed: "SCLK (IO3) while LE (IO4) is low, then raise LE. RF-MOD's MAX2871 and TRF3722 take the same three lines' timing."
- note removed: "cell (0,3)"
- note removed: "cell (1,3)"
- note removed: "pSemi PE43711 in serial mode: shift 8 bits (bit 7 = 0, then 4 x dB, least significant first) on SDATA (IO2) with"
- note removed: "where w 200 C = sqrt(3), 9.2 MHz; away from it the point circles the chart. The 200 ohm alone is the unmatched load."
- moved on the sheet: C2201, C2202, C2203, C2301, C2302, C2303, C2304, C2305, C2306, D2301, J2202, J2203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
