File: hardware/rf_mod_2.kicad_pcb (KiCad board)
At the start: 4 copper layers, 100 x 100 mm, 186 parts, among them J1001 USB-C, J101 SMA, J102 SMA, J103 SMA, J104 SMA, J1101 SMA, J1102 SMA, J1103 SMA, J201 SMA, J202 SMA, J203 SMA, J204 SMA, J301 SMA, J302 SMA, J303 SMA, J304 Pmod, J401 SMA, J402 SMA, J501 SMA, J502 SMA, J503 SMA, J504 SMA, J601 SMA, J602 SMA, J701 SMA, J801 SMA, J802 SMA, J901 SMA, J902 SMA, Q101 AO3401A, Q201 AO3401A, Q301 AO3401A, Q401 AO3401A, Q601 AO3401A, Q701 AO3401A, Q702 MMBT3904, Q801 AO3401A, SW101 ON, SW201 ON, SW301 ON, SW401 ON, SW601 ON, SW701 ON, SW801 ON, U1001 LM2664, U101 ADL5375, U1101 SKY13370, U201 ADL5380, U202 OPA810, U203 OPA810, U301 3.3V, U302 MAX2871, U401 QPL9547, U501 HHM22137A1, U502 HHM22137A1, U601 AD8318, U701 TPS22917, U702 ADL5611, U801 MAX2659, U802 3.3V

Commit message: Back-side panels on all six boards; P22 set by hand or by the FPGA; P15 dropped
Jason, Prompt 18: "I hope that the silkscreen (including on the back) is appropriately used to document anything that a
user definitely needs to know to use the tiles successfully and without damaging anything.  If there is additional room
on the back, putting plots of expected responses or other relevant parameters would be great."

- gen_pcb.back_panels: under each tile, mirrored on the back silk, its number and title and the lines in its board's
  BACK dict (levels, loads, supplies, cautions), and where there is one its expected response as a small plot
  (BACK_PLOTS, or the ladder tiles' own simulation; scripts/backplots.py for the rest: amplifiers, datasheet tables,
  the open stub, P23's tuning curve, P10's clipping curve).  A panel goes as one block or in two to four parts, each
  below the one before, clear of the back's tracks and vias where it can be; every panel and plot placed, DRC 0.
- Front silk: Y2 says PULSES ONLY, Y10 "start at mV", R5 and X4 their input level (IN -20 dBm) in place of the noise
  figure.
- P22 (PE43711) on two cells with an 8-way DIP switch: way 1 SPI, ways 2-8 the bits (direct parallel mode with LE pulled
  high), 100 k pull-downs; it still needs the Pmod's 3.3 V.  P15 (two Smith-chart loads) dropped for the cell; P23 moved
  to (3,0).

Co-Authored-By: Claude Opus 5.5 <noreply@anthropic.com>
Claude-Session: https://claude.ai/code/session_01RKeoKvFFzjk3cEBLCXXHnB
Other:
- board text added: "+20 dBm: 50 uT"
- board text added: "+22 dBm BURNS"
- board text added: "+30 dBm max"
- board text added: "+35 dBm through"
- board text added: "-60 to 0 dBm"
- board text added: "0.4-6 GHz"
- board text added: "0.5-6 GHz"
- board text added: "0.6G"
- board text added: "25 mV per dB"
- board text added: "3.5G"
- board text added: "50 ohm on an unused one"
- board text added: "50 ohm on an unused port"
- board text added: "50 ohm through"
- board text added: "ANT: 3.3 V on"
- board text added: "DC block for a"
- board text added: "FWD 0 to -40 dB"
- board text added: "FWD, REFL -25 dB"
- board text added: "I, Q +-1 V into 50 ohm"
- board text added: "IN -20 dBm"
- board text added: "IN < -20 dBm"
- board text added: "IO5, IO8 opposite"
- board text added: "IO6 high: on"
- board text added: "LO 0 dBm from X3"
- board text added: "OUT A+, A-: -4 to +5 dBm"
- board text added: "OUT: high-Z"
- board text added: "REF IN: the host's CLK OUT"
- board text added: "RF -4 dBm: +-1 V out"
- board text added: "USB-C 5 V; -5 V 40 mA"
- board text added: "X1 I/Q modulator"
- board text added: "X10 Power"
- board text added: "X11 Switch"
- board text added: "X2 I/Q demodulator"
- board text added: "X3 Synthesizer"
- board text added: "X4 Preamp"
- board text added: "X5 Coupler"
- board text added: "X6 Power meter"
- board text added: "X7 Noise source"
- board text added: "X8 GNSS preamp"
- board text added: "X9 ODMR loop"
- board text added: "calibrate ENR"
- board text added: "no metal near"
- board text added: "pad a strong signal"
- board text added: "passive antenna"
- board text added: "the centre pin:"
- board text removed: "NF 0.3 dB"
