File: hardware/amod_b.kicad_sch (KiCad schematic)
At the start: 147 parts, among them J1001 SMA, J1002 SMA, J101 USB-C, J102 rails, J1101 SMA, J1201 SMA, J201 SMA, J202 5-12V, J301 SMA, J302 SMA, J303 SMA, J304 motor, J305 Pmod, J401 SMA, J402 SMA, J701 SMA, J801 SMA, J802 piezo, J901 SMA, Q301 AO3401A, SW301 ON, U1001 OPA810, U1002 OPA810, U101 LM2664, U102 3.3V, U1101 INA240, U1102 OPA810, U1201 INA181, U1202 OPA810, U301 DRV8311H, U302 TLV3501, U401 OPA2171, U501 MT6701, U502 DRV5055, U503 DRV5055, U504 QRE1113, U601 LSM6DSO, U602 74LVC1G125, U701 OPA810, U801 OPA810, U901 OPA810

Commit message: Pre-order checks from CLAUDE_PCB.md's new lessons (Prompt 21): the KF301 terminals turned for their wire openings (CPL +180, body 3.7 / 4.0, a wire-face check), four oversold parts swapped (27R, 6.8k, 220n, OPA847IDBVT at its own +180), fourteen vias moved out of SMD pads (check_layout.py gates it and RF detours), 200-250 mW terminations, assembly drawings from Fab and silk fitted to Letter (fit_pdf.py from CostasLink), the stock gate on JLCPCB's free count, electrolytics in the rotation check, the RF gates surveyed (rf_extract.py, rf_survey.py) and written into the DOA lists; all nine boards rebuilt: ERC 0, DRC 0, every check
Co-Authored-By: Claude Opus 5.5 <noreply@anthropic.com>
Claude-Session: https://claude.ai/code/session_01RKeoKvFFzjk3cEBLCXXHnB
Parts:
- R1006, R1012, R1107, R1208, R201, R301, R407, R408, R706, R803, R903: LCSC C25120 -> C844112; MPN 0402WGF499JTCE -> CRCW040249R9FKEDHP
Changed lines of the file:
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@@
 			)
 		)
-		(property "LCSC" "C25120"
+		(property "LCSC" "C844112"
 			(at 516.89 99.06 90)
 			(hide yes)
@@
 			)
 		)
-		(property "MPN" "0402WGF499JTCE"
+		(property "MPN" "CRCW040249R9FKEDHP"
 			(at 516.89 99.06 90)
 			(hide yes)
@@
 			)
 		)
-		(property "LCSC" "C25120"
+		(property "LCSC" "C844112"
 			(at 44.45 236.22 90)
 			(hide yes)
@@
 			)
 		)
-		(property "MPN" "0402WGF499JTCE"
+		(property "MPN" "CRCW040249R9FKEDHP"
 			(at 44.45 236.22 90)
 			(hide yes)
@@
 			)
 		)
-		(property "LCSC" "C25120"
+		(property "LCSC" "C844112"
 			(at 74.93 492.76 90)
 			(hide yes)
@@
 			)
 		)
-		(property "MPN" "0402WGF499JTCE"
+		(property "MPN" "CRCW040249R9FKEDHP"
 			(at 74.93 492.76 90)
 			(hide yes)
@@
 			)
 		)
-		(property "LCSC" "C25120"
+		(property "LCSC" "C844112"
 			(at 412.75 492.76 90)
 			(hide yes)
@@
 			)
 		)
-		(property "MPN" "0402WGF499JTCE"
+		(property "MPN" "CRCW040249R9FKEDHP"
 			(at 412.75 492.76 90)
 			(hide yes)
@@
 			)
 		)
-		(property "LCSC" "C25120"
+		(property "LCSC" "C844112"
 			(at 44.45 111.76 90)
 			(hide yes)
@@
 			)
 		)
-		(property "MPN" "0402WGF499JTCE"
+		(property "MPN" "CRCW040249R9FKEDHP"
 			(at 44.45 111.76 90)
 			(hide yes)
@@
 			)
 		)
-		(property "LCSC" "C25120"
+		(property "LCSC" "C844112"
 			(at 748.03 365.76 90)
 			(hide yes)
@@
 			)
 		)
-		(property "MPN" "0402WGF499JTCE"
+		(property "MPN" "CRCW040249R9FKEDHP"
 			(at 748.03 365.76 90)
 			(hide yes)
@@
 			)
 		)
-		(property "LCSC" "C25120"
+		(property "LCSC" "C844112"
 			(at 646.43 99.06 90)
 			(hide yes)
@@
 			)
 		)
-		(property "MPN" "0402WGF499JTCE"
+		(property "MPN" "CRCW040249R9FKEDHP"
 			(at 646.43 99.06 90)
 			(hide yes)
@@
 			)
 		)
-		(property "LCSC" "C25120"
+		(property "LCSC" "C844112"
 			(at 676.91 492.76 90)
 			(hide yes)
@@
 			)
 		)
-		(property "MPN" "0402WGF499JTCE"
+		(property "MPN" "CRCW040249R9FKEDHP"
 			(at 676.91 492.76 90)
 			(hide yes)
@@
 			)
 		)
-		(property "LCSC" "C25120"
+		(property "LCSC" "C844112"
 			(at 77.47 248.92 90)
 			(hide yes)
@@
 			)
 		)
-		(property "MPN" "0402WGF499JTCE"
+		(property "MPN" "CRCW040249R9FKEDHP"
 			(at 77.47 248.92 90)
 			(hide yes)
@@
 			)
 		)
-		(property "LCSC" "C25120"
+		(property "LCSC" "C844112"
 			(at 326.39 99.06 90)
 			(hide yes)
@@
 			)
 		)
-		(property "MPN" "0402WGF499JTCE"
+		(property "MPN" "CRCW040249R9FKEDHP"
 			(at 326.39 99.06 90)
 			(hide yes)
@@
 			)
 		)
-		(property "LCSC" "C25120"
+		(property "LCSC" "C844112"
 			(at 105.41 492.76 90)
 			(hide yes)
@@
 			)
 		)
-		(property "MPN" "0402WGF499JTCE"
+		(property "MPN" "CRCW040249R9FKEDHP"
 			(at 105.41 492.76 90)
 			(hide yes)
