File: hardware/amod_m.kicad_sch (KiCad schematic)
At the start: 207 parts, among them J1001 SMA, J101 USB-C, J102 rails, J1101 SMA, J1102 cell, J201 SMA, J202 5-16V, J301 SMA, J302 SMA, J303 motor, J304 Pmod, J401 SMA, J402 SMA, J403 stepper, J501 SMA, J502 SMA, J503 servo, J601 SMA, J602 SMA, J603 SMA, J604 coil, J605 D Z, J701 SMA, J702 SMA, J703 load, J801 SMA, J802 SMA, J803 SMA, J804 out, J901 SMA, Q1001 AO3401A, Q301 AO3401A, Q401 AO3401A, Q501 AO3401A, Q601 AO3401A, Q602 NCE6020AK, Q801 AO3401A, Q802 AO3400A, Q803 AO3400A, Q901 AO3401A, SW1001 ON, SW301 ON, SW401 ON, SW501 ON, SW601 ON, SW801 ON, SW901 ON, U1001 QRE1113, U1002 OPA810, U101 LM2664, U102 3.3V, U1101 INA828, U301 DRV8251A, U302 OPA2171, U303 3.3V, U401 DRV8251A, U402 DRV8251A, U501 TLV3501, U502 INA181, U601 TLV3501, U602 INA181, U701 TCA0372, U702 INA181, U703 OPA810, U801 TLV3501, U802 TPS28225, U803 INA181, U901 DRV5055, U902 OPA810

Commit message: Pre-order checks from CLAUDE_PCB.md's new lessons (Prompt 21): the KF301 terminals turned for their wire openings (CPL +180, body 3.7 / 4.0, a wire-face check), four oversold parts swapped (27R, 6.8k, 220n, OPA847IDBVT at its own +180), fourteen vias moved out of SMD pads (check_layout.py gates it and RF detours), 200-250 mW terminations, assembly drawings from Fab and silk fitted to Letter (fit_pdf.py from CostasLink), the stock gate on JLCPCB's free count, electrolytics in the rotation check, the RF gates surveyed (rf_extract.py, rf_survey.py) and written into the DOA lists; all nine boards rebuilt: ERC 0, DRC 0, every check
Co-Authored-By: Claude Opus 5.5 <noreply@anthropic.com>
Claude-Session: https://claude.ai/code/session_01RKeoKvFFzjk3cEBLCXXHnB
Parts:
- C804: LCSC C47129 -> C16772; MPN CL05A224KA5NNNC -> CL05B224KO5NNNC
- R1004, R1102, R201, R304, R306, R501, R506, R601, R605, R608, R611, R705, R717, R801, R807, R810, R906: LCSC C25120 -> C844112; MPN 0402WGF499JTCE -> CRCW040249R9FKEDHP
Changed lines of the file:
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@@
 			)
 		)
-		(property "LCSC" "C25120"
+		(property "LCSC" "C844112"
 			(at 209.55 480.06 90)
 			(hide yes)
@@
 			)
 		)
-		(property "MPN" "0402WGF499JTCE"
+		(property "MPN" "CRCW040249R9FKEDHP"
 			(at 209.55 480.06 90)
 			(hide yes)
@@
 			)
 		)
-		(property "LCSC" "C25120"
+		(property "LCSC" "C844112"
 			(at 367.03 223.52 90)
 			(hide yes)
@@
 			)
 		)
-		(property "MPN" "0402WGF499JTCE"
+		(property "MPN" "CRCW040249R9FKEDHP"
 			(at 367.03 223.52 90)
 			(hide yes)
@@
 			)
 		)
-		(property "LCSC" "C25120"
+		(property "LCSC" "C844112"
 			(at 110.49 111.76 90)
 			(hide yes)
@@
 			)
 		)
-		(property "MPN" "0402WGF499JTCE"
+		(property "MPN" "CRCW040249R9FKEDHP"
 			(at 110.49 111.76 90)
 			(hide yes)
@@
 			)
 		)
-		(property "LCSC" "C25120"
+		(property "LCSC" "C844112"
 			(at 458.47 223.52 90)
 			(hide yes)
@@
 			)
 		)
-		(property "MPN" "0402WGF499JTCE"
+		(property "MPN" "CRCW040249R9FKEDHP"
 			(at 458.47 223.52 90)
 			(hide yes)
@@
 			)
 		)
-		(property "LCSC" "C25120"
+		(property "LCSC" "C844112"
 			(at 275.59 480.06 90)
 			(hide yes)
@@
 			)
 		)
-		(property "MPN" "0402WGF499JTCE"
+		(property "MPN" "CRCW040249R9FKEDHP"
 			(at 275.59 480.06 90)
 			(hide yes)
@@
 			)
 		)
-		(property "LCSC" "C25120"
+		(property "LCSC" "C844112"
 			(at 730.25 365.76 90)
 			(hide yes)
@@
 			)
 		)
-		(property "MPN" "0402WGF499JTCE"
+		(property "MPN" "CRCW040249R9FKEDHP"
 			(at 730.25 365.76 90)
 			(hide yes)
@@
 			)
 		)
-		(property "LCSC" "C25120"
+		(property "LCSC" "C844112"
 			(at 209.55 99.06 90)
 			(hide yes)
@@
 			)
 		)
-		(property "MPN" "0402WGF499JTCE"
+		(property "MPN" "CRCW040249R9FKEDHP"
 			(at 209.55 99.06 90)
 			(hide yes)
@@
 			)
 		)
-		(property "LCSC" "C25120"
+		(property "LCSC" "C844112"
 			(at 341.63 99.06 90)
 			(hide yes)
@@
 			)
 		)
-		(property "MPN" "0402WGF499JTCE"
+		(property "MPN" "CRCW040249R9FKEDHP"
 			(at 341.63 99.06 90)
 			(hide yes)
@@
 			)
 		)
-		(property "LCSC" "C25120"
+		(property "LCSC" "C844112"
 			(at 669.29 353.06 90)
 			(hide yes)
@@
 			)
 		)
-		(property "MPN" "0402WGF499JTCE"
+		(property "MPN" "CRCW040249R9FKEDHP"
 			(at 669.29 353.06 90)
 			(hide yes)
@@
 			)
 		)
-		(property "LCSC" "C25120"
+		(property "LCSC" "C844112"
 			(at 44.45 99.06 90)
 			(hide yes)
@@
 			)
 		)
-		(property "MPN" "0402WGF499JTCE"
+		(property "MPN" "CRCW040249R9FKEDHP"
 			(at 44.45 99.06 90)
 			(hide yes)
@@
 			)
 		)
-		(property "LCSC" "C25120"
+		(property "LCSC" "C844112"
 			(at 557.53 492.76 90)
 			(hide yes)
@@
 			)
 		)
-		(property "MPN" "0402WGF499JTCE"
+		(property "MPN" "CRCW040249R9FKEDHP"
 			(at 557.53 492.76 90)
 			(hide yes)
@@
 			)
 		)
-		(property "LCSC" "C25120"
+		(property "LCSC" "C844112"
 			(at 656.59 492.76 90)
 			(hide yes)
@@
 			)
 		)
-		(property "MPN" "0402WGF499JTCE"
+		(property "MPN" "CRCW040249R9FKEDHP"
 			(at 656.59 492.76 90)
 			(hide yes)
@@
 			)
 		)
-		(property "LCSC" "C47129"
+		(property "LCSC" "C16772"
 			(at 689.61 480.06 90)
 			(hide yes)
@@
 			)
 		)
-		(property "MPN" "CL05A224KA5NNNC"
+		(property "MPN" "CL05B224KO5NNNC"
 			(at 689.61 480.06 90)
 			(hide yes)
@@
 			)
 		)
-		(property "LCSC" "C25120"
+		(property "LCSC" "C844112"
 			(at 74.93 241.3 90)
 			(hide yes)
@@
 			)
 		)
-		(property "MPN" "0402WGF499JTCE"
+		(property "MPN" "CRCW040249R9FKEDHP"
 			(at 74.93 241.3 90)
 			(hide yes)
@@
 			)
 		)
-		(property "LCSC" "C25120"
+		(property "LCSC" "C844112"
 			(at 425.45 99.06 90)
 			(hide yes)
@@
 			)
 		)
-		(property "MPN" "0402WGF499JTCE"
+		(property "MPN" "CRCW040249R9FKEDHP"
 			(at 425.45 99.06 90)
 			(hide yes)
@@
 			)
 		)
-		(property "LCSC" "C25120"
+		(property "LCSC" "C844112"
 			(at 646.43 99.06 90)
 			(hide yes)
@@
 			)
 		)
-		(property "MPN" "0402WGF499JTCE"
+		(property "MPN" "CRCW040249R9FKEDHP"
 			(at 646.43 99.06 90)
 			(hide yes)
@@
 			)
 		)
-		(property "LCSC" "C25120"
+		(property "LCSC" "C844112"
 			(at 486.41 111.76 90)
 			(hide yes)
@@
 			)
 		)
-		(property "MPN" "0402WGF499JTCE"
+		(property "MPN" "CRCW040249R9FKEDHP"
 			(at 486.41 111.76 90)
 			(hide yes)
@@
 			)
 		)
-		(property "LCSC" "C25120"
+		(property "LCSC" "C844112"
 			(at 458.47 480.06 90)
 			(hide yes)
@@
 			)
 		)
-		(property "MPN" "0402WGF499JTCE"
+		(property "MPN" "CRCW040249R9FKEDHP"
 			(at 458.47 480.06 90)
 			(hide yes)
