File: hardware/amod_n.kicad_sch (KiCad schematic)
At the start: 88 parts, among them J1001 SMA, J1002 SMA, J101 SMA, J102 SMA, J103 SMA, J104 SMA, J105 SMA, J106 SMA, J1101 SMA, J1102 SMA, J201 SMA, J202 SMA, J203 SMA, J301 SMA, J302 SMA, J303 SMA, J401 SMA, J402 SMA, J501 SMA, J502 SMA, J601 SMA, J602 SMA, J701 SMA, J702 SMA, J801 SMA, J802 SMA, J803 Pmod, J901 SMA, J902 SMA, Q901 AO3401A, Q902 MMBT3904, SW1101 LOAD, SW801 SPI / dB, SW901 ON, T1001 TC1-1TG2+, T1101 TC4-1W+, U301 ADP-2-1+, U801 PE43711

Commit message: Pre-order checks from CLAUDE_PCB.md's new lessons (Prompt 21): the KF301 terminals turned for their wire openings (CPL +180, body 3.7 / 4.0, a wire-face check), four oversold parts swapped (27R, 6.8k, 220n, OPA847IDBVT at its own +180), fourteen vias moved out of SMD pads (check_layout.py gates it and RF detours), 200-250 mW terminations, assembly drawings from Fab and silk fitted to Letter (fit_pdf.py from CostasLink), the stock gate on JLCPCB's free count, electrolytics in the rotation check, the RF gates surveyed (rf_extract.py, rf_survey.py) and written into the DOA lists; all nine boards rebuilt: ERC 0, DRC 0, every check
Co-Authored-By: Claude Opus 5.5 <noreply@anthropic.com>
Claude-Session: https://claude.ai/code/session_01RKeoKvFFzjk3cEBLCXXHnB
Parts:
- R103, R104, R1102: LCSC C25120 -> C844112; MPN 0402WGF499JTCE -> CRCW040249R9FKEDHP
Changed lines of the file:
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@@
 			)
 		)
-		(property "LCSC" "C25120"
+		(property "LCSC" "C844112"
 			(at 110.49 99.06 90)
 			(hide yes)
@@
 			)
 		)
-		(property "MPN" "0402WGF499JTCE"
+		(property "MPN" "CRCW040249R9FKEDHP"
 			(at 110.49 99.06 90)
 			(hide yes)
@@
 			)
 		)
-		(property "LCSC" "C25120"
+		(property "LCSC" "C844112"
 			(at 646.43 480.06 90)
 			(hide yes)
@@
 			)
 		)
-		(property "MPN" "0402WGF499JTCE"
+		(property "MPN" "CRCW040249R9FKEDHP"
 			(at 646.43 480.06 90)
 			(hide yes)
@@
 			)
 		)
-		(property "LCSC" "C25120"
+		(property "LCSC" "C844112"
 			(at 143.51 99.06 90)
 			(hide yes)
@@
 			)
 		)
-		(property "MPN" "0402WGF499JTCE"
+		(property "MPN" "CRCW040249R9FKEDHP"
 			(at 143.51 99.06 90)
 			(hide yes)
