File: hardware/amod_p.kicad_pcb (KiCad board)
At the start: 2 copper layers, 100 x 100 mm, 151 parts, among them J1001 SMA, J1002 SMA, J101 SMA, J102 SMA, J1101 SMA, J1102 SMA, J1103 SMA, J1104 SMA, J1105 SMA, J1201 SMA, J1301 SMA, J1302 coil, J1303 VAR C, J201 SMA, J202 SMA, J301 SMA, J302 SMA, J401 SMA, J402 SMA, J501 SMA, J502 SMA, J601 SMA, J602 SMA, J701 SMA, J702 SMA, J801 SMA, J802 SMA, J901 SMA, J902 SMA, SW1201 DIP4, SW1301 DIP4, SW401 DIP2, Y801 4 MHz, Y901 455 kHz

Commit message: One letter per board, tiles in lower case: AMOD-P2 is AMOD-N (n1-n11), RF-MOD-2 is IQ-MOD (q1-q11), PhMOD's tiles h1-h10
Jason, Prompt 19: "If we can have a nice, well justified single-letter designator for each board, it would make
everything much more clear", and "d11, q11, and c11 don't look like obvious electronics or PCB things".

- p passive, n networks (AMOD-P2's P14, P16-P25), a active, r radio, h PhMOD (Y1-Y10), q quadrature (RF-MOD-2's X1-X11);
  c, m and b are taken for the conversion, motor and brushless boards to come.  PLAN.md section 13 has the table and
  the reasons (no letter moves to another board, no retired name is reused, no s: s11 is the reflection coefficient).
- Every tile name in lower case on the silk, in the code (Tile ids, BACK/BACK_PLOTS/DOCS keys, the nets built on them),
  the handbooks, README, DOA lists, KIT, PLAN and the review brief; pin names (USB-C A1...), the 4046's R1/C1, nets
  named N1/P1, part numbers ending -R7 and the paper size A1 left alone.  tiles.dump refuses a tile not named
  <letter><n>, a number twice, and a BACK key for a tile that does not exist.
- Board and file renames: boards/amod_n.py, boards/iq_mod.py, docs/DOA_amod_n.md, docs/DOA_iq_mod.md, the handbooks,
  the generated hardware, outputs and pictures.  Silk nudged where a lower-case p or q hung onto the line below.
- All six boards rebuilt: ERC 0, DRC 0, every check.

Co-Authored-By: Claude Opus 5.5 <noreply@anthropic.com>
Claude-Session: https://claude.ai/code/session_01RKeoKvFFzjk3cEBLCXXHnB
Connections:
- net /P10_IN renamed /p10_IN
- net /P10_OUT renamed /p10_OUT
- net /P11_OUT renamed /p11_OUT
- net /P11_T1 renamed /p11_T1
- net /P11_T2 renamed /p11_T2
- net /P11_T3 renamed /p11_T3
- net /P12_BUS renamed /p12_BUS
- net /P13_HOT renamed /p13_HOT
- net /P13_TAP renamed /p13_TAP
- net /P1_IN renamed /p1_IN
- net /P1_OUT renamed /p1_OUT
- net /P2_IN renamed /p2_IN
- net /P2_OUT renamed /p2_OUT
- net /P3_IN renamed /p3_IN
- net /P3_OUT renamed /p3_OUT
- net /P4_IN renamed /p4_IN
- net /P4_N1 renamed /p4_N1
- net /P4_OUT renamed /p4_OUT
- net /P5_IN renamed /p5_IN
- net /P5_N1 renamed /p5_N1
- net /P5_OUT renamed /p5_OUT
- net /P6_IN renamed /p6_IN
- net /P6_OUT renamed /p6_OUT
- net /P7_IN renamed /p7_IN
- net /P7_N1 renamed /p7_N1
- net /P7_N2 renamed /p7_N2
- net /P7_N3 renamed /p7_N3
- net /P7_OUT renamed /p7_OUT
- net /P8_IN renamed /p8_IN
- net /P8_OUT renamed /p8_OUT
- net /P9_IN renamed /p9_IN
- net /P9_OUT renamed /p9_OUT
Other:
- board text added: "expected response. p13: a 330 uH ferrite-rod coil along this edge, under cable ties; a tuning capacitor on VAR C."
- board text added: "p1"
- board text added: "p1 Pi pad"
- board text added: "p10"
- board text added: "p10 Clipper"
- board text added: "p11"
- board text added: "p11 Delay line"
- board text added: "p12"
- board text added: "p12 LEDs"
- board text added: "p13"
- board text added: "p13 AM loopstick"
- board text added: "p2"
- board text added: "p2 RC low-pass"
- board text added: "p3"
- board text added: "p3 RC high-pass"
- board text added: "p4"
- board text added: "p4 Series RLC"
- board text added: "p5"
- board text added: "p5 LC low-pass"
- board text added: "p6"
- board text added: "p6 LC low-pass"
- board text added: "p7"
- board text added: "p7 Band-pass"
- board text added: "p8"
- board text added: "p8 Quartz crystal"
- board text added: "p9"
- board text added: "p9 Ceramic res."
- board text added: "then a4's LNA"
- board text removed: "P1"
- board text removed: "P1 Pi pad"
- board text removed: "P10"
- board text removed: "P10 Clipper"
- board text removed: "P11"
- board text removed: "P11 Delay line"
- board text removed: "P12"
- board text removed: "P12 LEDs"
- board text removed: "P13"
- board text removed: "P13 AM loopstick"
- board text removed: "P2"
- board text removed: "P2 RC low-pass"
- board text removed: "P3"
- board text removed: "P3 RC high-pass"
- board text removed: "P4"
- board text removed: "P4 Series RLC"
- board text removed: "P5"
- board text removed: "P5 LC low-pass"
- board text removed: "P6"
- board text removed: "P6 LC low-pass"
- board text removed: "P7"
- board text removed: "P7 Band-pass"
- board text removed: "P8"
- board text removed: "P8 Quartz crystal"
- board text removed: "P9"
- board text removed: "P9 Ceramic res."
- board text removed: "expected response. P13: a 330 uH ferrite-rod coil along this edge, under cable ties; a tuning capacitor on VAR C."
- board text removed: "then A4's LNA"

Commit message: Pre-order checks from CLAUDE_PCB.md's new lessons (Prompt 21): the KF301 terminals turned for their wire openings (CPL +180, body 3.7 / 4.0, a wire-face check), four oversold parts swapped (27R, 6.8k, 220n, OPA847IDBVT at its own +180), fourteen vias moved out of SMD pads (check_layout.py gates it and RF detours), 200-250 mW terminations, assembly drawings from Fab and silk fitted to Letter (fit_pdf.py from CostasLink), the stock gate on JLCPCB's free count, electrolytics in the rotation check, the RF gates surveyed (rf_extract.py, rf_survey.py) and written into the DOA lists; all nine boards rebuilt: ERC 0, DRC 0, every check
Co-Authored-By: Claude Opus 5.5 <noreply@anthropic.com>
Claude-Session: https://claude.ai/code/session_01RKeoKvFFzjk3cEBLCXXHnB
Changed lines of the file:
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@@
 		(duplicate_pad_numbers_are_jumpers no)
 		(fp_line
-			(start 5.3 3.7)
-			(end -5.3 3.7)
+			(start 5.3 4.1)
+			(end -5.3 4.1)
 			(stroke
 				(width 0.15)
@@
 		)
 		(fp_line
-			(start 5.3 -4.1)
-			(end 5.3 3.7)
+			(start 5.3 -3.8)
+			(end 5.3 4.1)
 			(stroke
 				(width 0.15)
@@
 		)
 		(fp_line
-			(start 4 -4.1)
-			(end 4 -2.8)
+			(start 4 -3.8)
+			(end 4 -2.5)
 			(stroke
 				(width 0.15)
@@
 		)
 		(fp_line
-			(start 1 -2.8)
-			(end 4 -2.8)
+			(start 1 -2.5)
+			(end 4 -2.5)
 			(stroke
 				(width 0.15)
@@
 		)
 		(fp_line
-			(start 1 -4.1)
-			(end 1 -2.8)
+			(start 1 -3.8)
+			(end 1 -2.5)
 			(stroke
 				(width 0.15)
@@
 		)
 		(fp_line
-			(start -1 -4.1)
-			(end -1 -2.8)
+			(start -1 -3.8)
+			(end -1 -2.5)
 			(stroke
 				(width 0.15)
@@
 		)
 		(fp_line
-			(start -4 -2.8)
-			(end -1 -2.8)
+			(start -4 -2.5)
+			(end -1 -2.5)
 			(stroke
 				(width 0.15)
@@
 		)
 		(fp_line
-			(start -4 -4.1)
-			(end -4 -2.8)
+			(start -4 -3.8)
+			(end -4 -2.5)
 			(stroke
 				(width 0.15)
@@
 		)
 		(fp_line
-			(start -5.3 3.7)
-			(end -5.3 -4.1)
+			(start -5.3 4.1)
+			(end -5.3 -3.8)
 			(stroke
 				(width 0.15)
@@
 		)
 		(fp_line
-			(start -5.3 -4.1)
-			(end 5.3 -4.1)
+			(start -5.3 -3.8)
+			(end 5.3 -3.8)
 			(stroke
 				(width 0.15)
@@
 		)
 		(fp_line
-			(start 5.55 3.95)
-			(end -5.55 3.95)
+			(start 5.55 4.35)
+			(end -5.55 4.35)
 			(stroke
 				(width 0.05)
@@
 		)
 		(fp_line
-			(start 5.55 -4.35)
-			(end 5.55 3.95)
+			(start 5.55 -4.05)
+			(end 5.55 4.35)
 			(stroke
 				(width 0.05)
@@
 		)
 		(fp_line
-			(start -5.55 3.95)
-			(end -5.55 -4.35)
+			(start -5.55 4.35)
+			(end -5.55 -4.05)
 			(stroke
 				(width 0.05)
@@
 		)
 		(fp_line
-			(start -5.55 -4.35)
-			(end 5.55 -4.35)
+			(start -5.55 -4.05)
+			(end 5.55 -4.05)
 			(stroke
 				(width 0.05)
@@
 		)
 		(fp_line
-			(start 5.2 3.6)
-			(end -5.2 3.6)
+			(start 5.2 4)
+			(end -5.2 4)
 			(stroke
 				(width 0.1)
@@
 		)
 		(fp_line
-			(start 5.2 -4)
-			(end 5.2 3.6)
+			(start 5.2 -3.7)
+			(end 5.2 4)
 			(stroke
 				(width 0.1)
@@
 		)
 		(fp_line
-			(start -5.2 3.6)
-			(end -5.2 -4)
+			(start -5.2 4)
+			(end -5.2 -3.7)
 			(stroke
 				(width 0.1)
@@
 		)
 		(fp_line
-			(start -5.2 -4)
-			(end 5.2 -4)
+			(start -5.2 -3.7)
+			(end 5.2 -3.7)
 			(stroke
 				(width 0.1)
@@
 		(duplicate_pad_numbers_are_jumpers no)
 		(fp_line
-			(start 7.8 3.7)
-			(end -7.8 3.7)
+			(start 7.8 4.1)
+			(end -7.8 4.1)
 			(stroke
 				(width 0.15)
@@
 		)
 		(fp_line
-			(start 7.8 -4.1)
-			(end 7.8 3.7)
+			(start 7.8 -3.8)
+			(end 7.8 4.1)
 			(stroke
 				(width 0.15)
@@
 		)
 		(fp_line
-			(start 6.5 -4.1)
-			(end 6.5 -2.8)
+			(start 6.5 -3.8)
+			(end 6.5 -2.5)
 			(stroke
 				(width 0.15)
@@
 		)
 		(fp_line
-			(start 3.5 -2.8)
-			(end 6.5 -2.8)
+			(start 3.5 -2.5)
+			(end 6.5 -2.5)
 			(stroke
 				(width 0.15)
@@
 		)
 		(fp_line
-			(start 3.5 -4.1)
-			(end 3.5 -2.8)
+			(start 3.5 -3.8)
+			(end 3.5 -2.5)
 			(stroke
 				(width 0.15)
@@
 		)
 		(fp_line
-			(start 1.5 -4.1)
-			(end 1.5 -2.8)
+			(start 1.5 -3.8)
+			(end 1.5 -2.5)
 			(stroke
 				(width 0.15)
@@
 		)
 		(fp_line
-			(start -1.5 -2.8)
-			(end 1.5 -2.8)
+			(start -1.5 -2.5)
+			(end 1.5 -2.5)
 			(stroke
 				(width 0.15)
@@
 		)
 		(fp_line
-			(start -1.5 -4.1)
-			(end -1.5 -2.8)
+			(start -1.5 -3.8)
+			(end -1.5 -2.5)
 			(stroke
 				(width 0.15)
@@
 		)
 		(fp_line
-			(start -3.5 -4.1)
-			(end -3.5 -2.8)
+			(start -3.5 -3.8)
+			(end -3.5 -2.5)
 			(stroke
 				(width 0.15)
@@
 		)
 		(fp_line
-			(start -6.5 -2.8)
-			(end -3.5 -2.8)
+			(start -6.5 -2.5)
+			(end -3.5 -2.5)
 			(stroke
 				(width 0.15)
@@
 		)
 		(fp_line
-			(start -6.5 -4.1)
-			(end -6.5 -2.8)
+			(start -6.5 -3.8)
+			(end -6.5 -2.5)
 			(stroke
 				(width 0.15)
@@
 		)
 		(fp_line
-			(start -7.8 3.7)
-			(end -7.8 -4.1)
+			(start -7.8 4.1)
+			(end -7.8 -3.8)
 			(stroke
 				(width 0.15)
@@
 		)
 		(fp_line
-			(start -7.8 -4.1)
-			(end 7.8 -4.1)
+			(start -7.8 -3.8)
+			(end 7.8 -3.8)
 			(stroke
 				(width 0.15)
@@
 		)
 		(fp_line
-			(start 8.05 3.95)
-			(end -8.05 3.95)
+			(start 8.05 4.35)
+			(end -8.05 4.35)
 			(stroke
 				(width 0.05)
@@
 		)
 		(fp_line
-			(start 8.05 -4.35)
-			(end 8.05 3.95)
+			(start 8.05 -4.05)
+			(end 8.05 4.35)
 			(stroke
 				(width 0.05)
@@
 		)
 		(fp_line
-			(start -8.05 3.95)
-			(end -8.05 -4.35)
+			(start -8.05 4.35)
+			(end -8.05 -4.05)
 			(stroke
 				(width 0.05)
@@
 		)
 		(fp_line
-			(start -8.05 -4.35)
-			(end 8.05 -4.35)
+			(start -8.05 -4.05)
+			(end 8.05 -4.05)
 			(stroke
 				(width 0.05)
@@
 		)
 		(fp_line
-			(start 7.7 3.6)
-			(end -7.7 3.6)
+			(start 7.7 4)
+			(end -7.7 4)
 			(stroke
 				(width 0.1)
@@
 		)
 		(fp_line
-			(start 7.7 -4)
-			(end 7.7 3.6)
+			(start 7.7 -3.7)
+			(end 7.7 4)
 			(stroke
 				(width 0.1)
@@
 		)
 		(fp_line
-			(start -7.7 3.6)
-			(end -7.7 -4)
+			(start -7.7 4)
+			(end -7.7 -3.7)
 			(stroke
 				(width 0.1)
@@
 		)
 		(fp_line
-			(start -7.7 -4)
-			(end 7.7 -4)
+			(start -7.7 -3.7)
+			(end 7.7 -3.7)
 			(stroke
 				(width 0.1)
@@
 	)
 	(gr_line
-		(start 39.75 83.155)
+		(start 39.75 82.755)
 		(end 39.75 82.45)
 		(stroke
@@
 	(gr_line
 		(start 48.55 83.05)
-		(end 59.75 83.05)
+		(end 51.355 83.05)
 		(stroke
 			(width 0.3)
@@
 	)
 	(gr_line
-		(start 51.355 91.95)
-		(end 48.144999 91.95)
-		(stroke
-			(width 0.15)
-			(type default)
-		)
-		(layer "F.SilkS")
-	)
-	(gr_line
 		(start 51.55 62.68)
 		(end 51.95 62.68)
@@
 	)
 	(gr_line
-		(start 59.75 83.05)
-		(end 63.15 83.05)
-		(stroke
-			(width 0.3)
-			(type default)
-		)
-		(layer "F.SilkS")
-	)
-	(gr_line
 		(start 59.82 42.6)
 		(end 59.82 42.95)
@@
 	(gr_line
 		(start 67.555 91.95)
-		(end 63.144999 91.95)
+		(end 32.445 91.95)
 		(stroke
 			(width 0.15)
