File: hardware/iq_mod.kicad_sch (KiCad schematic)
At the start: 186 parts, among them J1001 USB-C, J101 SMA, J102 SMA, J103 SMA, J104 SMA, J1101 SMA, J1102 SMA, J1103 SMA, J201 SMA, J202 SMA, J203 SMA, J204 SMA, J301 SMA, J302 SMA, J303 SMA, J304 Pmod, J401 SMA, J402 SMA, J501 SMA, J502 SMA, J503 SMA, J504 SMA, J601 SMA, J602 SMA, J701 SMA, J801 SMA, J802 SMA, J901 SMA, J902 SMA, Q101 AO3401A, Q201 AO3401A, Q301 AO3401A, Q401 AO3401A, Q601 AO3401A, Q701 AO3401A, Q702 MMBT3904, Q801 AO3401A, SW101 ON, SW201 ON, SW301 ON, SW401 ON, SW601 ON, SW701 ON, SW801 ON, U1001 LM2664, U101 ADL5375, U1101 SKY13370, U201 ADL5380, U202 OPA810, U203 OPA810, U301 3.3V, U302 MAX2871, U401 QPL9547, U501 HHM22137A1, U502 HHM22137A1, U601 AD8318, U701 TPS22917, U702 ADL5611, U801 MAX2659, U802 3.3V

Commit message: Pre-order checks from CLAUDE_PCB.md's new lessons (Prompt 21): the KF301 terminals turned for their wire openings (CPL +180, body 3.7 / 4.0, a wire-face check), four oversold parts swapped (27R, 6.8k, 220n, OPA847IDBVT at its own +180), fourteen vias moved out of SMD pads (check_layout.py gates it and RF detours), 200-250 mW terminations, assembly drawings from Fab and silk fitted to Letter (fit_pdf.py from CostasLink), the stock gate on JLCPCB's free count, electrolytics in the rotation check, the RF gates surveyed (rf_extract.py, rf_survey.py) and written into the DOA lists; all nine boards rebuilt: ERC 0, DRC 0, every check
Co-Authored-By: Claude Opus 5.5 <noreply@anthropic.com>
Claude-Session: https://claude.ai/code/session_01RKeoKvFFzjk3cEBLCXXHnB
Parts:
- R206, R211: LCSC C25120 -> C844112; MPN 0402WGF499JTCE -> CRCW040249R9FKEDHP
Changed lines of the file:
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@@
 			)
 		)
-		(property "LCSC" "C25120"
+		(property "LCSC" "C844112"
 			(at 699.77 365.76 90)
 			(hide yes)
@@
 			)
 		)
-		(property "MPN" "0402WGF499JTCE"
+		(property "MPN" "CRCW040249R9FKEDHP"
 			(at 699.77 365.76 90)
 			(hide yes)
@@
 			)
 		)
-		(property "LCSC" "C25120"
+		(property "LCSC" "C844112"
 			(at 516.89 365.76 90)
 			(hide yes)
@@
 			)
 		)
-		(property "MPN" "0402WGF499JTCE"
+		(property "MPN" "CRCW040249R9FKEDHP"
 			(at 516.89 365.76 90)
 			(hide yes)
