File: hardware/phmod.kicad_sch (KiCad schematic)
At the start: 234 parts, among them J1001 SMA, J1002 SMA, J1003 SMA, J1004 SMA, J101 USB-C, J201 SMA, J202 SMA, J301 SMA, J302 SMA, J303 SMA, J304 SMA, J401 SMA, J402 VM in, J403 coil, J501 SMA, J502 SMA, J503 SMA, J504 SMA, J505 Pmod, J601 SMA, J602 SMA, J701 SMA, J702 SMA, J703 SMA, J704 SMA, J801 SMA, J802 SMA, J803 SMA, J804 SMA, J901 SMA, Q1001 AO3401A, Q1002 2N7002, Q1003 AO3401A, Q1004 AO3400A, Q301 AO3401A, Q401 AO3401A, Q501 AO3401A, Q601 AO3401A, Q701 AO3401A, Q801 AO3401A, Q901 AO3401A, Q902 MMBT3904, SW1001 ON, SW301 ON, SW401 ON, SW501 ON, SW601 ON, SW701 ON, SW801 ON, SW802 DIP4, SW901 ON, U1001 OPA810, U1002 OPA810, U101 TPS65131, U102 LM2664, U201 THS3491, U301 OPA847, U401 DRV8876, U402 OPA810, U501 LMH6629, U502 LMH6629, U601 OPA810, U701 OPA810, U702 OPA810, U901 TPS22917, U902 LMH6629

Commit message: Silk case convention on all six boards (Jason, Prompt 17: "To distinguish whole-tile labels from SMA or port labels, use different cases")
Ports (the jacks' names, terminal and loop names, a port named inside a note) stay UPPER CASE.  A tile's label (its
title on the frame, its name in the corner) is Mixed case: the first letter capitalised and the rest as written ("RC
low-pass", "Synthesizer", "I/Q demodulator"; tiles.label_case).  Ranges, values and notes are lower case except units,
acronyms and part numbers ("loss 1.7 dB", "OUT floats").  RF-MOD-2's X1 and X2 take word titles with their chips in
the info; RF-MOD's and RF-MOD-2's LNA tiles are titled "Preamp" ("Low-noise amp" does not fit a cell's frame); a few
two-line labels moved 0.15-0.3 mm for the descenders mixed case brings.  AMOD-P2's tile records (tile_docs), its DOA
list, KIT.md's AMOD-P2 section; X5's calibration points at P14.  All six boards: ERC 0, DRC 0, all fab checks.

Co-Authored-By: Claude Opus 5.5 <noreply@anthropic.com>
Claude-Session: https://claude.ai/code/session_01RKeoKvFFzjk3cEBLCXXHnB
Changed lines of the file:
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@@
 	(wire
 		(pts
-			(xy 340.36 60.96) (xy 345.44 60.96)
+			(xy 370.84 441.96) (xy 365.76 441.96)
+		)
+		(stroke
+			(width 0)
+			(type default)
+		)
+	)
+	(wire
+		(pts
+			(xy 751.84 314.96) (xy 746.76 314.96)
 		)
 		(stroke
@@
 	(wire
 		(pts
-			(xy 556.26 441.96) (xy 561.34 441.96)
-		)
-		(stroke
-			(width 0)
-			(type default)
-		)
-	)
-	(wire
-		(pts
 			(xy 718.82 236.22) (xy 716.28 236.22)
 		)
@@
 	(wire
 		(pts
-			(xy 340.36 314.96) (xy 345.44 314.96)
-		)
-		(stroke
-			(width 0)
-			(type default)
-		)
-	)
-	(wire
-		(pts
 			(xy 741.68 111.76) (xy 744.22 111.76)
 		)
@@
 	(wire
 		(pts
-			(xy 365.76 314.96) (xy 370.84 314.96)
+			(xy 566.42 447.04) (xy 566.42 449.58)
 		)
 		(stroke
@@
 	(wire
 		(pts
-			(xy 566.42 447.04) (xy 566.42 449.58)
+			(xy 345.44 314.96) (xy 340.36 314.96)
 		)
 		(stroke
@@
 	(wire
 		(pts
-			(xy 314.96 187.96) (xy 320.04 187.96)
-		)
-		(stroke
-			(width 0)
-			(type default)
-		)
-	)
-	(wire
-		(pts
 			(xy 513.08 492.76) (xy 510.54 492.76)
 		)
@@
 	(wire
 		(pts
+			(xy 370.84 60.96) (xy 365.76 60.96)
+		)
+		(stroke
+			(width 0)
+			(type default)
+		)
+	)
+	(wire
+		(pts
 			(xy 703.58 99.06) (xy 701.04 99.06)
 		)
@@
 	(wire
 		(pts
+			(xy 726.44 314.96) (xy 721.36 314.96)
+		)
+		(stroke
+			(width 0)
+			(type default)
+		)
+	)
+	(wire
+		(pts
 			(xy 205.74 480.06) (xy 203.2 480.06)
 		)
@@
 	(wire
 		(pts
-			(xy 668.02 81.28) (xy 668.02 83.82)
+			(xy 345.44 441.96) (xy 340.36 441.96)
 		)
 		(stroke
@@
 	(wire
 		(pts
-			(xy 429.26 492.76) (xy 431.8 492.76)
+			(xy 668.02 81.28) (xy 668.02 83.82)
 		)
 		(stroke
@@
 	(wire
 		(pts
-			(xy 147.32 492.76) (xy 149.86 492.76)
+			(xy 429.26 492.76) (xy 431.8 492.76)
 		)
 		(stroke
@@
 	(wire
 		(pts
-			(xy 728.98 457.2) (xy 726.44 457.2)
+			(xy 147.32 492.76) (xy 149.86 492.76)
 		)
 		(stroke
@@
 	(wire
 		(pts
-			(xy 81.28 223.52) (xy 83.82 223.52)
+			(xy 728.98 457.2) (xy 726.44 457.2)
 		)
 		(stroke
@@
 	(wire
 		(pts
-			(xy 759.46 228.6) (xy 762 228.6)
+			(xy 81.28 223.52) (xy 83.82 223.52)
 		)
 		(stroke
@@
 	(wire
 		(pts
-			(xy 487.68 236.22) (xy 485.14 236.22)
+			(xy 759.46 228.6) (xy 762 228.6)
 		)
 		(stroke
@@
 	(wire
 		(pts
-			(xy 180.34 492.76) (xy 182.88 492.76)
+			(xy 487.68 236.22) (xy 485.14 236.22)
 		)
 		(stroke
@@
 	(wire
 		(pts
-			(xy 556.26 60.96) (xy 561.34 60.96)
+			(xy 180.34 492.76) (xy 182.88 492.76)
 		)
 		(stroke
@@
 	(wire
 		(pts
+			(xy 751.84 60.96) (xy 746.76 60.96)
+		)
+		(stroke
+			(width 0)
+			(type default)
+		)
+	)
+	(wire
+		(pts
 			(xy 429.26 243.84) (xy 431.8 243.84)
 		)
@@
 	(wire
 		(pts
-			(xy 340.36 187.96) (xy 345.44 187.96)
-		)
-		(stroke
-			(width 0)
-			(type default)
-		)
-	)
-	(wire
-		(pts
 			(xy 452.12 492.76) (xy 449.58 492.76)
 		)
@@
 	(wire
 		(pts
-			(xy 365.76 60.96) (xy 370.84 60.96)
-		)
-		(stroke
-			(width 0)
-			(type default)
-		)
-	)
-	(wire
-		(pts
 			(xy 762 73.66) (xy 764.54 73.66)
 		)
@@
 	(wire
 		(pts
-			(xy 365.76 187.96) (xy 370.84 187.96)
-		)
-		(stroke
-			(width 0)
-			(type default)
-		)
-	)
-	(wire
-		(pts
 			(xy 619.76 515.62) (xy 622.3 515.62)
 		)
@@
 	(wire
 		(pts
-			(xy 340.36 441.96) (xy 345.44 441.96)
-		)
-		(stroke
-			(width 0)
-			(type default)
-		)
-	)
-	(wire
-		(pts
 			(xy 48.26 223.52) (xy 50.8 223.52)
 		)
@@
 	(wire
 		(pts
+			(xy 561.34 441.96) (xy 556.26 441.96)
+		)
+		(stroke
+			(width 0)
+			(type default)
+		)
+	)
+	(wire
+		(pts
 			(xy 520.7 243.84) (xy 518.16 243.84)
 		)
@@
 	(wire
 		(pts
-			(xy 746.76 60.96) (xy 751.84 60.96)
-		)
-		(stroke
-			(width 0)
-			(type default)
-		)
-	)
-	(wire
-		(pts
 			(xy 360.68 99.06) (xy 358.14 99.06)
 		)
@@
 	(wire
 		(pts
-			(xy 746.76 441.96) (xy 751.84 441.96)
-		)
-		(stroke
-			(width 0)
-			(type default)
-		)
-	)
-	(wire
-		(pts
 			(xy 566.42 175.26) (xy 568.96 175.26)
 		)
@@
 	(wire
 		(pts
-			(xy 721.36 314.96) (xy 726.44 314.96)
-		)
-		(stroke
-			(width 0)
-			(type default)
-		)
-	)
-	(wire
-		(pts
 			(xy 741.68 99.06) (xy 744.22 99.06)
 		)
@@
 	(wire
 		(pts
+			(xy 320.04 187.96) (xy 314.96 187.96)
+		)
+		(stroke
+			(width 0)
+			(type default)
+		)
+	)
+	(wire
+		(pts
 			(xy 457.2 210.82) (xy 457.2 213.36)
 		)
@@
 	(wire
 		(pts
+			(xy 561.34 60.96) (xy 556.26 60.96)
+		)
+		(stroke
+			(width 0)
+			(type default)
+		)
+	)
+	(wire
+		(pts
 			(xy 63.5 66.04) (xy 63.5 68.58)
 		)
@@
 	(wire
 		(pts
+			(xy 370.84 187.96) (xy 365.76 187.96)
+		)
+		(stroke
+			(width 0)
+			(type default)
+		)
+	)
+	(wire
+		(pts
 			(xy 703.58 73.66) (xy 706.12 73.66)
 		)
@@
 	(wire
 		(pts
+			(xy 370.84 314.96) (xy 365.76 314.96)
+		)
+		(stroke
+			(width 0)
+			(type default)
+		)
+	)
+	(wire
+		(pts
 			(xy 119.38 99.06) (xy 121.92 99.06)
 		)
@@
 	(wire
 		(pts
-			(xy 365.76 441.96) (xy 370.84 441.96)
-		)
-		(stroke
-			(width 0)
-			(type default)
-		)
-	)
-	(wire
-		(pts
 			(xy 246.38 492.76) (xy 248.92 492.76)
 		)
@@
 	(wire
 		(pts
+			(xy 751.84 441.96) (xy 746.76 441.96)
+		)
+		(stroke
+			(width 0)
+			(type default)
+		)
+	)
+	(wire
+		(pts
 			(xy 520.7 480.06) (xy 523.24 480.06)
 		)
@@
 	(wire
 		(pts
-			(xy 619.76 523.24) (xy 622.3 523.24)
+			(xy 345.44 60.96) (xy 340.36 60.96)
 		)
 		(stroke
@@
 	(wire
 		(pts
-			(xy 449.58 314.96) (xy 454.66 314.96)
+			(xy 619.76 523.24) (xy 622.3 523.24)
 		)
 		(stroke
@@
 	(wire
 		(pts
-			(xy 88.9 457.2) (xy 86.36 457.2)
+			(xy 449.58 314.96) (xy 454.66 314.96)
 		)
 		(stroke
@@
 	(wire
 		(pts
-			(xy 746.76 314.96) (xy 751.84 314.96)
+			(xy 88.9 457.2) (xy 86.36 457.2)
 		)
 		(stroke
@@
 		)
 		(stroke
+			(width 0)
+			(type default)
+		)
+	)
+	(wire
+		(pts
+			(xy 345.44 187.96) (xy 340.36 187.96)
+		)
+		(stroke

Commit message: One letter per board, tiles in lower case: AMOD-P2 is AMOD-N (n1-n11), RF-MOD-2 is IQ-MOD (q1-q11), PhMOD's tiles h1-h10
Jason, Prompt 19: "If we can have a nice, well justified single-letter designator for each board, it would make
everything much more clear", and "d11, q11, and c11 don't look like obvious electronics or PCB things".

- p passive, n networks (AMOD-P2's P14, P16-P25), a active, r radio, h PhMOD (Y1-Y10), q quadrature (RF-MOD-2's X1-X11);
  c, m and b are taken for the conversion, motor and brushless boards to come.  PLAN.md section 13 has the table and
  the reasons (no letter moves to another board, no retired name is reused, no s: s11 is the reflection coefficient).
- Every tile name in lower case on the silk, in the code (Tile ids, BACK/BACK_PLOTS/DOCS keys, the nets built on them),
  the handbooks, README, DOA lists, KIT, PLAN and the review brief; pin names (USB-C A1...), the 4046's R1/C1, nets
  named N1/P1, part numbers ending -R7 and the paper size A1 left alone.  tiles.dump refuses a tile not named
  <letter><n>, a number twice, and a BACK key for a tile that does not exist.
- Board and file renames: boards/amod_n.py, boards/iq_mod.py, docs/DOA_amod_n.md, docs/DOA_iq_mod.md, the handbooks,
  the generated hardware, outputs and pictures.  Silk nudged where a lower-case p or q hung onto the line below.
- All six boards rebuilt: ERC 0, DRC 0, every check.

Co-Authored-By: Claude Opus 5.5 <noreply@anthropic.com>
Claude-Session: https://claude.ai/code/session_01RKeoKvFFzjk3cEBLCXXHnB
Connections:
- net Y10_G renamed h10_G
- net Y10_GA renamed h10_GA
- net Y10_GB renamed h10_GB
- net Y10_GQ renamed h10_GQ
- net Y10_ID renamed h10_ID
- net Y10_LDN renamed h10_LDN
- net Y10_LM renamed h10_LM
- net Y10_MON renamed h10_MON
- net Y10_NA renamed h10_NA
- net Y10_NS renamed h10_NS
- net Y10_REF renamed h10_REF
- net Y10_RF renamed h10_RF
- net Y10_RFC renamed h10_RFC
- net Y10_SET renamed h10_SET
- net Y10_SETF renamed h10_SETF
- net Y10_SQ renamed h10_SQ
- net Y10_VS renamed h10_VS
- net Y1_CAPN renamed h1_CAPN
- net Y1_CAPP renamed h1_CAPP
- net Y1_CC1 renamed h1_CC1
- net Y1_CC2 renamed h1_CC2
- net Y1_CN renamed h1_CN
- net Y1_CP renamed h1_CP
- net Y1_FBN renamed h1_FBN
- net Y1_FBP renamed h1_FBP
- net Y1_LEDG renamed h1_LEDG
- net Y1_LEDR renamed h1_LEDR
- net Y1_LEDY renamed h1_LEDY
- net Y1_SWN renamed h1_SWN
- net Y1_SWP renamed h1_SWP
- net Y1_VBUS renamed h1_VBUS
- net Y1_VINF renamed h1_VINF
- net Y1_VREF renamed h1_VREF
- net Y2_FBO renamed h2_FBO
- net Y2_IN renamed h2_IN
- net Y2_INN renamed h2_INN
- net Y2_OUT renamed h2_OUT
- net Y2_PD renamed h2_PD
- net Y3_FB renamed h3_FB
- net Y3_G renamed h3_G
- net Y3_IN renamed h3_IN
- net Y3_M renamed h3_M
- net Y3_OUT renamed h3_OUT
- net Y3_OUT_A renamed h3_OUT_A
- net Y3_PRB renamed h3_PRB
- net Y3_TX renamed h3_TX
- net Y3_VS renamed h3_VS
- net Y4_CPH renamed h4_CPH
- net Y4_CPL renamed h4_CPL
- net Y4_G renamed h4_G
- net Y4_IP renamed h4_IP
- net Y4_MO renamed h4_MO
- net Y4_MON renamed h4_MON
- net Y4_OUT1 renamed h4_OUT1
- net Y4_OUT2 renamed h4_OUT2
- net Y4_VCP renamed h4_VCP
- net Y4_VEXT renamed h4_VEXT
- net Y4_VM renamed h4_VM
- net Y4_VREF renamed h4_VREF
- net Y4_VS renamed h4_VS
- net Y5_CG renamed h5_CG
- net Y5_CGB renamed h5_CGB
- net Y5_FB renamed h5_FB
- net Y5_FBB renamed h5_FBB
- net Y5_G renamed h5_G
- net Y5_IN renamed h5_IN
- net Y5_IN2 renamed h5_IN2
- net Y5_IN2B renamed h5_IN2B
- net Y5_INB renamed h5_INB
- net Y5_OA renamed h5_OA
- net Y5_OAB renamed h5_OAB
- net Y5_OC renamed h5_OC
- net Y5_OCB renamed h5_OCB
- net Y5_OUT renamed h5_OUT
- net Y5_OUTB renamed h5_OUTB
- net Y5_VS renamed h5_VS
- net Y6_CG renamed h6_CG
- net Y6_FB renamed h6_FB
- net Y6_G renamed h6_G
- net Y6_IN renamed h6_IN
- net Y6_IN2 renamed h6_IN2
- net Y6_OA renamed h6_OA
- net Y6_OC renamed h6_OC
- net Y6_OUT renamed h6_OUT
- net Y6_VS renamed h6_VS
- net Y7_A renamed h7_A
- net Y7_B renamed h7_B
- net Y7_DRV renamed h7_DRV
- net Y7_G renamed h7_G
- net Y7_INC renamed h7_INC
- net Y7_N1 renamed h7_N1
- net Y7_N2 renamed h7_N2
- net Y7_O1 renamed h7_O1
- net Y7_O2 renamed h7_O2
- net Y7_REFL renamed h7_REFL
- net Y7_VS renamed h7_VS
- net Y8_CA renamed h8_CA
- net Y8_CB renamed h8_CB
- net Y8_G renamed h8_G
- net Y8_K1 renamed h8_K1
- net Y8_K2 renamed h8_K2
- net Y8_OUT1 renamed h8_OUT1
- net Y8_OUT2 renamed h8_OUT2
- net Y8_RDA renamed h8_RDA
- net Y8_RDB renamed h8_RDB
- net Y8_SIG renamed h8_SIG
- net Y8_T1 renamed h8_T1
- net Y8_T2 renamed h8_T2
- net Y8_TP renamed h8_TP
- net Y8_VS renamed h8_VS
- net Y9_CG renamed h9_CG
- net Y9_FB renamed h9_FB
- net Y9_G renamed h9_G
- net Y9_IN renamed h9_IN
- net Y9_IN2 renamed h9_IN2
- net Y9_OA renamed h9_OA
- net Y9_OC renamed h9_OC
- net Y9_OUT renamed h9_OUT
- net Y9_VN renamed h9_VN
- net Y9_VS renamed h9_VS
Other:
- note added: "+15 V = 1.213 V x (1 + 1 M / 88.7 k) = 14.9 V, -15 V = -1.213 V x 1.3 M / 105 k = -15.0 V. Only h2 draws them, through"
- note added: "h1 power, USB-C 5 V in: +5, -5, +15, -15 out"
- note added: "h10 laser driver, current source + bias-T"
- note added: "h2 pulse amplifier, THS3491"
- note added: "h3 duplexer and preamp, OPA847"
- note added: "h4 coil driver, DRV8876"
- note added: "h5 HF receiver, 2 x LMH6629"
- note added: "h5's IN A, or two boards) give a lightning stroke's bearing from the ratio of the two signals."
- note added: "h6 VLF loop amplifier, OPA810 x101"
- note added: "h7 reflection bridge, 2 x OPA810"
- note added: "h8 coupled resonators, 2 x LC + BB133"
- note added: "h9 noise source, MMBT3904 + LMH6629"
- note added: "two back-side tracks; everything else runs from +5 V and the LM2664's -5 V (40 mA: h3, h7 and h9 draw about 30)."
- note removed: "+15 V = 1.213 V x (1 + 1 M / 88.7 k) = 14.9 V, -15 V = -1.213 V x 1.3 M / 105 k = -15.0 V. Only Y2 draws them, through"
- note removed: "Y1 power, USB-C 5 V in: +5, -5, +15, -15 out"
- note removed: "Y10 laser driver, current source + bias-T"
- note removed: "Y2 pulse amplifier, THS3491"
- note removed: "Y3 duplexer and preamp, OPA847"
- note removed: "Y4 coil driver, DRV8876"
- note removed: "Y5 HF receiver, 2 x LMH6629"
- note removed: "Y5's IN A, or two boards) give a lightning stroke's bearing from the ratio of the two signals."
- note removed: "Y6 VLF loop amplifier, OPA810 x101"
- note removed: "Y7 reflection bridge, 2 x OPA810"
- note removed: "Y8 coupled resonators, 2 x LC + BB133"
- note removed: "Y9 noise source, MMBT3904 + LMH6629"
- note removed: "two back-side tracks; everything else runs from +5 V and the LM2664's -5 V (40 mA: Y3, Y7 and Y9 draw about 30)."

Commit message: Pre-order checks from CLAUDE_PCB.md's new lessons (Prompt 21): the KF301 terminals turned for their wire openings (CPL +180, body 3.7 / 4.0, a wire-face check), four oversold parts swapped (27R, 6.8k, 220n, OPA847IDBVT at its own +180), fourteen vias moved out of SMD pads (check_layout.py gates it and RF detours), 200-250 mW terminations, assembly drawings from Fab and silk fitted to Letter (fit_pdf.py from CostasLink), the stock gate on JLCPCB's free count, electrolytics in the rotation check, the RF gates surveyed (rf_extract.py, rf_survey.py) and written into the DOA lists; all nine boards rebuilt: ERC 0, DRC 0, every check
Co-Authored-By: Claude Opus 5.5 <noreply@anthropic.com>
Claude-Session: https://claude.ai/code/session_01RKeoKvFFzjk3cEBLCXXHnB
Parts:
- C104: LCSC C47129 -> C16772; MPN CL05A224KA5NNNC -> CL05B224KO5NNNC
- R1001, R203, R301, R406, R501, R506, R507, R512, R605, R701, R702, R703, R706, R709, R801, R906: LCSC C25120 -> C844112; MPN 0402WGF499JTCE -> CRCW040249R9FKEDHP
- R303: LCSC C23185 -> C6230117; MPN 0603WAF499JT5E -> SR0603FR-7T49R9L
- R505, R511, R905: LCSC C25100 -> C100353; MPN 0402WGF270JTCE -> CR0402FF27R0G
- U301: LCSC C160422 -> C2059024; MPN OPA847IDBVR -> OPA847IDBVT
Changed lines of the file:
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@@
 			)
 		)
-		(property "LCSC" "C25120"
+		(property "LCSC" "C844112"
 			(at 425.45 353.06 90)
 			(hide yes)
@@
 			)
 		)
-		(property "MPN" "0402WGF499JTCE"
+		(property "MPN" "CRCW040249R9FKEDHP"
 			(at 425.45 353.06 90)
 			(hide yes)
@@
 			)
 		)
-		(property "LCSC" "C25100"
+		(property "LCSC" "C100353"
 			(at 176.53 492.76 90)
 			(hide yes)
@@
 			)
 		)
-		(property "MPN" "0402WGF270JTCE"
+		(property "MPN" "CR0402FF27R0G"
 			(at 176.53 492.76 90)
 			(hide yes)
@@
 			)
 		)
-		(property "LCSC" "C25120"
+		(property "LCSC" "C844112"
 			(at 44.45 223.52 90)
 			(hide yes)
@@
 			)
 		)
-		(property "MPN" "0402WGF499JTCE"
+		(property "MPN" "CRCW040249R9FKEDHP"
 			(at 44.45 223.52 90)
 			(hide yes)
@@
 			)
 		)
-		(property "LCSC" "C160422"
+		(property "LCSC" "C2059024"
 			(at 119.38 76.2 0)
 			(hide yes)
@@
 			)
 		)
-		(property "MPN" "OPA847IDBVR"
+		(property "MPN" "OPA847IDBVT"
 			(at 119.38 76.2 0)
 			(hide yes)
@@
 			)
 		)
-		(property "LCSC" "C25100"
+		(property "LCSC" "C100353"
 			(at 737.87 111.76 90)
 			(hide yes)
@@
 			)
 		)
-		(property "MPN" "0402WGF270JTCE"
+		(property "MPN" "CR0402FF27R0G"
 			(at 737.87 111.76 90)
 			(hide yes)
@@
 			)
 		)
-		(property "LCSC" "C25120"
+		(property "LCSC" "C844112"
 			(at 374.65 480.06 90)
 			(hide yes)
@@
 			)
 		)
-		(property "MPN" "0402WGF499JTCE"
+		(property "MPN" "CRCW040249R9FKEDHP"
 			(at 374.65 480.06 90)
 			(hide yes)
@@
 			)
 		)
-		(property "LCSC" "C25120"
+		(property "LCSC" "C844112"
 			(at 516.89 492.76 90)
 			(hide yes)
@@
 			)
 		)
-		(property "MPN" "0402WGF499JTCE"
+		(property "MPN" "CRCW040249R9FKEDHP"
 			(at 516.89 492.76 90)
 			(hide yes)
@@
 			)
 		)
-		(property "LCSC" "C25120"
+		(property "LCSC" "C844112"
 			(at 486.41 99.06 90)
 			(hide yes)
@@
 			)
 		)
-		(property "MPN" "0402WGF499JTCE"
+		(property "MPN" "CRCW040249R9FKEDHP"
 			(at 486.41 99.06 90)
 			(hide yes)
@@
 			)
 		)
-		(property "LCSC" "C25120"
+		(property "LCSC" "C844112"
 			(at 257.81 99.06 90)
 			(hide yes)
@@
 			)
 		)
-		(property "MPN" "0402WGF499JTCE"
+		(property "MPN" "CRCW040249R9FKEDHP"
 			(at 257.81 99.06 90)
 			(hide yes)
@@
 			)
 		)
-		(property "LCSC" "C25120"
+		(property "LCSC" "C844112"
 			(at 209.55 223.52 90)
 			(hide yes)
@@
 			)
 		)
-		(property "MPN" "0402WGF499JTCE"
+		(property "MPN" "CRCW040249R9FKEDHP"
 			(at 209.55 223.52 90)
 			(hide yes)
@@
 			)
 		)
-		(property "LCSC" "C25120"
+		(property "LCSC" "C844112"
 			(at 308.61 223.52 90)
 			(hide yes)
@@
 			)
 		)
-		(property "MPN" "0402WGF499JTCE"
+		(property "MPN" "CRCW040249R9FKEDHP"
 			(at 308.61 223.52 90)
 			(hide yes)
@@
 			)
 		)
-		(property "LCSC" "C25120"
+		(property "LCSC" "C844112"
 			(at 275.59 492.76 90)
 			(hide yes)
@@
 			)
 		)
-		(property "MPN" "0402WGF499JTCE"
+		(property "MPN" "CRCW040249R9FKEDHP"
 			(at 275.59 492.76 90)
 			(hide yes)
@@
 			)
 		)
-		(property "LCSC" "C25120"
+		(property "LCSC" "C844112"
 			(at 77.47 223.52 90)
 			(hide yes)
@@
 			)
 		)
-		(property "MPN" "0402WGF499JTCE"
+		(property "MPN" "CRCW040249R9FKEDHP"
 			(at 77.47 223.52 90)
 			(hide yes)
@@
 			)
 		)
-		(property "LCSC" "C25120"
+		(property "LCSC" "C844112"
 			(at 676.91 124.46 90)
 			(hide yes)
@@
 			)
 		)
-		(property "MPN" "0402WGF499JTCE"
+		(property "MPN" "CRCW040249R9FKEDHP"
 			(at 676.91 124.46 90)
 			(hide yes)
@@
 			)
 		)
-		(property "LCSC" "C25120"
+		(property "LCSC" "C844112"
 			(at 44.45 480.06 90)
 			(hide yes)
@@
 			)
 		)
-		(property "MPN" "0402WGF499JTCE"
+		(property "MPN" "CRCW040249R9FKEDHP"
 			(at 44.45 480.06 90)
 			(hide yes)
@@
 			)
 		)
-		(property "LCSC" "C47129"
+		(property "LCSC" "C16772"
 			(at 557.53 228.6 90)
 			(hide yes)
@@
 			)
 		)
-		(property "MPN" "CL05A224KA5NNNC"
+		(property "MPN" "CL05B224KO5NNNC"
 			(at 557.53 228.6 90)
 			(hide yes)
@@
 			)
 		)
-		(property "LCSC" "C25100"
+		(property "LCSC" "C100353"
 			(at 209.55 480.06 90)
 			(hide yes)
@@
 			)
 		)
-		(property "MPN" "0402WGF270JTCE"
+		(property "MPN" "CR0402FF27R0G"
 			(at 209.55 480.06 90)
 			(hide yes)
@@
 			)
 		)
-		(property "LCSC" "C25120"
+		(property "LCSC" "C844112"
 			(at 308.61 480.06 90)
 			(hide yes)
@@
 			)
 		)
-		(property "MPN" "0402WGF499JTCE"
+		(property "MPN" "CRCW040249R9FKEDHP"
 			(at 308.61 480.06 90)
 			(hide yes)
@@
 			)
 		)
-		(property "LCSC" "C25120"
+		(property "LCSC" "C844112"
 			(at 44.45 353.06 90)
 			(hide yes)
@@
 			)
 		)
-		(property "MPN" "0402WGF499JTCE"
+		(property "MPN" "CRCW040249R9FKEDHP"
 			(at 44.45 353.06 90)
 			(hide yes)
@@
 			)
 		)
-		(property "LCSC" "C23185"
+		(property "LCSC" "C6230117"
 			(at 364.49 99.06 90)
 			(hide yes)
@@
 			)
 		)
-		(property "MPN" "0603WAF499JT5E"
+		(property "MPN" "SR0603FR-7T49R9L"
 			(at 364.49 99.06 90)
 			(hide yes)
@@
 			)
 		)
-		(property "LCSC" "C25120"
+		(property "LCSC" "C844112"
 			(at 110.49 223.52 90)
 			(hide yes)
@@
 			)
 		)
-		(property "MPN" "0402WGF499JTCE"
+		(property "MPN" "CRCW040249R9FKEDHP"
 			(at 110.49 223.52 90)
 			(hide yes)
@@
 			)
 		)
-		(property "LCSC" "C25120"
+		(property "LCSC" "C844112"
 			(at 615.95 523.24 90)
 			(hide yes)
@@
 			)
 		)
-		(property "MPN" "0402WGF499JTCE"
+		(property "MPN" "CRCW040249R9FKEDHP"
 			(at 615.95 523.24 90)
 			(hide yes)
